File: plate/plate.kicad_pcb (KiCad board)
At the start: 2 copper layers, 299 x 122.8 mm, 73 parts

Commit message: M  border.py A  notes/cnc.md M  notes/components.md M  notes/nRF52840.md M  notes/notes.md A  notes/parts M  pcb/pcb.kicad_pcb M  plate/plate.kicad_pcb
Other:
- board size 299 x 122.8 mm -> 299.5 x 123 mm

Commit message: M  border.py M  notes/cnc.md M  notes/nRF52840.md M  notes/notes.md M  pcb/pcb.kicad_pcb M  pcb/pcb.kicad_sch M  pcb/sym-lib-table M  place.py M  plate/plate.kicad_pcb M  plate/plate.kicad_sch A  tmr-footprints/IS31FL3731-SSOP-28_5.3x10.2mm_P0.65mm.kicad_mod A  tmr-footprints/MCP3208-SOIC-16_3.9x9.9mm_P1.27mm.kicad_mod M  tmr-footprints/sw_lowpro_combo_MDT.kicad_mod D  tmr-footprints/sw_lowpro_combo_MDT_led.kicad_mod
Parts:
- S1: footprint tmr-lib:Switch_Cutout_1.25u -> tmr-lib:Switch_Cutout
- moved S1 2.38 mm to (19.0, 0.00)
Other:
- outline, holes or cut-outs redrawn
