File: plate/plate.kicad_sch (KiCad schematic)
At the start: 73 parts

Commit message: M  border.py M  place.py M  plate/plate.kicad_pcb M  plate/plate.kicad_sch
Parts:
- S63: footprint tmr-lib:Switch_Cutout2_MX_1.25u -> tmr-lib:Switch_Cutout2_MX
Changed lines of the file:
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@@
 			)
 		)
-		(property "Footprint" "tmr-lib:Switch_Cutout2_MX_1.25u"
+		(property "Footprint" "tmr-lib:Switch_Cutout2_MX"
 			(at 102.87 91.44 0)
 			(effects

Commit message: A  RP2040_Minimal.kicad_sym A  RP2040_minimal.pretty/8-USON-Handsolder.kicad_mod A  RP2040_minimal.pretty/8-USON.kicad_mod A  RP2040_minimal.pretty/C_0402_1005Metric.kicad_mod A  RP2040_minimal.pretty/C_0603_1608Metric.kicad_mod A  RP2040_minimal.pretty/C_0603_1608Metric_Pad1.08x0.95mm_HandSolder.kicad_mod A  RP2040_minimal.pretty/C_1206_3216Metric.kicad_mod A  RP2040_minimal.pretty/Crystal_SMD_2520-4Pin_2.5x2.0mm-Handsolder.kicad_mod A  RP2040_minimal.pretty/Crystal_SMD_HC49-US.kicad_mod A  RP2040_minimal.pretty/D_0402_1005Metric.kicad_mod A  RP2040_minimal.pretty/D_SOD-523.kicad_mod A  RP2040_minimal.pretty/Diodes_U_DFN1212_3.kicad_mod A  RP2040_minimal.pretty/Diodes_U_DFN1212_3_Handsolder.kicad_mod A  RP2040_minimal.pretty/LED_0402_1005Metric.kicad_mod A  RP2040_minimal.pretty/LED_Driver_Mod_Conn.kicad_mod A  RP2040_minimal.pretty/LED_Driver_Mod_Conn_1.27.kicad_mod A  RP2040_minimal.pretty/Module_Conn_Regular.kicad_mod A  RP2040_minimal.pretty/Module_Conn_Regular2.kicad_mod A  RP2040_minimal.pretty/Module_Conn_Regular_Outline.kicad_mod A  RP2040_minimal.pretty/QFN-28-1EP_4x4mm_P0.4mm_EP2.3x2.3mm-Handsolder.kicad_mod A  RP2040_minimal.pretty/QFN-28-1EP_4x4mm_P0.4mm_EP2.3x2.3mm.kicad_mod A  RP2040_minimal.pretty/RP2040-QFN-56-Handsolder.kicad_mod A  RP2040_minimal.pretty/RP2040-QFN-56.kicad_mod A  RP2040_minimal.pretty/R_0402_1005Metric.kicad_mod A  RP2040_minimal.pretty/R_0603_1608Metric_Pad0.98x0.95mm_HandSolder.kicad_mod A  RP2040_minimal.pretty/SW_CK_KXT3.kicad_mod A  RP2040_minimal.pretty/SW_SPST_Panasonic_EVPAF.kicad_mod A  RP2040_minimal.pretty/SW_Side_EVPAV.kicad_mod A  RP2040_minimal.pretty/SW_XKB_TS_2030.kicad_mod A  RP2040_minimal.pretty/USB_Micro-B_Amphenol_10103594-0001LF_Horizontal_modified.kicad_mod A  RP2040_minimal.pretty/XSON-8-1EP_4x4mm.kicad_mod M  border.py M  notes/notes.md M  pcb/fp-lib-table M  pcb/pcb.kicad_pcb M  pcb/pcb.kicad_prl M  pcb/pcb.kicad_sch M  plate/plate.kicad_pcb M  plate/plate.kicad_sch R  tmr-footprints/Switch_Cutout2_MX.kic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
Parts:
- S1, S10, S11, S12, S13, S14, S15, S16, S17, S18, S19, S2, S20, S21, S22, S23, S24, S25, S26, S27, S28, S29, S3, S31, S32, S33, S34, S35, S36, S37, S38, S39, S4, S40, S41, S43, S44, S47, S48, S49, S5, S50, S51, S52, S53, S54, S55, S56, S58, S6, S61, S63, S65, S67, S68, S69, S7, S71, S72, S8, S9: footprint tmr-lib:Switch_Cutout2_MX -> tmr-lib:Switch_Cutout
- S30, S42, S45, S59, S60, S62, S70: footprint tmr-lib:Switch_Cutout2_MX_1.25u -> tmr-lib:Switch_Cutout_1.25u
- S46, S57: footprint tmr-lib:Switch_Cutout2_MX_1.75u -> tmr-lib:Switch_Cutout_1.75u
- S64, S66: footprint tmr-lib:Switch_Cutout2_MX_2u -> tmr-lib:Switch_Cutout_2u

Commit message: M  border.py M  notes/components.md A  notes/mcu M  pcb/pcb.kicad_pcb M  place.py M  plate/plate.kicad_pcb M  plate/plate.kicad_sch
Parts:
- S1: footprint tmr-lib:Switch_Cutout -> tmr-lib:Switch_Cutout_1.25u
- S62: footprint tmr-lib:Switch_Cutout_1.25u -> tmr-lib:Switch_Cutout
Changed lines of the file:
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@@
 			)
 		)
-		(property "Footprint" "tmr-lib:Switch_Cutout"
+		(property "Footprint" "tmr-lib:Switch_Cutout_1.25u"
 			(at 57.15 39.37 0)
 			(effects
@@
 			)
 		)
-		(property "Footprint" "tmr-lib:Switch_Cutout_1.25u"
+		(property "Footprint" "tmr-lib:Switch_Cutout"
 			(at 91.44 91.44 0)
 			(effects

Commit message: M  border.py M  notes/cnc.md M  notes/nRF52840.md M  notes/notes.md M  pcb/pcb.kicad_pcb M  pcb/pcb.kicad_sch M  pcb/sym-lib-table M  place.py M  plate/plate.kicad_pcb M  plate/plate.kicad_sch A  tmr-footprints/IS31FL3731-SSOP-28_5.3x10.2mm_P0.65mm.kicad_mod A  tmr-footprints/MCP3208-SOIC-16_3.9x9.9mm_P1.27mm.kicad_mod M  tmr-footprints/sw_lowpro_combo_MDT.kicad_mod D  tmr-footprints/sw_lowpro_combo_MDT_led.kicad_mod
Parts:
- S1: footprint tmr-lib:Switch_Cutout_1.25u -> tmr-lib:Switch_Cutout
Changed lines of the file:
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@@
 			)
 		)
-		(property "Footprint" "tmr-lib:Switch_Cutout_1.25u"
+		(property "Footprint" "tmr-lib:Switch_Cutout"
 			(at 57.15 39.37 0)
 			(effects
