File: pcb/pcb.kicad_pcb (KiCad board)
At the start: 2 copper layers, 299.5 x 113.5 mm, 236 parts, among them SW1 SW_DIP_x01_XKB_TS_2030, SW2 SW_DIP_x01_XKB_TS_2030, U1 RP2040, U2 Memory_Flash_W25Q64_XSON, U3 NCP114ASN330T1G, X1 12.000MHz

Commit message: M  notes/nRF52840.md M  notes/notes.md A  notes/spi M  pcb/pcb.kicad_pcb M  pcb/pcb.kicad_prl M  pcb/pcb.kicad_pro M  pcb/pcb.kicad_sch M  pickle.py D  place.py A  placefp.py D  remove_tracks.py A  rmtracks.py M  tmr-footprints/MCP3208-SOIC-16_3.9x9.9mm_P1.27mm.kicad_mod M  tmr-footprints/sw_lowpro_gateron_MDT.kicad_mod A  tmr-footprints/sw_lowpro_gateron_MDT_2.kicad_mod A  tmr-footprints/sw_lowpro_gateron_MDT_3.kicad_mod A  tmr-footprints/sw_lowpro_gateron_MDT_4.kicad_mod
Parts:
- removed the C2 at (215.0, 96.5)
- removed the C3 at (215.0, 99.0)
- removed the C4 at (215.0, 101.5)
- removed the C5 at (215.0, 104.0)
- removed the C6 at (215.0, 106.5)
- removed the C7 at (215.0, 109.1)
- removed the C8 at (215.0, 111.6)
- removed the C9 at (215.0, 114.1)
- removed Hs11, Hs12, Hs13, Hs14, Hs15, Hs16, Hs17, Hs18: ~, tmr-lib:SMTSO_M1.6
- added C21: C_Small_US, tmr-lib:C_0603_1608Metric, F.Cu at (98.0, 38.7)
- added C22: C_Small_US, tmr-lib:C_0603_1608Metric, F.Cu at (87.7, 57.7)
- added C23: C_Small_US, tmr-lib:C_0603_1608Metric, F.Cu at (49.1, 47.1)
- added C24: C_Small_US, tmr-lib:C_0603_1608Metric, F.Cu at (43.9, 50.8)
- added C25: C_Small_US, tmr-lib:C_0603_1608Metric, F.Cu at (225.7, 20.0)
- added C26: C_Small_US, tmr-lib:C_0603_1608Metric, F.Cu at (261.3, 24.3)
- added C27: C_Small_US, tmr-lib:C_0603_1608Metric, F.Cu at (255.2, 35.6)
- added C28: C_Small_US, tmr-lib:C_0603_1608Metric, F.Cu at (229.0, 76.8)
- USBCon1: footprint Connector_USB:USB_C_Receptacle_XKB_U262-16XN-4BVC11 -> Connector_USB:USB_C_Receptacle_G-Switch_GT-USB-7025; moved to F.Cu
- moved R10 248.3 mm to (268.0, 97.1)
- moved R11 242.8 mm to (261.8, 90.0)
- moved C15 229.1 mm to (-3.77, 69.5)
- moved C16 229.1 mm to (-3.77, 72.0)
- moved C17 229.1 mm to (-3.77, 74.5)
- moved C10 226.8 mm to (-2.50, 65.5)
- moved C11 213.6 mm to (14.1, 56.5), turned to -45 degrees
- moved C12 213.3 mm to (12.9, 57.7), turned to -45 degrees
- moved C1 209.6 mm to (15.9, 51.2)
- moved C7 208.6 mm to (14.3, 66.5)
- moved C6 208.4 mm to (14.3, 65.0)
- moved C5 208.2 mm to (14.3, 63.5)
- moved C2 208.1 mm to (15.7, 49.6)
- moved C4 208.1 mm to (14.3, 62.0)
- moved C3 207.9 mm to (14.3, 60.4)
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- renumbered C10 to C1, C19 to C10, C20 to C11, C21 to C12, C22 to C13, C23 to C14, C24 to C15, C25 to C16, C26 to C17, C31 to C18, C32 to C19, C11 to C2, C1 to C20, C27 to C29, C12 to C3, C28 to C30, C29 to C31, C30 to C32, C13 to C4, C14 to C5, C15 to C6, C16 to C7, C17 to C8, C18 to C9, R8 to R10, R9 to R11, R10 to R12, R11 to R13, R12 to R15, R13 to R16, R14 to R8
Connections:
- ADC1 pad 1: unconnected-(ADC1-CH0-Pad1) -> ANA_01
- ADC1 pad 11: unconnected-(ADC1-Din-Pad11) -> MOSI
- ADC1 pad 12: unconnected-(ADC1-Dout-Pad12) -> MISO
- ADC1 pad 2: unconnected-(ADC1-CH1-Pad2) -> ANA_02
- ADC1 pad 3: unconnected-(ADC1-CH2-Pad3) -> ANA_03
- ADC1 pad 4: unconnected-(ADC1-CH3-Pad4) -> ANA_04
- ADC1 pad 5: unconnected-(ADC1-CH4-Pad5) -> ANA_05
- ADC1 pad 6: unconnected-(ADC1-CH5-Pad6) -> ANA_06
- ADC1 pad 7: unconnected-(ADC1-CH6-Pad7) -> ANA_07
- ADC1 pad 8: unconnected-(ADC1-CH7-Pad8) -> ANA_08
- ADC2 pad 1: unconnected-(ADC2-CH0-Pad1) -> ANA_16
- ADC2 pad 11: unconnected-(ADC2-Din-Pad11) -> MOSI
- ADC2 pad 12: unconnected-(ADC2-Dout-Pad12) -> MISO
- ADC2 pad 2: unconnected-(ADC2-CH1-Pad2) -> ANA_17
- ADC2 pad 3: unconnected-(ADC2-CH2-Pad3) -> ANA_18
- ADC2 pad 4: unconnected-(ADC2-CH3-Pad4) -> ANA_19
- ADC2 pad 5: unconnected-(ADC2-CH4-Pad5) -> ANA_20
- ADC2 pad 6: unconnected-(ADC2-CH5-Pad6) -> ANA_21
- ADC2 pad 7: unconnected-(ADC2-CH6-Pad7) -> ANA_22
- ADC2 pad 8: unconnected-(ADC2-CH7-Pad8) -> ANA_23
- ADC3 pad 1: unconnected-(ADC3-CH0-Pad1) -> ANA_30
- ADC3 pad 11: unconnected-(ADC3-Din-Pad11) -> MOSI
- ADC3 pad 12: unconnected-(ADC3-Dout-Pad12) -> MISO
- ADC3 pad 2: unconnected-(ADC3-CH1-Pad2) -> ANA_31
- ADC3 pad 3: unconnected-(ADC3-CH2-Pad3) -> ANA_32
- ADC3 pad 4: unconnected-(ADC3-CH3-Pad4) -> ANA_33
- ADC3 pad 5: unconnected-(ADC3-CH4-Pad5) -> ANA_34
- ADC3 pad 6: unconnected-(ADC3-CH5-Pad6) -> ANA_35
- ADC3 pad 7: unconnected-(ADC3-CH6-Pad7) -> ANA_36
- ADC3 pad 8: unconnected-(ADC3-CH7-Pad8) -> ANA_37
- ADC4 pad 1: unconnected-(ADC4-CH0-Pad1) -> ANA_47
- ADC4 pad 11: unconnected-(ADC4-Din-Pad11) -> MOSI
- ADC4 pad 12: unconnected-(ADC4-Dout-Pad12) -> MISO
- ADC4 pad 2: unconnected-(ADC4-CH1-Pad2) -> ANA_62
- ADC4 pad 3: unconnected-(ADC4-CH2-Pad3) -> ANA_63
- ADC4 pad 4: unconnected-(ADC4-CH3-Pad4) -> ANA_61
- ADC4 pad 5: unconnected-(ADC4-CH4-Pad5) -> ANA_60
- ADC4 pad 6: unconnected-(ADC4-CH5-Pad6) -> ANA_59
- ADC4 pad 7: unconnected-(ADC4-CH6-Pad7) -> ANA_45
- ADC4 pad 8: unconnected-(ADC4-CH7-Pad8) -> ANA_46
- ADC5 pad 1: unconnected-(ADC5-CH0-Pad1) -> ANA_52
- ADC5 pad 11: unconnected-(ADC5-Din-Pad11) -> MOSI
- ADC5 pad 12: unconnected-(ADC5-Dout-Pad12) -> MISO
- ADC5 pad 2: unconnected-(ADC5-CH1-Pad2) -> ANA_66
- ADC5 pad 3: unconnected-(ADC5-CH2-Pad3) -> ANA_65
- ADC5 pad 4: unconnected-(ADC5-CH3-Pad4) -> ANA_64
- ADC5 pad 5: unconnected-(ADC5-CH4-Pad5) -> ANA_48
- ADC5 pad 6: unconnected-(ADC5-CH5-Pad6) -> ANA_49
- ADC5 pad 7: unconnected-(ADC5-CH6-Pad7) -> ANA_50
- ADC5 pad 8: unconnected-(ADC5-CH7-Pad8) -> ANA_51
- ADC6 pad 1: unconnected-(ADC6-CH0-Pad1) -> ANA_09
- ADC6 pad 11: unconnected-(ADC6-Din-Pad11) -> MOSI
- ADC6 pad 12: unconnected-(ADC6-Dout-Pad12) -> MISO
- ADC6 pad 2: unconnected-(ADC6-CH1-Pad2) -> ANA_10
- ADC6 pad 3: unconnected-(ADC6-CH2-Pad3) -> ANA_11
- ADC6 pad 4: unconnected-(ADC6-CH3-Pad4) -> ANA_12
- ADC6 pad 5: unconnected-(ADC6-CH4-Pad5) -> ANA_13
- ADC6 pad 6: unconnected-(ADC6-CH5-Pad6) -> ANA_14
- ADC6 pad 7: unconnected-(ADC6-CH6-Pad7) -> ANA_15
- ADC6 pad 8: unconnected-(ADC6-CH7-Pad8) -> ANA_29
- ADC7 pad 1: unconnected-(ADC7-CH0-Pad1) -> ANA_44
- ADC7 pad 11: unconnected-(ADC7-Din-Pad11) -> MOSI
- ADC7 pad 12: unconnected-(ADC7-Dout-Pad12) -> MISO
- ADC7 pad 2: unconnected-(ADC7-CH1-Pad2) -> ANA_58
- ADC7 pad 3: unconnected-(ADC7-CH2-Pad3) -> ANA_72
- ADC7 pad 4: unconnected-(ADC7-CH3-Pad4) -> ANA_24
- ADC7 pad 5: unconnected-(ADC7-CH4-Pad5) -> ANA_25
- ADC7 pad 6: unconnected-(ADC7-CH5-Pad6) -> ANA_26
- ADC7 pad 7: unconnected-(ADC7-CH6-Pad7) -> ANA_27
- ADC7 pad 8: unconnected-(ADC7-CH7-Pad8) -> ANA_28
- ADC8 pad 1: unconnected-(ADC8-CH0-Pad1) -> ANA_43
- ADC8 pad 11: unconnected-(ADC8-Din-Pad11) -> MOSI
- ADC8 pad 12: unconnected-(ADC8-Dout-Pad12) -> MISO
- ADC8 pad 2: unconnected-(ADC8-CH1-Pad2) -> ANA_71
- ADC8 pad 3: unconnected-(ADC8-CH2-Pad3) -> ANA_57
- ADC8 pad 4: unconnected-(ADC8-CH3-Pad4) -> ANA_38
- ADC8 pad 5: unconnected-(ADC8-CH4-Pad5) -> ANA_39
- ADC8 pad 6: unconnected-(ADC8-CH5-Pad6) -> ANA_40
- ADC8 pad 7: unconnected-(ADC8-CH6-Pad7) -> ANA_41
- ADC8 pad 8: unconnected-(ADC8-CH7-Pad8) -> ANA_42
- ADC9 pad 1: unconnected-(ADC9-CH0-Pad1) -> ANA_69
- ADC9 pad 11: unconnected-(ADC9-Din-Pad11) -> MOSI
- ADC9 pad 12: unconnected-(ADC9-Dout-Pad12) -> MISO
- ADC9 pad 2: unconnected-(ADC9-CH1-Pad2) -> ANA_68
- ADC9 pad 3: unconnected-(ADC9-CH2-Pad3) -> ANA_67
- ADC9 pad 4: unconnected-(ADC9-CH3-Pad4) -> ANA_53
- ADC9 pad 5: unconnected-(ADC9-CH4-Pad5) -> ANA_54
- ADC9 pad 6: unconnected-(ADC9-CH5-Pad6) -> ANA_55
- ADC9 pad 7: unconnected-(ADC9-CH6-Pad7) -> ANA_56
- ADC9 pad 8: unconnected-(ADC9-CH7-Pad8) -> ANA_70
- S1 pad 2: unconnected-(S1-V_{OUT}-Pad2) -> ANA_01
- S10 pad 2: unconnected-(S10-V_{OUT}-Pad2) -> ANA_10
- S11 pad 2: unconnected-(S11-V_{OUT}-Pad2) -> ANA_11
- S12 pad 2: unconnected-(S12-V_{OUT}-Pad2) -> ANA_12
- S13 pad 2: unconnected-(S13-V_{OUT}-Pad2) -> ANA_13
- S14 pad 2: unconnected-(S14-V_{OUT}-Pad2) -> ANA_14
- S15 pad 2: unconnected-(S15-V_{OUT}-Pad2) -> ANA_15
- S16 pad 2: unconnected-(S16-V_{OUT}-Pad2) -> ANA_16
- S17 pad 2: unconnected-(S17-V_{OUT}-Pad2) -> ANA_17
- S18 pad 2: unconnected-(S18-V_{OUT}-Pad2) -> ANA_18
- S19 pad 2: unconnected-(S19-V_{OUT}-Pad2) -> ANA_19
- S2 pad 2: unconnected-(S2-V_{OUT}-Pad2) -> ANA_02
- S20 pad 2: unconnected-(S20-V_{OUT}-Pad2) -> ANA_20
- S21 pad 2: unconnected-(S21-V_{OUT}-Pad2) -> ANA_21
- S22 pad 2: unconnected-(S22-V_{OUT}-Pad2) -> ANA_22
- S23 pad 2: unconnected-(S23-V_{OUT}-Pad2) -> ANA_23
- S24 pad 2: unconnected-(S24-V_{OUT}-Pad2) -> ANA_24
- S25 pad 2: unconnected-(S25-V_{OUT}-Pad2) -> ANA_25
- S26 pad 2: unconnected-(S26-V_{OUT}-Pad2) -> ANA_26
- S27 pad 2: unconnected-(S27-V_{OUT}-Pad2) -> ANA_27
- S28 pad 2: unconnected-(S28-V_{OUT}-Pad2) -> ANA_28
- S29 pad 2: unconnected-(S29-V_{OUT}-Pad2) -> ANA_29
- S3 pad 2: unconnected-(S3-V_{OUT}-Pad2) -> ANA_03
- S30 pad 2: unconnected-(S30-V_{OUT}-Pad2) -> ANA_30
- S31 pad 2: unconnected-(S31-V_{OUT}-Pad2) -> ANA_31
- S32 pad 2: unconnected-(S32-V_{OUT}-Pad2) -> ANA_32
- S33 pad 2: unconnected-(S33-V_{OUT}-Pad2) -> ANA_33
- S34 pad 2: unconnected-(S34-V_{OUT}-Pad2) -> ANA_34
- S35 pad 2: unconnected-(S35-V_{OUT}-Pad2) -> ANA_35
- S36 pad 2: unconnected-(S36-V_{OUT}-Pad2) -> ANA_36
- S37 pad 2: unconnected-(S37-V_{OUT}-Pad2) -> ANA_37
- S38 pad 2: unconnected-(S38-V_{OUT}-Pad2) -> ANA_38
- S39 pad 2: unconnected-(S39-V_{OUT}-Pad2) -> ANA_39
- S4 pad 2: unconnected-(S4-V_{OUT}-Pad2) -> ANA_04
- S40 pad 2: unconnected-(S40-V_{OUT}-Pad2) -> ANA_40
- S41 pad 2: unconnected-(S41-V_{OUT}-Pad2) -> ANA_41
- S42 pad 2: unconnected-(S42-V_{OUT}-Pad2) -> ANA_42
- S43 pad 2: unconnected-(S43-V_{OUT}-Pad2) -> ANA_43
- S44 pad 2: unconnected-(S44-V_{OUT}-Pad2) -> ANA_44
- S45 pad 2: unconnected-(S45-V_{OUT}-Pad2) -> ANA_45
- S46 pad 2: unconnected-(S46-V_{OUT}-Pad2) -> ANA_46
- S47 pad 2: unconnected-(S47-V_{OUT}-Pad2) -> ANA_47
- S48 pad 2: unconnected-(S48-V_{OUT}-Pad2) -> ANA_48
- S49 pad 2: unconnected-(S49-V_{OUT}-Pad2) -> ANA_49
- S5 pad 2: unconnected-(S5-V_{OUT}-Pad2) -> ANA_05
- S50 pad 2: unconnected-(S50-V_{OUT}-Pad2) -> ANA_50
- S51 pad 2: unconnected-(S51-V_{OUT}-Pad2) -> ANA_51
- S52 pad 2: unconnected-(S52-V_{OUT}-Pad2) -> ANA_52
- S53 pad 2: unconnected-(S53-V_{OUT}-Pad2) -> ANA_53
- S54 pad 2: unconnected-(S54-V_{OUT}-Pad2) -> ANA_54
- S55 pad 2: unconnected-(S55-V_{OUT}-Pad2) -> ANA_55
- S56 pad 2: unconnected-(S56-V_{OUT}-Pad2) -> ANA_56
- S57 pad 2: unconnected-(S57-V_{OUT}-Pad2) -> ANA_57
- S58 pad 2: unconnected-(S58-V_{OUT}-Pad2) -> ANA_58
- S59 pad 2: unconnected-(S59-V_{OUT}-Pad2) -> ANA_59
- S6 pad 2: unconnected-(S6-V_{OUT}-Pad2) -> ANA_06
- S60 pad 2: unconnected-(S60-V_{OUT}-Pad2) -> ANA_60
- S61 pad 2: unconnected-(S61-V_{OUT}-Pad2) -> ANA_61
- S62 pad 2: unconnected-(S62-V_{OUT}-Pad2) -> ANA_62
- S63 pad 2: unconnected-(S63-V_{OUT}-Pad2) -> ANA_63
- S64 pad 2: unconnected-(S64-V_{OUT}-Pad2) -> ANA_64
- S65 pad 2: unconnected-(S65-V_{OUT}-Pad2) -> ANA_65
- S66 pad 2: unconnected-(S66-V_{OUT}-Pad2) -> ANA_66
- S67 pad 2: unconnected-(S67-V_{OUT}-Pad2) -> ANA_67
- S68 pad 2: unconnected-(S68-V_{OUT}-Pad2) -> ANA_68
- S69 pad 2: unconnected-(S69-V_{OUT}-Pad2) -> ANA_69
- S7 pad 2: unconnected-(S7-V_{OUT}-Pad2) -> ANA_07
- S70 pad 2: unconnected-(S70-V_{OUT}-Pad2) -> ANA_70
- S71 pad 2: unconnected-(S71-V_{OUT}-Pad2) -> ANA_71
- S72 pad 2: unconnected-(S72-V_{OUT}-Pad2) -> ANA_72
- S8 pad 2: unconnected-(S8-V_{OUT}-Pad2) -> ANA_08
- S9 pad 2: unconnected-(S9-V_{OUT}-Pad2) -> ANA_09
- U1 pad 2: /GPIO0 -> MISO
