File: pcb/pcb.kicad_pcb (KiCad board)
At the start: 2 copper layers, 299.5 x 113.5 mm, 481 parts, among them M1 nRF54L15 module, Q1 DMC2400UV, Q2 Si2302CDS, SW1 SW_DIP_x01, U1 nPM1100-QDXX, U2 ADG706BRU, U3 ADG706BRU, U4 ADG706BRU, U5 ADG706BRU, U6 ADG706BRU, U7 TPS22902

Commit message: M  pcb/pcb.kicad_pcb M  pcb/pcb.kicad_sch M  pcb/switch.kicad_sch M  placefp.py A  tmr-footprints/Texas_DYY0016A_TSOT-23-16_2x4.2mm_P0.5mm.kicad_mod M  tmr-symbols.kicad_sym
Parts:
- removed the C6 at (-26.6, 48.3)
- removed Q1: DMC2400UV, Package_TO_SOT_SMD:SOT-563
- removed Q2: Si2302CDS, Package_TO_SOT_SMD:SOT-23-3
- removed R10, R7: 100k, Resistor_SMD:R_0603_1608Metric
- removed R5: 1M0, Resistor_SMD:R_0603_1608Metric
- removed R6: 220k, Resistor_SMD:R_0603_1608Metric
- removed R8: 220R, Resistor_SMD:R_0603_1608Metric
- removed R9: 10k, Resistor_SMD:R_0603_1608Metric
- removed Rd1, Rd10, Rd11, Rd12, Rd13, Rd14, Rd15, Rd16, Rd17, Rd18, Rd19, Rd2, Rd20, Rd21, Rd22, Rd23, Rd24, Rd25, Rd26, Rd27, Rd28, Rd29, Rd3, Rd30, Rd31, Rd32, Rd33, Rd34, Rd35, Rd36, Rd37, Rd38, Rd39, Rd4, Rd40, Rd41, Rd42, Rd43, Rd44, Rd45, Rd46, Rd47, Rd48, Rd49, Rd5, Rd50, Rd51, Rd52, Rd53, Rd54, Rd55, Rd56, Rd57, Rd58, Rd59, Rd6, Rd60, Rd61, Rd62, Rd63, Rd64, Rd65, Rd66, Rd67, Rd68, Rd69, Rd7, Rd70, Rd71, Rd72, Rd8, Rd9: 220R, tmr-lib:R_0402_1005Metric
- removed SW1: SW_DIP_x01, TestPoint:TestPoint_Bridge_Pitch3.81mm_Drill1.3mm
- removed U1: nPM1100-QDXX, Package_DFN_QFN:QFN-24-1EP_4x4mm_P0.5mm_EP2.6x2.6mm_ThermalVias
- removed U2, U3, U4, U5, U6: ADG706BRU, Package_SO:TSSOP-28_4.4x9.7mm_P0.65mm
- removed U7: TPS22902, tmr-lib:Texas_DSBGA-4_0.8x0.8mm_Layout2x2_P0.4mm
- added C1: 10uF, Capacitor_SMD:C_0603_1608Metric, B.Cu at (35.0, 23.8)
- added C12: 2.2uF, Capacitor_SMD:C_0603_1608Metric, B.Cu at (34.7, 13.9)
- added C13: .1uF, Capacitor_SMD:C_0402_1005Metric, B.Cu at (117.7, 6.13)
- added C14: 1nF, Capacitor_SMD:C_0603_1608Metric, B.Cu at (140.2, 27.9)
- added C15: 1uF, Capacitor_SMD:C_0603_1608Metric, B.Cu at (136.3, 27.9)
- added C16: 1uF, Capacitor_SMD:C_0603_1608Metric, B.Cu at (141.9, 30.2)
- added C17: .1uF, Capacitor_SMD:C_0402_1005Metric, B.Cu at (127.2, 6.66)
- added C18: 1uF, Capacitor_SMD:C_0603_1608Metric, B.Cu at (136.8, 35.5)
- added L2: 2.2uH, tmr-lib:L_Samsung_CIGT201610EH2R2MNE, B.Cu at (36.0, 25.6)
- added LEDDR1: LP5864, Package_DFN_QFN:VQFN-32-1EP_4x4mm_P0.4mm_EP2.8x2.8mm_ThermalVias, B.Cu at (137.8, 31.3)
- added MUXA1: TMUX1574DYY, tmr-lib:Texas_DYY0016A_TSOT-23-16_2x4.2mm_P0.5mm, B.Cu at (156.5, 8.93)
- added MUXA2: TMUX1574DYY, tmr-lib:Texas_DYY0016A_TSOT-23-16_2x4.2mm_P0.5mm, B.Cu at (166.5, 8.93)
- added MUXB1: TMUX1108PW, Package_SO:TSSOP-16_4.4x5mm_P0.65mm, B.Cu at (122.3, 6.58)
- added PMIC1: nPM1300-QEXX, Package_DFN_QFN:QFN-32-1EP_5x5mm_P0.5mm_EP3.6x3.6mm_ThermalVias, B.Cu at (36.0, 19.2)
- added USB1: USB_C_Receptacle_PowerOnly_6P, Connector_USB:USB_C_Receptacle_GCT_USB4125-xx-x-0190_6P_TopMnt_Horizontal, F.Cu at (47.5, -6.20)
- C10, C9: value 0.1uF -> 10uF; footprint Capacitor_SMD:C_0402_1005Metric -> Capacitor_SMD:C_0603_1608Metric; moved to B.Cu
- C11: value 10uF -> 2.2uF; moved to B.Cu
- C2: moved to B.Cu
- C3: value 1uF -> 10uF; moved to B.Cu
- C4: value 10uF -> 0.1uF; footprint Capacitor_SMD:C_0603_1608Metric -> Capacitor_SMD:C_0402_1005Metric; moved to B.Cu
- C5: value 10uF -> 1uF; moved to B.Cu
- C6: renamed from C1; value 2.2uF -> 1uF
- C7, C8: value 0.1uF -> .1uF; moved to B.Cu
- D1, D10, D11, D12, D13, D14, D15, D16, D17, D18, D19, D2, D20, D21, D22, D23, D24, D25, D26, D27, D28, D29, D3, D30, D31, D32, D33, D34, D35, D36, D37, D38, D39, D4, D40, D41, D42, D43, D44, D45, D46, D47, D48, D49, D5, D50, D51, D52, D53, D54, D55, D56, D57, D58, D59, D6, D60, D61, D62, D63, D64, D65, D66, D67, D68, D69, D7, D70, D71, D72, D8, D9: value LED -> Green LED
- L1: value 2.2uF -> 2.2uH; footprint tmr-lib:Murata_DFE201210U -> tmr-lib:L_Samsung_CIGT201610EH2R2MNE; moved to B.Cu
- M1: value nRF54L15 module -> Ezurio BL54L15 (nrf54L15) module
- R1: value 1M0 -> 10k; footprint Resistor_SMD:R_0603_1608Metric -> Resistor_SMD:R_0402_1005Metric; moved to B.Cu
- R2: value 5.1k -> 10k; footprint Resistor_SMD:R_0603_1608Metric -> Resistor_SMD:R_0402_1005Metric; moved to B.Cu
- R3: value 5.1k -> 47k; footprint Resistor_SMD:R_0603_1608Metric -> Resistor_SMD:R_0402_1005Metric; moved to B.Cu
- R4: value 1M5 -> 47k; footprint Resistor_SMD:R_0603_1608Metric -> Resistor_SMD:R_0402_1005Metric; moved to B.Cu
- moved C8 253.7 mm to (163.6, 6.82), turned to 90 degrees
- moved C7 243.6 mm to (153.6, 6.32), turned to -90 degrees
- moved M1 144.9 mm to (155.8, 4.40), turned to 90 degrees
- moved C10 134.1 mm to (40.5, 21.1), turned to 90 degrees
- moved C9 132.3 mm to (40.9, 24.6), turned to 90 degrees
- moved C6 105.5 mm to (47.6, -0.27)
- moved C11 96.5 mm to (40.5, 18.1), turned to -90 degrees
- moved C5 95.1 mm to (37.8, 13.9), turned to 90 degrees
- moved C3 91.0 mm to (36.2, 13.9), turned to 90 degrees
- moved C2 86.9 mm to (38.0, 23.8)
- moved R3 85.0 mm to (33.4, 14.5), turned to -90 degrees
- moved C4 84.3 mm to (31.1, 21.0), turned to 90 degrees
- moved BAT1 84.2 mm to (-40.9, 4.41), turned to 0 degrees
- moved R4 83.1 mm to (31.0, 16.9)
- moved L1 79.8 mm to (38.7, 25.6), turned to 180 degrees
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Connections:
- BAT1 pad 1: /VBAT -> Net-(BAT1-VBAT)
- C10 pad 1: +2V1_TMR -> VCCS
- C11 pad 1: GND -> /VCC_tmr
- C11 pad 2: +2V1 -> GND
- C3 pad 1: /VBAT -> /VSYS
- C4 pad 1: Net-(U1-DEC) -> GND
- C4 pad 2: GND -> /VDDIO
- C5 pad 1: +2V1 -> Net-(PMIC1-VBUSOUT)
- C7 pad 1: +2V1_TMR -> GND
- C7 pad 2: GND -> VCCS
- C8 pad 1: +2V1_TMR -> GND
- C8 pad 2: GND -> VCCS
- C9 pad 1: +2V1_TMR -> /VDDIO
- Cvcc1 pad 1: +2V1_TMR -> VCCS
- Cvcc10 pad 1: +2V1_TMR -> VCCS
- Cvcc11 pad 1: +2V1_TMR -> VCCS
- Cvcc12 pad 1: +2V1_TMR -> VCCS
- Cvcc13 pad 1: +2V1_TMR -> VCCS
- Cvcc14 pad 1: +2V1_TMR -> VCCS
- Cvcc15 pad 1: +2V1_TMR -> VCCS
- Cvcc16 pad 1: +2V1_TMR -> VCCS
- Cvcc17 pad 1: +2V1_TMR -> VCCS
- Cvcc18 pad 1: +2V1_TMR -> VCCS
- Cvcc19 pad 1: +2V1_TMR -> VCCS
- Cvcc2 pad 1: +2V1_TMR -> VCCS
- Cvcc20 pad 1: +2V1_TMR -> VCCS
- Cvcc21 pad 1: +2V1_TMR -> VCCS
- Cvcc22 pad 1: +2V1_TMR -> VCCS
- Cvcc23 pad 1: +2V1_TMR -> VCCS
- Cvcc24 pad 1: +2V1_TMR -> VCCS
- Cvcc25 pad 1: +2V1_TMR -> VCCS
- Cvcc26 pad 1: +2V1_TMR -> VCCS
- Cvcc27 pad 1: +2V1_TMR -> VCCS
- Cvcc28 pad 1: +2V1_TMR -> VCCS
- Cvcc29 pad 1: +2V1_TMR -> VCCS
- Cvcc3 pad 1: +2V1_TMR -> VCCS
- Cvcc30 pad 1: +2V1_TMR -> VCCS
- Cvcc31 pad 1: +2V1_TMR -> VCCS
- Cvcc32 pad 1: +2V1_TMR -> VCCS
- Cvcc33 pad 1: +2V1_TMR -> VCCS
- Cvcc34 pad 1: +2V1_TMR -> VCCS
- Cvcc35 pad 1: +2V1_TMR -> VCCS
- Cvcc36 pad 1: +2V1_TMR -> VCCS
- Cvcc37 pad 1: +2V1_TMR -> VCCS
- Cvcc38 pad 1: +2V1_TMR -> VCCS
- Cvcc39 pad 1: +2V1_TMR -> VCCS
- Cvcc4 pad 1: +2V1_TMR -> VCCS
- Cvcc40 pad 1: +2V1_TMR -> VCCS
- Cvcc41 pad 1: +2V1_TMR -> VCCS
- Cvcc42 pad 1: +2V1_TMR -> VCCS
- Cvcc43 pad 1: +2V1_TMR -> VCCS
- Cvcc44 pad 1: +2V1_TMR -> VCCS
- Cvcc45 pad 1: +2V1_TMR -> VCCS
- Cvcc46 pad 1: +2V1_TMR -> VCCS
- Cvcc47 pad 1: +2V1_TMR -> VCCS
- Cvcc48 pad 1: +2V1_TMR -> VCCS
- Cvcc49 pad 1: +2V1_TMR -> VCCS
- Cvcc5 pad 1: +2V1_TMR -> VCCS
- Cvcc50 pad 1: +2V1_TMR -> VCCS
- Cvcc51 pad 1: +2V1_TMR -> VCCS
- Cvcc52 pad 1: +2V1_TMR -> VCCS
- Cvcc53 pad 1: +2V1_TMR -> VCCS
- Cvcc54 pad 1: +2V1_TMR -> VCCS
- Cvcc55 pad 1: +2V1_TMR -> VCCS
- Cvcc56 pad 1: +2V1_TMR -> VCCS
- Cvcc57 pad 1: +2V1_TMR -> VCCS
- Cvcc58 pad 1: +2V1_TMR -> VCCS
- Cvcc59 pad 1: +2V1_TMR -> VCCS
- Cvcc6 pad 1: +2V1_TMR -> VCCS
- Cvcc60 pad 1: +2V1_TMR -> VCCS
- Cvcc61 pad 1: +2V1_TMR -> VCCS
- Cvcc62 pad 1: +2V1_TMR -> VCCS
- Cvcc63 pad 1: +2V1_TMR -> VCCS
- Cvcc64 pad 1: +2V1_TMR -> VCCS
- Cvcc65 pad 1: +2V1_TMR -> VCCS
- Cvcc66 pad 1: +2V1_TMR -> VCCS
- Cvcc67 pad 1: +2V1_TMR -> VCCS
- Cvcc68 pad 1: +2V1_TMR -> VCCS
- Cvcc69 pad 1: +2V1_TMR -> VCCS
- Cvcc7 pad 1: +2V1_TMR -> VCCS
- Cvcc70 pad 1: +2V1_TMR -> VCCS
- Cvcc71 pad 1: +2V1_TMR -> VCCS
- Cvcc72 pad 1: +2V1_TMR -> VCCS
- Cvcc8 pad 1: +2V1_TMR -> VCCS
- Cvcc9 pad 1: +2V1_TMR -> VCCS
- D1 pad 1: LED_CATH -> unconnected-(D1-K-Pad1)
- D1 pad 2: Net-(D1-A) -> unconnected-(D1-A-Pad2)
- D10 pad 1: LED_CATH -> unconnected-(D10-K-Pad1)
- D10 pad 2: Net-(D10-A) -> unconnected-(D10-A-Pad2)
- D11 pad 1: LED_CATH -> unconnected-(D11-K-Pad1)
- D11 pad 2: Net-(D11-A) -> unconnected-(D11-A-Pad2)
- D12 pad 1: LED_CATH -> unconnected-(D12-K-Pad1)
- D12 pad 2: Net-(D12-A) -> unconnected-(D12-A-Pad2)
- D13 pad 1: LED_CATH -> unconnected-(D13-K-Pad1)
- D13 pad 2: Net-(D13-A) -> unconnected-(D13-A-Pad2)
- D14 pad 1: LED_CATH -> unconnected-(D14-K-Pad1)
- D14 pad 2: Net-(D14-A) -> unconnected-(D14-A-Pad2)
- D15 pad 1: LED_CATH -> unconnected-(D15-K-Pad1)
- D15 pad 2: Net-(D15-A) -> unconnected-(D15-A-Pad2)
- D16 pad 1: LED_CATH -> unconnected-(D16-K-Pad1)
- D16 pad 2: Net-(D16-A) -> unconnected-(D16-A-Pad2)
- D17 pad 1: LED_CATH -> unconnected-(D17-K-Pad1)
- D17 pad 2: Net-(D17-A) -> unconnected-(D17-A-Pad2)
- D18 pad 1: LED_CATH -> unconnected-(D18-K-Pad1)
- D18 pad 2: Net-(D18-A) -> unconnected-(D18-A-Pad2)
- D19 pad 1: LED_CATH -> unconnected-(D19-K-Pad1)
- D19 pad 2: Net-(D19-A) -> unconnected-(D19-A-Pad2)
- D2 pad 1: LED_CATH -> unconnected-(D2-K-Pad1)
- D2 pad 2: Net-(D2-A) -> unconnected-(D2-A-Pad2)
- D20 pad 1: LED_CATH -> unconnected-(D20-K-Pad1)
- D20 pad 2: Net-(D20-A) -> unconnected-(D20-A-Pad2)
- D21 pad 1: LED_CATH -> unconnected-(D21-K-Pad1)
- D21 pad 2: Net-(D21-A) -> unconnected-(D21-A-Pad2)
- D22 pad 1: LED_CATH -> unconnected-(D22-K-Pad1)
- D22 pad 2: Net-(D22-A) -> unconnected-(D22-A-Pad2)
- D23 pad 1: LED_CATH -> unconnected-(D23-K-Pad1)
- D23 pad 2: Net-(D23-A) -> unconnected-(D23-A-Pad2)
- D24 pad 1: LED_CATH -> unconnected-(D24-K-Pad1)
- D24 pad 2: Net-(D24-A) -> unconnected-(D24-A-Pad2)
- D25 pad 1: LED_CATH -> unconnected-(D25-K-Pad1)
- D25 pad 2: Net-(D25-A) -> unconnected-(D25-A-Pad2)
- D26 pad 1: LED_CATH -> unconnected-(D26-K-Pad1)
- D26 pad 2: Net-(D26-A) -> unconnected-(D26-A-Pad2)
- D27 pad 1: LED_CATH -> unconnected-(D27-K-Pad1)
- D27 pad 2: Net-(D27-A) -> unconnected-(D27-A-Pad2)
- D28 pad 1: LED_CATH -> unconnected-(D28-K-Pad1)
- D28 pad 2: Net-(D28-A) -> unconnected-(D28-A-Pad2)
- D29 pad 1: LED_CATH -> unconnected-(D29-K-Pad1)
- D29 pad 2: Net-(D29-A) -> unconnected-(D29-A-Pad2)
- D3 pad 1: LED_CATH -> unconnected-(D3-K-Pad1)
- D3 pad 2: Net-(D3-A) -> unconnected-(D3-A-Pad2)
- D30 pad 1: LED_CATH -> unconnected-(D30-K-Pad1)
- D30 pad 2: Net-(D30-A) -> unconnected-(D30-A-Pad2)
- D31 pad 1: LED_CATH -> unconnected-(D31-K-Pad1)
- D31 pad 2: Net-(D31-A) -> unconnected-(D31-A-Pad2)
- D32 pad 1: LED_CATH -> unconnected-(D32-K-Pad1)
- D32 pad 2: Net-(D32-A) -> unconnected-(D32-A-Pad2)
- D33 pad 1: LED_CATH -> unconnected-(D33-K-Pad1)
- D33 pad 2: Net-(D33-A) -> unconnected-(D33-A-Pad2)
- D34 pad 1: LED_CATH -> unconnected-(D34-K-Pad1)
- D34 pad 2: Net-(D34-A) -> unconnected-(D34-A-Pad2)
- D35 pad 1: LED_CATH -> unconnected-(D35-K-Pad1)
- D35 pad 2: Net-(D35-A) -> unconnected-(D35-A-Pad2)
- D36 pad 1: LED_CATH -> unconnected-(D36-K-Pad1)
- D36 pad 2: Net-(D36-A) -> unconnected-(D36-A-Pad2)
- D37 pad 1: LED_CATH -> unconnected-(D37-K-Pad1)
- D37 pad 2: Net-(D37-A) -> unconnected-(D37-A-Pad2)
- D38 pad 1: LED_CATH -> unconnected-(D38-K-Pad1)
- D38 pad 2: Net-(D38-A) -> unconnected-(D38-A-Pad2)
- D39 pad 1: LED_CATH -> unconnected-(D39-K-Pad1)
- D39 pad 2: Net-(D39-A) -> unconnected-(D39-A-Pad2)
- D4 pad 1: LED_CATH -> unconnected-(D4-K-Pad1)
- D4 pad 2: Net-(D4-A) -> unconnected-(D4-A-Pad2)
- D40 pad 1: LED_CATH -> unconnected-(D40-K-Pad1)
- D40 pad 2: Net-(D40-A) -> unconnected-(D40-A-Pad2)
- D41 pad 1: LED_CATH -> unconnected-(D41-K-Pad1)
- D41 pad 2: Net-(D41-A) -> unconnected-(D41-A-Pad2)
- D42 pad 1: LED_CATH -> unconnected-(D42-K-Pad1)
- D42 pad 2: Net-(D42-A) -> unconnected-(D42-A-Pad2)
- D43 pad 1: LED_CATH -> unconnected-(D43-K-Pad1)
- D43 pad 2: Net-(D43-A) -> unconnected-(D43-A-Pad2)
- D44 pad 1: LED_CATH -> unconnected-(D44-K-Pad1)
- D44 pad 2: Net-(D44-A) -> unconnected-(D44-A-Pad2)
- D45 pad 1: LED_CATH -> unconnected-(D45-K-Pad1)
- D45 pad 2: Net-(D45-A) -> unconnected-(D45-A-Pad2)
- D46 pad 1: LED_CATH -> unconnected-(D46-K-Pad1)
- D46 pad 2: Net-(D46-A) -> unconnected-(D46-A-Pad2)
- D47 pad 1: LED_CATH -> unconnected-(D47-K-Pad1)
- D47 pad 2: Net-(D47-A) -> unconnected-(D47-A-Pad2)
- D48 pad 1: LED_CATH -> unconnected-(D48-K-Pad1)
- D48 pad 2: Net-(D48-A) -> unconnected-(D48-A-Pad2)
- D49 pad 1: LED_CATH -> unconnected-(D49-K-Pad1)
- D49 pad 2: Net-(D49-A) -> unconnected-(D49-A-Pad2)
- D5 pad 1: LED_CATH -> unconnected-(D5-K-Pad1)
- D5 pad 2: Net-(D5-A) -> unconnected-(D5-A-Pad2)
- D50 pad 1: LED_CATH -> unconnected-(D50-K-Pad1)
- D50 pad 2: Net-(D50-A) -> unconnected-(D50-A-Pad2)
- D51 pad 1: LED_CATH -> unconnected-(D51-K-Pad1)
- D51 pad 2: Net-(D51-A) -> unconnected-(D51-A-Pad2)
- D52 pad 1: LED_CATH -> unconnected-(D52-K-Pad1)
- D52 pad 2: Net-(D52-A) -> unconnected-(D52-A-Pad2)
- D53 pad 1: LED_CATH -> unconnected-(D53-K-Pad1)
- D53 pad 2: Net-(D53-A) -> unconnected-(D53-A-Pad2)
- D54 pad 1: LED_CATH -> unconnected-(D54-K-Pad1)
- D54 pad 2: Net-(D54-A) -> unconnected-(D54-A-Pad2)
- D55 pad 1: LED_CATH -> unconnected-(D55-K-Pad1)
- D55 pad 2: Net-(D55-A) -> unconnected-(D55-A-Pad2)
- D56 pad 1: LED_CATH -> unconnected-(D56-K-Pad1)
- D56 pad 2: Net-(D56-A) -> unconnected-(D56-A-Pad2)
- D57 pad 1: LED_CATH -> unconnected-(D57-K-Pad1)
- D57 pad 2: Net-(D57-A) -> unconnected-(D57-A-Pad2)
- D58 pad 1: LED_CATH -> unconnected-(D58-K-Pad1)
- D58 pad 2: Net-(D58-A) -> unconnected-(D58-A-Pad2)
- D59 pad 1: LED_CATH -> unconnected-(D59-K-Pad1)
- D59 pad 2: Net-(D59-A) -> unconnected-(D59-A-Pad2)
- D6 pad 1: LED_CATH -> unconnected-(D6-K-Pad1)
- D6 pad 2: Net-(D6-A) -> unconnected-(D6-A-Pad2)
- D60 pad 1: LED_CATH -> unconnected-(D60-K-Pad1)
- D60 pad 2: Net-(D60-A) -> unconnected-(D60-A-Pad2)
- D61 pad 1: LED_CATH -> unconnected-(D61-K-Pad1)
- D61 pad 2: Net-(D61-A) -> unconnected-(D61-A-Pad2)
- D62 pad 1: LED_CATH -> unconnected-(D62-K-Pad1)
- D62 pad 2: Net-(D62-A) -> unconnected-(D62-A-Pad2)
- D63 pad 1: LED_CATH -> unconnected-(D63-K-Pad1)
- D63 pad 2: Net-(D63-A) -> unconnected-(D63-A-Pad2)
- D64 pad 1: LED_CATH -> unconnected-(D64-K-Pad1)
- D64 pad 2: Net-(D64-A) -> unconnected-(D64-A-Pad2)
- D65 pad 1: LED_CATH -> unconnected-(D65-K-Pad1)
- D65 pad 2: Net-(D65-A) -> unconnected-(D65-A-Pad2)
- D66 pad 1: LED_CATH -> unconnected-(D66-K-Pad1)
- D66 pad 2: Net-(D66-A) -> unconnected-(D66-A-Pad2)
- D67 pad 1: LED_CATH -> unconnected-(D67-K-Pad1)
- D67 pad 2: Net-(D67-A) -> unconnected-(D67-A-Pad2)
- D68 pad 1: LED_CATH -> unconnected-(D68-K-Pad1)
- D68 pad 2: Net-(D68-A) -> unconnected-(D68-A-Pad2)
- D69 pad 1: LED_CATH -> unconnected-(D69-K-Pad1)
- D69 pad 2: Net-(D69-A) -> unconnected-(D69-A-Pad2)
- D7 pad 1: LED_CATH -> unconnected-(D7-K-Pad1)
- D7 pad 2: Net-(D7-A) -> unconnected-(D7-A-Pad2)
- D70 pad 1: LED_CATH -> unconnected-(D70-K-Pad1)
- D70 pad 2: Net-(D70-A) -> unconnected-(D70-A-Pad2)
- D71 pad 1: LED_CATH -> unconnected-(D71-K-Pad1)
- D71 pad 2: Net-(D71-A) -> unconnected-(D71-A-Pad2)
- D72 pad 1: LED_CATH -> unconnected-(D72-K-Pad1)
- D72 pad 2: Net-(D72-A) -> unconnected-(D72-A-Pad2)
- D8 pad 1: LED_CATH -> unconnected-(D8-K-Pad1)
- D8 pad 2: Net-(D8-A) -> unconnected-(D8-A-Pad2)
- D9 pad 1: LED_CATH -> unconnected-(D9-K-Pad1)
- D9 pad 2: Net-(D9-A) -> unconnected-(D9-A-Pad2)
- L1 pad 1: +2V1 -> /VDDIO
- M1 pad 20: unconnected-(M1-P1.07/AIN3-Pad20) -> /AIN3
- M1 pad 21: unconnected-(M1-P1.06/AIN2-Pad21) -> /AIN2
- M1 pad 22: unconnected-(M1-P1.05/AIN1-Pad22) -> /AIN1
- M1 pad 23: unconnected-(M1-P1.04/AIN0/CLK-Pad23) -> /AIN0
- M1 pad 26: unconnected-(M1-VDD_nRF-Pad26) -> /VDDIO
- M1 pad 32: unconnected-(M1-P1.14/AIN7-Pad32) -> /AIN7
- M1 pad 33: unconnected-(M1-P1.13/AIN6-Pad33) -> /AIN6
- M1 pad 34: unconnected-(M1-P1.12/AIN5/CLK-Pad34) -> /AIN5
- M1 pad 35: unconnected-(M1-P1.11/AIN4/CLK-Pad35) -> /AIN4
- R1 pad 1: /VBAT -> /VDDIO
- R1 pad 2: Net-(Q1A-D) -> /SCL
- R2 pad 1: Net-(J1-CC2) -> /VDDIO
- R2 pad 2: GND -> /SDA
- R3 pad 1: Net-(J1-CC1) -> GND
- R3 pad 2: GND -> Net-(PMIC1-VSET1)
- R4 pad 1: Net-(Q1B-D) -> GND
- R4 pad 2: /BAT_MON -> Net-(PMIC1-VSET2)
- TMR1 pad 1: +2V1_TMR -> VCCS
- TMR10 pad 1: +2V1_TMR -> VCCS
- TMR11 pad 1: +2V1_TMR -> VCCS
- TMR12 pad 1: +2V1_TMR -> VCCS
- TMR13 pad 1: +2V1_TMR -> VCCS
- TMR14 pad 1: +2V1_TMR -> VCCS
- TMR15 pad 1: +2V1_TMR -> VCCS
- TMR16 pad 1: +2V1_TMR -> VCCS
- TMR17 pad 1: +2V1_TMR -> VCCS
- TMR18 pad 1: +2V1_TMR -> VCCS
- TMR19 pad 1: +2V1_TMR -> VCCS
- TMR2 pad 1: +2V1_TMR -> VCCS
- TMR20 pad 1: +2V1_TMR -> VCCS
- TMR21 pad 1: +2V1_TMR -> VCCS
- TMR22 pad 1: +2V1_TMR -> VCCS
- TMR23 pad 1: +2V1_TMR -> VCCS
- TMR24 pad 1: +2V1_TMR -> VCCS
- TMR25 pad 1: +2V1_TMR -> VCCS
- TMR26 pad 1: +2V1_TMR -> VCCS
- TMR27 pad 1: +2V1_TMR -> VCCS
- TMR28 pad 1: +2V1_TMR -> VCCS
- TMR29 pad 1: +2V1_TMR -> VCCS
- TMR3 pad 1: +2V1_TMR -> VCCS
- TMR30 pad 1: +2V1_TMR -> VCCS
- TMR31 pad 1: +2V1_TMR -> VCCS
- TMR32 pad 1: +2V1_TMR -> VCCS
- TMR33 pad 1: +2V1_TMR -> VCCS
- TMR34 pad 1: +2V1_TMR -> VCCS
- TMR35 pad 1: +2V1_TMR -> VCCS
- TMR36 pad 1: +2V1_TMR -> VCCS
- TMR37 pad 1: +2V1_TMR -> VCCS
- TMR38 pad 1: +2V1_TMR -> VCCS
- TMR39 pad 1: +2V1_TMR -> VCCS
- TMR4 pad 1: +2V1_TMR -> VCCS
- TMR40 pad 1: +2V1_TMR -> VCCS
- TMR41 pad 1: +2V1_TMR -> VCCS
- TMR42 pad 1: +2V1_TMR -> VCCS
- TMR43 pad 1: +2V1_TMR -> VCCS
- TMR44 pad 1: +2V1_TMR -> VCCS
- TMR45 pad 1: +2V1_TMR -> VCCS
- TMR46 pad 1: +2V1_TMR -> VCCS
- TMR47 pad 1: +2V1_TMR -> VCCS
- TMR48 pad 1: +2V1_TMR -> VCCS
- TMR49 pad 1: +2V1_TMR -> VCCS
- TMR5 pad 1: +2V1_TMR -> VCCS
- TMR50 pad 1: +2V1_TMR -> VCCS
- TMR51 pad 1: +2V1_TMR -> VCCS
- TMR52 pad 1: +2V1_TMR -> VCCS
- TMR53 pad 1: +2V1_TMR -> VCCS
- TMR54 pad 1: +2V1_TMR -> VCCS
- TMR55 pad 1: +2V1_TMR -> VCCS
- TMR56 pad 1: +2V1_TMR -> VCCS
- TMR57 pad 1: +2V1_TMR -> VCCS
- TMR58 pad 1: +2V1_TMR -> VCCS
- TMR59 pad 1: +2V1_TMR -> VCCS
- TMR6 pad 1: +2V1_TMR -> VCCS
- TMR60 pad 1: +2V1_TMR -> VCCS
- TMR61 pad 1: +2V1_TMR -> VCCS
- TMR62 pad 1: +2V1_TMR -> VCCS
- TMR63 pad 1: +2V1_TMR -> VCCS
- TMR64 pad 1: +2V1_TMR -> VCCS
- TMR65 pad 1: +2V1_TMR -> VCCS
- TMR66 pad 1: +2V1_TMR -> VCCS
- TMR67 pad 1: +2V1_TMR -> VCCS
- TMR68 pad 1: +2V1_TMR -> VCCS
- TMR69 pad 1: +2V1_TMR -> VCCS
- TMR7 pad 1: +2V1_TMR -> VCCS
- TMR70 pad 1: +2V1_TMR -> VCCS
- TMR71 pad 1: +2V1_TMR -> VCCS
- TMR72 pad 1: +2V1_TMR -> VCCS
- TMR8 pad 1: +2V1_TMR -> VCCS
- TMR9 pad 1: +2V1_TMR -> VCCS
