File: pcb/pcb.kicad_sch (KiCad schematic)
At the start: 228 parts, among them SW1 SW_DIP_x01_XKB_TS_2030, SW2 SW_DIP_x01_XKB_TS_2030, U1 RP2040, U2 Memory_Flash_W25Q64_XSON, U3 NCP114ASN330T1G, X1 12.000MHz

Commit message: M  notes/nRF52840.md M  notes/notes.md A  notes/spi M  pcb/pcb.kicad_pcb M  pcb/pcb.kicad_prl M  pcb/pcb.kicad_pro M  pcb/pcb.kicad_sch M  pickle.py D  place.py A  placefp.py D  remove_tracks.py A  rmtracks.py M  tmr-footprints/MCP3208-SOIC-16_3.9x9.9mm_P1.27mm.kicad_mod M  tmr-footprints/sw_lowpro_gateron_MDT.kicad_mod A  tmr-footprints/sw_lowpro_gateron_MDT_2.kicad_mod A  tmr-footprints/sw_lowpro_gateron_MDT_3.kicad_mod A  tmr-footprints/sw_lowpro_gateron_MDT_4.kicad_mod
Parts:
- removed C2, C3, C4, C5, C6, C7, C8, C9: C_Small_US, tmr-lib:C_0603_1608Metric, symbol Device:C_Small_US
- added C21, C22, C23, C24, C25, C26, C27, C28: C_Small_US, tmr-lib:C_0603_1608Metric, symbol Device:C_Small_US
- added R14, R17, R18, R19, R20, R21, R22, R23, R24, R25, R9: 33R, symbol Device:R_Small
- USB1: renamed from USBCon1; footprint Connector_USB:USB_C_Receptacle_XKB_U262-16XN-4BVC11 -> Connector_USB:USB_C_Receptacle_G-Switch_GT-USB-7025
- renumbered C10 to C1, C19 to C10, C20 to C11, C21 to C12, C22 to C13, C23 to C14, C24 to C15, C25 to C16, C26 to C17, C31 to C18, C32 to C19, C11 to C2, C1 to C20, C27 to C29, C12 to C3, C28 to C30, C29 to C31, C30 to C32, C13 to C4, C14 to C5, C15 to C6, C16 to C7, C17 to C8, C18 to C9, LedDr1 to LD1, R8 to R10, R9 to R11, R10 to R12, R11 to R13, R12 to R15, R13 to R16, R14 to R8
Connections:
- net GPIO0 is gone; now on net MISO: U1.2 (GPIO0)
- net +3V3: now also C21.1, C22.1, C23.1, C24.1, C25.1, C26.1, C27.1, C28.1
- net GND: now also C21.2, C22.2, C23.2, C24.2, C25.2, C26.2, C27.2, C28.2
- net GPIO2: now also R14.1
- net GPIO3: now also R9.2
- net ANA_40: now reaches S40.2 (V_{OUT})
- net ANA_40: now also ADC8.6 (CH5)
- net ANA_15: now reaches S15.2 (V_{OUT})
- net ANA_15: now also ADC6.7 (CH6)
- net ANA_69: now reaches ADC9.1 (CH0)
- net ANA_69: now also S69.2 (V_{OUT})
- net MOSI: now reaches ADC9.11 (Din)
- net MOSI: now also ADC1.11 (Din), ADC2.11 (Din), ADC3.11 (Din), ADC4.11 (Din), ADC5.11 (Din), ADC6.11 (Din), ADC7.11 (Din), ADC8.11 (Din), R9.1
- net MISO: now reaches ADC9.12 (Dout)
- net MISO: now also ADC1.12 (Dout), ADC2.12 (Dout), ADC3.12 (Dout), ADC4.12 (Dout), ADC5.12 (Dout), ADC6.12 (Dout), ADC7.12 (Dout), ADC8.12 (Dout)
- net SCK: now reaches ADC9.13 (CLK)
- net SCK: now also ADC1.13 (CLK), ADC2.13 (CLK), ADC3.13 (CLK), ADC4.13 (CLK), ADC5.13 (CLK), ADC6.13 (CLK), ADC7.13 (CLK), ADC8.13 (CLK), R14.2
- net ANA_68: now reaches ADC9.2 (CH1)
- net ANA_68: now also S68.2 (V_{OUT})
- net ANA_67: now reaches ADC9.3 (CH2)
- net ANA_67: now also S67.2 (V_{OUT})
- net ANA_53: now reaches ADC9.4 (CH3)
- net ANA_53: now also S53.2 (V_{OUT})
- net ANA_54: now reaches ADC9.5 (CH4)
- net ANA_54: now also S54.2 (V_{OUT})
- net ANA_55: now reaches ADC9.6 (CH5)
- net ANA_55: now also S55.2 (V_{OUT})
- net ANA_56: now reaches ADC9.7 (CH6)
- net ANA_56: now also S56.2 (V_{OUT})
- net ANA_70: now reaches ADC9.8 (CH7)
- net ANA_70: now also S70.2 (V_{OUT})
- net ANA_43: now reaches ADC8.1 (CH0)
- net ANA_43: now also S43.2 (V_{OUT})
- net ANA_71: now reaches ADC8.2 (CH1)
- net ANA_71: now also S71.2 (V_{OUT})
- net ANA_57: now reaches ADC8.3 (CH2)
- net ANA_57: now also S57.2 (V_{OUT})
- net ANA_38: now reaches ADC8.4 (CH3)
- net ANA_38: now also S38.2 (V_{OUT})
- net ANA_39: now reaches ADC8.5 (CH4)
- net ANA_39: now also S39.2 (V_{OUT})
- net ANA_41: now reaches ADC8.7 (CH6)
- net ANA_41: now also S41.2 (V_{OUT})
- net ANA_42: now reaches ADC8.8 (CH7)
- net ANA_42: now also S42.2 (V_{OUT})
- net ANA_44: now reaches ADC7.1 (CH0)
- net ANA_44: now also S44.2 (V_{OUT})
- net ANA_58: now reaches ADC7.2 (CH1)
- net ANA_58: now also S58.2 (V_{OUT})
- net ANA_72: now reaches ADC7.3 (CH2)
- net ANA_72: now also S72.2 (V_{OUT})
- net ANA_24: now reaches ADC7.4 (CH3)
- net ANA_24: now also S24.2 (V_{OUT})
- net ANA_25: now reaches ADC7.5 (CH4)
- net ANA_25: now also S25.2 (V_{OUT})
- net ANA_26: now reaches ADC7.6 (CH5)
- net ANA_26: now also S26.2 (V_{OUT})
- net ANA_27: now reaches ADC7.7 (CH6)
- net ANA_27: now also S27.2 (V_{OUT})
- net ANA_28: now reaches ADC7.8 (CH7)
- net ANA_28: now also S28.2 (V_{OUT})
- net ANA_64: now reaches S64.2 (V_{OUT})
- net ANA_64: now also ADC5.4 (CH3)
- net ANA_35: now reaches S35.2 (V_{OUT})
- net ANA_35: now also ADC3.6 (CH5)
- net ANA_19: now reaches S19.2 (V_{OUT})
- net ANA_19: now also ADC2.4 (CH3)
- net ANA_52: now reaches S52.2 (V_{OUT})
- net ANA_52: now also ADC5.1 (CH0)
- net ANA_34: now reaches S34.2 (V_{OUT})
- net ANA_34: now also ADC3.5 (CH4)
- net ANA_17: now reaches S17.2 (V_{OUT})
- net ANA_17: now also ADC2.2 (CH1)
- net ANA_30: now reaches S30.2 (V_{OUT})
- net ANA_30: now also ADC3.1 (CH0)
- net ANA_14: now reaches S14.2 (V_{OUT})
- net ANA_14: now also ADC6.6 (CH5)
- net ANA_02: now reaches S2.2 (V_{OUT})
- net ANA_02: now also ADC1.2 (CH1)
- net ANA_09: now reaches S9.2 (V_{OUT})
- net ANA_09: now also ADC6.1 (CH0)
- net ANA_20: now reaches S20.2 (V_{OUT})
- net ANA_20: now also ADC2.5 (CH4)
- net ANA_18: now reaches S18.2 (V_{OUT})
- net ANA_18: now also ADC2.3 (CH2)
- net ANA_22: now reaches S22.2 (V_{OUT})
- net ANA_22: now also ADC2.7 (CH6)
- net ANA_66: now reaches ADC5.2 (CH1)
- net ANA_66: now also S66.2 (V_{OUT})
- net ANA_65: now reaches ADC5.3 (CH2)
- net ANA_65: now also S65.2 (V_{OUT})
- net ANA_48: now reaches ADC5.5 (CH4)
- net ANA_48: now also S48.2 (V_{OUT})
- net ANA_49: now reaches ADC5.6 (CH5)
- net ANA_49: now also S49.2 (V_{OUT})
- net ANA_50: now reaches ADC5.7 (CH6)
- net ANA_50: now also S50.2 (V_{OUT})
- net ANA_51: now reaches ADC5.8 (CH7)
- net ANA_51: now also S51.2 (V_{OUT})
- net ANA_63: now reaches S63.2 (V_{OUT})
- net ANA_63: now also ADC4.3 (CH2)
- net ANA_36: now reaches S36.2 (V_{OUT})
- net ANA_36: now also ADC3.7 (CH6)
- net ANA_37: now reaches S37.2 (V_{OUT})
- net ANA_37: now also ADC3.8 (CH7)
- net ANA_16: now reaches S16.2 (V_{OUT})
- net ANA_16: now also ADC2.1 (CH0)
- net ANA_21: now reaches S21.2 (V_{OUT})
- net ANA_21: now also ADC2.6 (CH5)
- net ANA_23: now reaches ADC2.8 (CH7)
- net ANA_23: now also S23.2 (V_{OUT})
- net ANA_31: now reaches ADC3.2 (CH1)
- net ANA_31: now also S31.2 (V_{OUT})
- net ANA_32: now reaches ADC3.3 (CH2)
- net ANA_32: now also S32.2 (V_{OUT})
- net ANA_33: now reaches ADC3.4 (CH3)
- net ANA_33: now also S33.2 (V_{OUT})
- net ANA_03: now reaches S3.2 (V_{OUT})
- net ANA_03: now also ADC1.3 (CH2)
- net ANA_04: now reaches S4.2 (V_{OUT})
- net ANA_04: now also ADC1.4 (CH3)
- net ANA_11: now reaches S11.2 (V_{OUT})
- net ANA_11: now also ADC6.3 (CH2)
- net ANA_60: now reaches S60.2 (V_{OUT})
- net ANA_60: now also ADC4.5 (CH4)
- net ANA_08: now reaches S8.2 (V_{OUT})
- net ANA_08: now also ADC1.8 (CH7)
- net ANA_29: now reaches S29.2 (V_{OUT})
- net ANA_29: now also ADC6.8 (CH7)
- net ANA_05: now reaches S5.2 (V_{OUT})
- net ANA_05: now also ADC1.5 (CH4)
- net ANA_46: now reaches S46.2 (V_{OUT})
- net ANA_46: now also ADC4.8 (CH7)
- net ANA_62: now reaches S62.2 (V_{OUT})
- net ANA_62: now also ADC4.2 (CH1)
- net ANA_01: now reaches ADC1.1 (CH0)
- net ANA_01: now also S1.2 (V_{OUT})
- net ANA_06: now reaches ADC1.6 (CH5)
- net ANA_06: now also S6.2 (V_{OUT})
- net ANA_07: now reaches ADC1.7 (CH6)
- net ANA_07: now also S7.2 (V_{OUT})
- net ANA_47: now reaches S47.2 (V_{OUT})
- net ANA_47: now also ADC4.1 (CH0)
- net ANA_61: now reaches ADC4.4 (CH3)
- net ANA_61: now also S61.2 (V_{OUT})
- net ANA_59: now reaches ADC4.6 (CH5)
- net ANA_59: now also S59.2 (V_{OUT})
- net ANA_45: now reaches ADC4.7 (CH6)
- net ANA_45: now also S45.2 (V_{OUT})
- net ANA_10: now reaches S10.2 (V_{OUT})
- net ANA_10: now also ADC6.2 (CH1)
- net ANA_12: now reaches ADC6.4 (CH3)
- net ANA_12: now also S12.2 (V_{OUT})
- net ANA_13: now reaches ADC6.5 (CH4)
- net ANA_13: now also S13.2 (V_{OUT})
- new net CS_1: R17.2
- new net CS_2: R18.2
- new net CS_3: R19.2
- new net CS_4: R20.2
- new net CS_5: R21.2
- new net CS_6: R22.2
- new net CS_7: R23.2
- new net CS_8: R24.2
- new net CS_9: R25.2
Other:
- moved on the sheet: ADC1, C1, C10, C11, C12, C13, C14, C15, C16, C17, C18, C19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

Commit message: R  pickle.py -> dumploc.py M  notes/spi M  pcb/pcb.kicad_pcb M  pcb/pcb.kicad_prl M  pcb/pcb.kicad_pro M  pcb/pcb.kicad_sch M  placefp.py M  tmr-footprints/LED-6028.kicad_mod
Parts:
- R14, R17, R18, R19, R20, R21, R22, R23, R24, R25, R9: footprint (none) -> tmr-lib:R_0603_1608Metric
Connections:
- net GPIO8 is gone; now on net MISO: U1.11 (GPIO8)
- net ANA_14: now also ADC6.8 (CH7); no longer ADC6.6 (CH5)
- net ANA_16: now also ADC2.2 (CH1); no longer ADC2.1 (CH0)
- net ANA_17: now also ADC2.3 (CH2); no longer ADC2.2 (CH1)
- net ANA_18: now also ADC2.8 (CH7); no longer ADC2.3 (CH2)
- net ANA_19: now also ADC2.7 (CH6); no longer ADC2.4 (CH3)
- net ANA_20: now also ADC2.6 (CH5); no longer ADC2.5 (CH4)
- net ANA_21: now also ADC2.5 (CH4); no longer ADC2.6 (CH5)
- net ANA_22: now also ADC2.4 (CH3); no longer ADC2.7 (CH6)
- net ANA_23: now also ADC2.1 (CH0); no longer ADC2.8 (CH7)
- net ANA_24: now also ADC7.1 (CH0); no longer ADC7.4 (CH3)
- net ANA_25: now also ADC7.2 (CH1); no longer ADC7.5 (CH4)
- net ANA_26: now also ADC7.3 (CH2); no longer ADC7.6 (CH5)
- net ANA_27: now also ADC7.4 (CH3); no longer ADC7.7 (CH6)
- net ANA_28: now also ADC7.5 (CH4); no longer ADC7.8 (CH7)
- net ANA_29: now also ADC6.6 (CH5); no longer ADC6.8 (CH7)
- net ANA_30: now also ADC3.8 (CH7); no longer ADC3.1 (CH0)
- net ANA_31: now also ADC3.1 (CH0); no longer ADC3.2 (CH1)
- net ANA_32: now also ADC3.2 (CH1); no longer ADC3.3 (CH2)
- net ANA_33: now also ADC3.3 (CH2); no longer ADC3.4 (CH3)
- net ANA_34: now also ADC3.4 (CH3); no longer ADC3.5 (CH4)
- net ANA_35: now also ADC3.5 (CH4); no longer ADC3.6 (CH5)
- net ANA_36: now also ADC3.6 (CH5); no longer ADC3.7 (CH6)
- net ANA_37: now also ADC3.7 (CH6); no longer ADC3.8 (CH7)
- net ANA_38: now also ADC8.1 (CH0); no longer ADC8.4 (CH3)
- net ANA_39: now also ADC8.2 (CH1); no longer ADC8.5 (CH4)
- net ANA_40: now also ADC8.3 (CH2); no longer ADC8.6 (CH5)
- net ANA_41: now also ADC8.4 (CH3); no longer ADC8.7 (CH6)
- net ANA_42: now also ADC8.5 (CH4); no longer ADC8.8 (CH7)
- net ANA_43: now also ADC8.6 (CH5); no longer ADC8.1 (CH0)
- net ANA_44: now also ADC7.6 (CH5); no longer ADC7.1 (CH0)
- net ANA_53: now also ADC9.6 (CH5); no longer ADC9.4 (CH3)
- net ANA_54: now also ADC9.7 (CH6); no longer ADC9.5 (CH4)
- net ANA_55: now also ADC9.8 (CH7); no longer ADC9.6 (CH5)
- net ANA_56: now also ADC9.1 (CH0); no longer ADC9.7 (CH6)
- net ANA_57: now also ADC8.7 (CH6); no longer ADC8.3 (CH2)
- net ANA_58: now also ADC7.7 (CH6); no longer ADC7.2 (CH1)
- net ANA_67: now also ADC9.4 (CH3); no longer ADC9.3 (CH2)
- net ANA_68: now also ADC9.5 (CH4); no longer ADC9.2 (CH1)
- net ANA_69: now also ADC9.3 (CH2); no longer ADC9.1 (CH0)
- net ANA_70: now also ADC9.2 (CH1); no longer ADC9.8 (CH7)
- net ANA_71: now also ADC8.8 (CH7); no longer ADC8.2 (CH1)
- net ANA_72: now also ADC7.8 (CH7); no longer ADC7.3 (CH2)
- net GPIO1: now also ADC7.10 (~{CS}/SHDN)
- net GPIO10: now also R14.1
- net GPIO11: now also ADC4.10 (~{CS}/SHDN)
- net GPIO12: now also ADC5.10 (~{CS}/SHDN)
- net GPIO13: now also ADC9.10 (~{CS}/SHDN)
- net GPIO14: now also ADC8.10 (~{CS}/SHDN)
- net GPIO2: now also ADC1.10 (~{CS}/SHDN); no longer R14.1
- net GPIO3: now also ADC2.10 (~{CS}/SHDN); no longer R9.2
- net GPIO7: now also R9.2
- net GPIO9: now also ADC3.10 (~{CS}/SHDN)
- net MISO: no longer U1.2 (GPIO0)
- net GPIO0: now reaches ADC6.10 (~{CS}/SHDN)
- net GPIO0: now also U1.2 (GPIO0)
Other:
- moved on the sheet: R9

Commit message: M  notes/spi M  pcb/pcb.kicad_pcb M  pcb/pcb.kicad_sch M  placefp.py A  tracks.py
Parts:
- removed R17, R18, R19, R20, R21, R22, R23, R24, R25: 33R, tmr-lib:R_0603_1608Metric, symbol Device:R_Small
