File: pcb/pcb.kicad_sch (KiCad schematic)
At the start: 230 parts, among them SW1 SW_DIP_x01_XKB_TS_2030, SW2 SW_DIP_x01_XKB_TS_2030, U1 RP2040, U2 Memory_Flash_W25Q64_XSON, U3 NCP114ASN330T1G, X1 12.000MHz

Commit message: M  notes/nRF52840.md A  notes/soldering M  pcb/pcb.kicad_pcb M  pcb/pcb.kicad_pro M  pcb/pcb.kicad_sch M  placefp.py M  tmr-footprints/sw_lowpro_gateron_MDT.kicad_mod M  tmr-symbols.kicad_sym M  tracks.py
Parts:
- removed C32: 100nF, tmr-lib:C_0603_1608Metric, symbol Device:C_Small
- added F1: 500ma, Fuse:Fuse_0603_1608Metric, symbol Device:Polyfuse_Small
- added Q2: AO3401A, Package_TO_SOT_SMD:SOT-23, symbol Transistor_FET:AO3401A
- added R17: 100k, tmr-lib:R_0603_1608Metric, symbol Device:R_Small
- added R18: 100R, tmr-lib:R_0603_1608Metric, symbol Device:R_Small
Connections:
- net GPIO16 is gone; now on net SDA: U1.27 (GPIO16)
- net GPIO17 is gone; now on net SCL: U1.28 (GPIO17)
- net RESET is gone; now on net RUN: R1.2, SW1.2
- net SDB is gone; now on net GPIO18: LD1.3 (~{SDB}), R13.2
- net +3V3: now also Q2.2 (S), R17.2; no longer ADC1.15 (Vref), ADC1.16 (Vdd), ADC2.15 (Vref), ADC2.16 (Vdd), ADC3.15 (Vref), ADC3.16 (Vdd), ADC4.15 (Vref), ADC4.16 (Vdd), ADC5.15 (Vref), ADC5.16 (Vdd), ADC6.15 (Vref), ADC6.16 (Vdd), ADC7.15 (Vref), ADC7.16 (Vdd), ADC8.15 (Vref), ADC8.16 (Vdd), ADC9.15 (Vref), ADC9.16 (Vdd), C20.1, C21.1, C22.1, C23.1, C24.1, C25.1, C26.1, C27.1, C28.1, S1.1 (V_{CC}), S10.1 (V_{CC}), S11.1 (V_{CC}), S12.1 (V_{CC}), S13.1 (V_{CC}), S14.1 (V_{CC}), S15.1 (V_{CC}), S16.1 (V_{CC}), S17.1 (V_{CC}), S18.1 (V_{CC}), S19.1 (V_{CC}), S2.1 (V_{CC}), S20.1 (V_{CC}), S21.1 (V_{CC}), S22.1 (V_{CC}), S23.1 (V_{CC}), S24.1 (V_{CC}), S25.1 (V_{CC}), S26.1 (V_{CC}), S27.1 (V_{CC}), S28.1 (V_{CC}), S29.1 (V_{CC}), S3.1 (V_{CC}), S30.1 (V_{CC}), S31.1 (V_{CC}), S32.1 (V_{CC}), S33.1 (V_{CC}), S34.1 (V_{CC}), S35.1 (V_{CC}), S36.1 (V_{CC}), S37.1 (V_{CC}), S38.1 (V_{CC}), S39.1 (V_{CC}), S4.1 (V_{CC}), S40.1 (V_{CC}), S41.1 (V_{CC}), S42.1 (V_{CC}), S43.1 (V_{CC}), S44.1 (V_{CC}), S45.1 (V_{CC}), S46.1 (V_{CC}), S47.1 (V_{CC}), S48.1 (V_{CC}), S49.1 (V_{CC}), S5.1 (V_{CC}), S50.1 (V_{CC}), S51.1 (V_{CC}), S52.1 (V_{CC}), S53.1 (V_{CC}), S54.1 (V_{CC}), S55.1 (V_{CC}), S56.1 (V_{CC}), S57.1 (V_{CC}), S58.1 (V_{CC}), S59.1 (V_{CC}), S6.1 (V_{CC}), S60.1 (V_{CC}), S61.1 (V_{CC}), S62.1 (V_{CC}), S63.1 (V_{CC}), S64.1 (V_{CC}), S65.1 (V_{CC}), S66.1 (V_{CC}), S67.1 (V_{CC}), S68.1 (V_{CC}), S69.1 (V_{CC}), S7.1 (V_{CC}), S70.1 (V_{CC}), S71.1 (V_{CC}), S72.1 (V_{CC}), S8.1 (V_{CC}), S9.1 (V_{CC})
- net +5V: now also F1.2
- net GPIO19: now also R18.1
- net VBUS: now also F1.1
- new net: Q2.1 (G), R17.1, R18.2
- new net VCC: ADC1.15 (Vref), ADC1.16 (Vdd), ADC2.15 (Vref), ADC2.16 (Vdd), ADC3.15 (Vref), ADC3.16 (Vdd), ADC4.15 (Vref), ADC4.16 (Vdd), ADC5.15 (Vref), ADC5.16 (Vdd), ADC6.15 (Vref), ADC6.16 (Vdd), ADC7.15 (Vref), ADC7.16 (Vdd), ADC8.15 (Vref), ADC8.16 (Vdd), ADC9.15 (Vref), ADC9.16 (Vdd), C20.1, C21.1, C22.1, C23.1, C24.1, C25.1, C26.1, C27.1, C28.1, Q2.3 (D), S1.1 (V_{CC}), S10.1 (V_{CC}), S11.1 (V_{CC}), S12.1 (V_{CC}), S13.1 (V_{CC}), S14.1 (V_{CC}), S15.1 (V_{CC}), S16.1 (V_{CC}), S17.1 (V_{CC}), S18.1 (V_{CC}), S19.1 (V_{CC}), S2.1 (V_{CC}), S20.1 (V_{CC}), S21.1 (V_{CC}), S22.1 (V_{CC}), S23.1 (V_{CC}), S24.1 (V_{CC}), S25.1 (V_{CC}), S26.1 (V_{CC}), S27.1 (V_{CC}), S28.1 (V_{CC}), S29.1 (V_{CC}), S3.1 (V_{CC}), S30.1 (V_{CC}), S31.1 (V_{CC}), S32.1 (V_{CC}), S33.1 (V_{CC}), S34.1 (V_{CC}), S35.1 (V_{CC}), S36.1 (V_{CC}), S37.1 (V_{CC}), S38.1 (V_{CC}), S39.1 (V_{CC}), S4.1 (V_{CC}), S40.1 (V_{CC}), S41.1 (V_{CC}), S42.1 (V_{CC}), S43.1 (V_{CC}), S44.1 (V_{CC}), S45.1 (V_{CC}), S46.1 (V_{CC}), S47.1 (V_{CC}), S48.1 (V_{CC}), S49.1 (V_{CC}), S5.1 (V_{CC}), S50.1 (V_{CC}), S51.1 (V_{CC}), S52.1 (V_{CC}), S53.1 (V_{CC}), S54.1 (V_{CC}), S55.1 (V_{CC}), S56.1 (V_{CC}), S57.1 (V_{CC}), S58.1 (V_{CC}), S59.1 (V_{CC}), S6.1 (V_{CC}), S60.1 (V_{CC}), S61.1 (V_{CC}), S62.1 (V_{CC}), S63.1 (V_{CC}), S64.1 (V_{CC}), S65.1 (V_{CC}), S66.1 (V_{CC}), S67.1 (V_{CC}), S68.1 (V_{CC}), S69.1 (V_{CC}), S7.1 (V_{CC}), S70.1 (V_{CC}), S71.1 (V_{CC}), S72.1 (V_{CC}), S8.1 (V_{CC}), S9.1 (V_{CC})
Other:
- note added: "ADC Expanders"
- note added: "To Turn Power for Sensors MCU drives GPIO LOW. V_GS becomes -3.3V, turning the P-FET ON. Choose between AO3401A and Si2301."
- moved on the sheet: C1, C10, C11, C12, C13, C14, C15, C16, C17, C18, C19, C2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

Commit message: A  nordic-lib-kicad-npm.kicad_sym M  notes/analog A  notes/charging A  notes/leds A  notes/loadsw R  notes/notes.md -> notes/notes A  notes/nuts M  notes/parts A  notes/scan A  pcb/LED.kicad_sch M  pcb/pcb.kicad_prl M  pcb/pcb.kicad_pro M  pcb/pcb.kicad_sch A  pcb/switch.kicad_sch M  pcb/sym-lib-table R  tmr-footprints/gateron_sw_lowpro.kicad_mod -> tmr-footprints/Gateron_Switch_Lowpro.kicad_mod A  tmr-footprints/LED_1206_3216Metric_ReverseMount_Hole2.2x1.8mm.kicad_mod A  tmr-footprints/Stabilizer_Lowpro_2U.kicad_mod A  tmr-footprints/Texas_DSBGA-4_0.8x0.8mm_Layout2x2_P0.4mm.kicad_mod D  tmr-footprints/sw_lowpro_gateron_MDT_2.kicad_mod D  tmr-footprints/sw_lowpro_gateron_MDT_3.kicad_mod D  tmr-footprints/sw_lowpro_gateron_MDT_4.kicad_mod M  tmr-symbols.kicad_sym
Parts:
- removed ADC1, ADC2, ADC3, ADC4, ADC5, ADC6, ADC7, ADC8, ADC9: MCP3208, tmr-lib:MCP3208-SOIC-16_3.9x9.9mm_P1.27mm, symbol Analog_ADC:MCP3208
- removed C20, C21, C22, C23, C24, C25, C26, C27, C28: C_Small_US, tmr-lib:C_0603_1608Metric, symbol Device:C_Small_US
- removed R14, R9: 33R, tmr-lib:R_0603_1608Metric, symbol Device:R_Small
- removed S1, S10, S11, S12, S13, S14, S15, S16, S17, S18, S19, S2, S20, S21, S22, S23, S24, S25, S26, S27, S28, S29, S3, S30, S31, S32, S33, S34, S35, S36, S37, S38, S39, S4, S40, S41, S42, S43, S44, S45, S46, S47, S48, S49, S5, S50, S51, S52, S53, S54, S55, S56, S57, S58, S59, S6, S60, S61, S62, S63, S64, S65, S66, S67, S68, S69, S7, S70, S71, S72, S8, S9: TMR_switch_MDT, tmr-lib:sw_lowpro_gateron_MDT, symbol tmr-lib:TMR_switch_MDT
- added BT1: Battery_Cell, symbol Device:Battery_Cell
- added C33, C34, C35, C36, C37, C86: C_Small, symbol Device:C_Small
- added C60: 0.1uF, Capacitor_SMD:C_0603_1608Metric, symbol Device:C_Small_US
- added J1: USB_C_Receptacle_PowerOnly_6P, symbol Connector:USB_C_Receptacle_PowerOnly_6P
- added L1: L_Small, symbol Device:L_Small
- added Q1: DMC2400UV, Package_TO_SOT_SMD:SOT-563, symbol tmr-lib:DMC2400UV
- added Q3: Si2302CDS, Package_TO_SOT_SMD:SOT-23-3, symbol tmr-lib:Si2302CDS
- added R1, R19, R20, R21, R22, R? (x2): R_Small, symbol Device:R_Small
- added R14, R23, R9: R, symbol Device:R
- added SW3: SW_DIP_x01, symbol Switch:SW_DIP_x01
- added TH1: Thermistor_NTC, symbol Device:Thermistor_NTC
- added U33: TPS22902, tmr-lib:Texas_DSBGA-4_0.8x0.8mm_Layout2x2_P0.4mm, symbol tmr-lib:TPS22902
- added U4: nPM1100-QDXX, Package_DFN_QFN:QFN-24-1EP_4x4mm_P0.5mm_EP2.6x2.6mm_ThermalVias, symbol nordic-npm:nPM1100-QDXX
- added U8: ADG706BRU, Package_SO:TSSOP-28_4.4x9.7mm_P0.65mm, symbol tmr-lib:ADG706BRU
- C1, C13, C2, C3, C31, C4, C5, C6, C7, C8, C9: value 100nF -> C_Small; footprint tmr-lib:C_0603_1608Metric -> (none); ALTIUM_VALUE 100nF -> (none); CAPACITANCE 100nF -> (none); COMPONENT BODY 1.00 x 0.50mm -> (none); COMPONENT HEIGHT TBD -> (none); COMPONENT SUBTYPE MLCC -> (none); COMPONENT TYPE Capacitor -> (none); DIELECTRIC X7R -> (none); FEATURES TBD -> (none); ID CAP-0026 -> (none); LCSC C155422 -> (none); MANUFACTURER Samsung Electro-Mechanics -> (none); MOUNTING TYPE SMD -> (none); MPN CL05B104KA5NNNC -> (none); OPERATING TEMPERATURE TBD -> (none); PACKAGE (CASE) 0402 (1005) -> (none); PACKAGING TYPE TBD -> (none); ROHS STATUS TBD -> (none); SUPPLIER 1 LCSC -> (none); SUPPLIER 2 Farnell -> (none); SUPPLIER 3 Mouser -> (none); SUPPLIER PART NUMBER 1 C155422 -> (none); SUPPLIER PART NUMBER 2 2496772 -> (none); SUPPLIER PART NUMBER 3 187-CL05B104KA5NNNC -> (none); TOLERANCE TBD -> (none); VOLTAGE RATING 25V -> (none)
- C10, C14, C16: value 2.2uF -> C_Small; footprint tmr-lib:C_0603_1608Metric -> (none); ALTIUM_VALUE 2.2uF -> (none); CAPACITANCE 2.2uF -> (none); COMPONENT BODY 1.00 x 0.50mm -> (none); COMPONENT HEIGHT TBD -> (none); COMPONENT SUBTYPE MLCC -> (none); COMPONENT TYPE Capacitor -> (none); DIELECTRIC X5R -> (none); FEATURES TBD -> (none); ID CAP-0026 -> (none); LCSC C107371 -> (none); MANUFACTURER Samsung Electro-Mechanics -> (none); MOUNTING TYPE SMD -> (none); MPN CL05A225MQ5NNNC -> (none); OPERATING TEMPERATURE TBD -> (none); PACKAGE (CASE) 0402 (1005) -> (none); PACKAGING TYPE TBD -> (none); ROHS STATUS TBD -> (none); SUPPLIER 1 LCSC -> (none); SUPPLIER 2 Farnell -> (none); SUPPLIER 3 Mouser -> (none); SUPPLIER PART NUMBER 1 C107371 -> (none); SUPPLIER PART NUMBER 2 3013335 -> (none); SUPPLIER PART NUMBER 3 187-CL05A225MQ5NNNC -> (none); TOLERANCE TBD -> (none); VOLTAGE RATING 6.3V -> (none)
- C11, C12, C17: value 1uF -> C_Small; footprint tmr-lib:C_0603_1608Metric -> (none); CAPACITANCE 1uf -> (none); COMPONENT SUBTYPE MLCC -> (none); COMPONENT TYPE Capacitor -> (none); ID CAP-0026 -> (none); LCSC C106254 -> (none); MANUFACTURER YAGEO -> (none); MOUNTING TYPE SMD -> (none); MPN CC0402KRX5R6BB105 -> (none); PACKAGE (CASE) 0402 (1005) -> (none)
- C15, C30: value 10uF -> C_Small; footprint tmr-lib:C_0603_1608Metric -> (none); LCSC C596327 -> (none); MPN CC0603MRX5R8BB106 -> (none); Manuf. YAGEO -> (none); Package 0603 -> (none)
- C18, C19: value 15pF -> C_Small; footprint tmr-lib:C_0603_1608Metric -> (none); ALTIUM_VALUE 15pF -> (none); CAPACITANCE 15pF -> (none); COMPONENT BODY 1.00 x 0.50mm -> (none); COMPONENT HEIGHT TBD -> (none); COMPONENT SUBTYPE MLCC -> (none); COMPONENT TYPE Capacitor -> (none); DIELECTRIC C0G/NP0 -> (none); FEATURES TBD -> (none); ID CAP-0026 -> (none); LCSC C106997 -> (none); MANUFACTURER KEMET Corporation -> (none); MOUNTING TYPE SMD -> (none); MPN C0402C150J5GACTU -> (none); OPERATING TEMPERATURE TBD -> (none); PACKAGE (CASE) 0402 (1005) -> (none); PACKAGING TYPE TBD -> (none); ROHS STATUS TBD -> (none); SUPPLIER 1 LCSC -> (none); SUPPLIER 2 Farnell -> (none); SUPPLIER 3 Mouser -> (none); SUPPLIER PART NUMBER 1 C106997 -> (none); SUPPLIER PART NUMBER 2 1414577 -> (none); SUPPLIER PART NUMBER 3 80-C0402C150J5G -> (none); TOLERANCE TBD -> (none); VOLTAGE RATING 50V -> (none)
- C29: value 10uF -> C_Small; footprint tmr-lib:C_1206_3216Metric -> (none); JLC 10uF_tantalum -> (none); LCSC2 C7171 -> (none); Type Tantalum -> (none)
- D1, D10, D11, D12, D13, D14, D15, D16, D17, D18, D19, D2, D20, D21, D22, D23, D24, D25, D26, D27, D28, D29, D3, D30, D31, D32, D33, D34, D35, D36, D37, D38, D39, D4, D40, D41, D42, D43, D44, D45, D46, D47, D48, D49, D5, D50, D51, D52, D53, D54, D55, D56, D57, D58, D59, D6, D60, D61, D62, D63, D64, D65, D66, D67, D68, D69, D7, D70, D71, D72, D8, D9: footprint tmr-lib:LED-6028 -> (none)
- F1: value 500ma -> Polyfuse_Small; footprint Fuse:Fuse_0603_1608Metric -> (none); LCSC C210357 -> (none)
- H1, H2, H3, H4, H5, H6, H7, H8: footprint tmr-lib:MountingHole_5.3mm_M5_ISO14580_Pad_TopBottom -> (none); now left out of the parts list
- R1, R2: value 10k -> R; footprint tmr-lib:R_0603_1608Metric -> (none); ALTIUM_VALUE 10k -> (none); COMPONENT BODY 1.00 x 0.50mm -> (none); COMPONENT HEIGHT 0.35mm -> (none); COMPONENT SUBTYPE Thick Film -> (none); COMPONENT TYPE Resistor -> (none); FEATURES Standard -> (none); ID RES-0004 -> (none); LCSC C60490 -> (none); MANUFACTURER Yageo Corporation -> (none); MOUNTING TYPE SMD -> (none); MPN RC0402FR-0710KL -> (none); OPERATING TEMPERATURE -55°C to +155°C -> (none); PACKAGE (CASE) 0402 (1005) -> (none); PACKAGING TYPE Tape & Reel -> (none); POWER RATING 62.5mW -> (none); RESISTANCE 10k -> (none); ROHS STATUS RoHS Compliant -> (none); SUPPLIER 1 LCSC -> (none); SUPPLIER 2 Farnell -> (none); SUPPLIER 3 Mouser -> (none); SUPPLIER PART NUMBER 1 C60490 -> (none); SUPPLIER PART NUMBER 2 9239359 -> (none); SUPPLIER PART NUMBER 3 603-RC0402FR-0710KL -> (none); TCR 100PPM -> (none); TOLERANCE 1% -> (none); VOLTAGE RATING 50V -> (none)
- R10, R11, R12: value 4.7k -> R_Small; footprint tmr-lib:R_0603_1608Metric -> (none); LCSC C105871 -> (none); Manufacturer Yageo -> (none); Tolerance 1% -> (none); Type Thick Film -> (none)
- R13, R17: value 100k -> R_Small; footprint tmr-lib:R_0603_1608Metric -> (none); JLC 20k -> (none); LCSC C144783 -> (none); Manufacturer Yageo -> (none); Tolerance 1% -> (none); Type Thick Film -> (none)
- R15, R16: value 20k -> R_Small; footprint tmr-lib:R_0603_1608Metric -> (none); JLC 20k -> (none); LCSC C144783 -> (none); Manufacturer Yageo -> (none); Tolerance 1% -> (none); Type Thick Film -> (none)
- R18: value 100R -> R_Small; footprint tmr-lib:R_0603_1608Metric -> (none); Manufacturer Yageo -> (none); Tolerance 1% -> (none); Type Thick Film -> (none)
- R3, R8: value 1k -> R; footprint tmr-lib:R_0603_1608Metric -> (none); ALTIUM_VALUE 1k -> (none); COMPONENT BODY 1.00 x 0.50mm -> (none); COMPONENT HEIGHT 0.35mm -> (none); COMPONENT SUBTYPE Thick Film -> (none); COMPONENT TYPE Resistor -> (none); FEATURES Standard -> (none); ID RES-0003 -> (none); LCSC C106235 -> (none); MANUFACTURER Yageo Corporation -> (none); MOUNTING TYPE SMD -> (none); MPN RC0402FR-071KL -> (none); OPERATING TEMPERATURE -55°C to +155°C -> (none); PACKAGE (CASE) 0402 (1005) -> (none); PACKAGING TYPE Tape & Reel -> (none); POWER RATING 62.5mW -> (none); RESISTANCE 1k -> (none); ROHS STATUS RoHS Compliant -> (none); SUPPLIER 1 LCSC -> (none); SUPPLIER 2 Farnell -> (none); SUPPLIER 3 Mouser -> (none); SUPPLIER PART NUMBER 1 C106235 -> (none); SUPPLIER PART NUMBER 2 9239235 -> (none); SUPPLIER PART NUMBER 3 603-RC0402FR-071KL -> (none); TCR 100PPM -> (none); TOLERANCE 1% -> (none); VOLTAGE RATING 50V -> (none)
- R4, R5: value 27R -> R; footprint tmr-lib:R_0603_1608Metric -> (none); ALTIUM_VALUE 27R -> (none); COMPONENT BODY 1.00 x 0.50mm -> (none); COMPONENT HEIGHT TBD -> (none); COMPONENT SUBTYPE Thick Film -> (none); COMPONENT TYPE Resistor -> (none); FEATURES TBD -> (none); ID RES-0058 -> (none); LCSC C138021 -> (none); MANUFACTURER Yageo Corporation -> (none); MOUNTING TYPE SMD -> (none); MPN RC0402FR-0727RL -> (none); OPERATING TEMPERATURE TBD -> (none); PACKAGE (CASE) 0402 (1005) -> (none); PACKAGING TYPE TBD -> (none); POWER RATING 62.5mW -> (none); RESISTANCE 27R -> (none); ROHS STATUS TBD -> (none); SUPPLIER 1 LCSC -> (none); SUPPLIER 2 Farnell -> (none); SUPPLIER 3 Mouser -> (none); SUPPLIER PART NUMBER 1 C138021 -> (none); SUPPLIER PART NUMBER 2 9239049 -> (none); SUPPLIER PART NUMBER 3 603-RC0402FR-0727RL -> (none); TCR TBD -> (none); TOLERANCE 1% -> (none); VOLTAGE RATING 50V -> (none)
- R6, R7: value 5.1k -> R; footprint tmr-lib:R_0603_1608Metric -> (none); COMPONENT SUBTYPE Thick Film -> (none); COMPONENT TYPE Resistor -> (none); ID RES-0004 -> (none); LCSC C105872 -> (none); MANUFACTURER Yageo Corporation -> (none); MOUNTING TYPE SMD -> (none); MPN RC0402FR-075K1L -> (none); PACKAGE (CASE) 0402 (1005) -> (none); POWER RATING 62.5mW -> (none); TOLERANCE 1% -> (none)
- Stb1, Stb2: footprint tmr-lib:sw_lowpro_stab_2u -> tmr-lib:stabilizer_lowpro_2u
- U1: renamed from LD1; footprint rp2040:QFN-28-1EP_4x4mm_P0.4mm_EP2.3x2.3mm -> Package_DFN_QFN:QFN-28-1EP_4x4mm_P0.4mm_EP2.3x2.3mm; JLCPCB IS31FL3731-QFLS2-TR -> (none); LCSC C191206 -> (none)
Connections:
- net GND: now also BT1.2 (-), C33.2, C34.2, C35.2, C36.2, C37.2, C60.2, C86.1, Q1.1 (S), Q3.2 (S), R1.2, R14.2, R19.2, R22.2, R9.2, R?.2, SW3.2, TH1.2, U33.B1 (GND), U4.12 (ICHG), U4.19 (D-), U4.2 (VOUTBSET1), U4.23 (PVSS), U4.25 (AVSS), U4.4 (AVSS), U4.7 (MODE), U8.12 (GND), U8.27 (VSS)
- net MISO renamed GPIO8
- new net: Q1.5 (G), Q1.6 (D), R20.2
- new net: R23.2, SW3.1, U4.11 (SHPHLD)
- new net: Q3.1 (G), R?.1, R?.1
- new net: C35.1, U4.21 (DEC)
- new net: J1.A12 (GND), J1.B12 (GND)
- new net: J1.A5 (CC1), R14.1
- new net: C36.1, J1.A9 (VBUS), J1.B9 (VBUS), U4.17 (VBUS)
- new net: J1.B5 (CC2), R9.1
- new net: Q1.3 (D), R21.1
- new net: TH1.1, U4.14 (NTC)
- new net: L1.2, U4.22 (SW)
- new net +2V1: C33.1, C86.2, L1.1, U33.A2 (VIN), U4.1 (VOUTB)
- new net +2V1_TMR: C60.1, U33.A1 (VOUT), U8.1 (VDD), U8.18 (EN)
- new net BAT_MON: R21.2, R22.1
- new net BAT_MON_EN: Q1.2 (G), R19.1
- new net BL_PWM: R?.2
- new net CHG: U4.8 (CHG)
- new net ERR: U4.10 (ERR)
- new net LED_CATH: Q3.3 (D)
- new net SHPACT: U4.6 (SHPACT)
- new net TMR_PWR_EN: R1.1, U33.B2 (ON)
- new net VBAT: BT1.1 (+), C37.1, Q1.4 (S), R20.1, R23.1, U4.15 (VBAT)
- new net VSYS: C34.1, U4.16 (VSYS), U4.3 (VOUTBSET0), U4.5 (ISET), U4.9 (VTERMSET)
- no-connect marks 5 -> 6
Other:
- added sheet LED (LED.kicad_sch)
- added sheet LED1 (LED.kicad_sch)
- added sheet LED10 (LED.kicad_sch)
- added sheet LED11 (LED.kicad_sch)
- added sheet LED12 (LED.kicad_sch)
- added sheet LED13 (LED.kicad_sch)
- added sheet LED14 (LED.kicad_sch)
- added sheet LED15 (LED.kicad_sch)
- added sheet LED16 (LED.kicad_sch)
- added sheet LED17 (LED.kicad_sch)
- added sheet LED18 (LED.kicad_sch)
- added sheet LED19 (LED.kicad_sch)
- added sheet LED2 (LED.kicad_sch)
- added sheet LED20 (LED.kicad_sch)
- added sheet LED21 (LED.kicad_sch)
- added sheet LED22 (LED.kicad_sch)
- added sheet LED23 (LED.kicad_sch)
- added sheet LED24 (LED.kicad_sch)
- added sheet LED25 (LED.kicad_sch)
- added sheet LED26 (LED.kicad_sch)
- added sheet LED27 (LED.kicad_sch)
- added sheet LED28 (LED.kicad_sch)
- added sheet LED3 (LED.kicad_sch)
- added sheet LED30 (LED.kicad_sch)
- added sheet LED31 (LED.kicad_sch)
- added sheet LED32 (LED.kicad_sch)
- added sheet LED33 (LED.kicad_sch)
- added sheet LED34 (LED.kicad_sch)
- added sheet LED35 (LED.kicad_sch)
- added sheet LED36 (LED.kicad_sch)
- added sheet LED37 (LED.kicad_sch)
- added sheet LED38 (LED.kicad_sch)
- added sheet LED39 (LED.kicad_sch)
- added sheet LED4 (LED.kicad_sch)
- added sheet LED40 (LED.kicad_sch)
- added sheet LED41 (LED.kicad_sch)
- added sheet LED42 (LED.kicad_sch)
- added sheet LED43 (LED.kicad_sch)
- added sheet LED44 (LED.kicad_sch)
- added sheet LED45 (LED.kicad_sch)
- added sheet LED46 (LED.kicad_sch)
- added sheet LED47 (LED.kicad_sch)
- added sheet LED48 (LED.kicad_sch)
- added sheet LED49 (LED.kicad_sch)
- added sheet LED5 (LED.kicad_sch)
- added sheet LED50 (LED.kicad_sch)
- added sheet LED51 (LED.kicad_sch)
- added sheet LED52 (LED.kicad_sch)
- added sheet LED53 (LED.kicad_sch)
- added sheet LED54 (LED.kicad_sch)
- added sheet LED55 (LED.kicad_sch)
- added sheet LED56 (LED.kicad_sch)
- added sheet LED57 (LED.kicad_sch)
- added sheet LED58 (LED.kicad_sch)
- added sheet LED6 (LED.kicad_sch)
- added sheet LED60 (LED.kicad_sch)
- added sheet LED61 (LED.kicad_sch)
- added sheet LED62 (LED.kicad_sch)
- added sheet LED63 (LED.kicad_sch)
- added sheet LED64 (LED.kicad_sch)
- added sheet LED65 (LED.kicad_sch)
- added sheet LED66 (LED.kicad_sch)
- added sheet LED67 (LED.kicad_sch)
- added sheet LED68 (LED.kicad_sch)
- added sheet LED69 (LED.kicad_sch)
- added sheet LED7 (LED.kicad_sch)
- added sheet LED70 (LED.kicad_sch)
- added sheet LED71 (LED.kicad_sch)
- added sheet LED72 (LED.kicad_sch)
- added sheet LED73 (LED.kicad_sch)
- added sheet LED8 (LED.kicad_sch)
- added sheet LED9 (LED.kicad_sch)
- added sheet Switch58 (switch.kicad_sch)
- added sheet Switch59 (switch.kicad_sch)
- added sheet Switch60 (switch.kicad_sch)
- added sheet Switch61 (switch.kicad_sch)
- added sheet Switch62 (switch.kicad_sch)
- added sheet Switch63 (switch.kicad_sch)
- added sheet Switch64 (switch.kicad_sch)
- added sheet Switch65 (switch.kicad_sch)
- added sheet Switch66 (switch.kicad_sch)
- added sheet Switch67 (switch.kicad_sch)
- added sheet Switch68 (switch.kicad_sch)
- added sheet Switch69 (switch.kicad_sch)
- added sheet Switch70 (switch.kicad_sch)
- added sheet Switch71 (switch.kicad_sch)
- added sheet Switch72 (switch.kicad_sch)
- added sheet Switch73 (switch.kicad_sch)
- note added: "NOTE: - Star Power: Run the 2.1V power from the TPS22902 VOUT to the sensors in a "star" or "tree" pattern, rather than one long daisy chain. This prevents the sensors at the end of the line from seeing a different voltage than the sensors at the start. - The Mux Placement: Place the 5 muxes as close to the nRF54L15 as possible. It is better to have long traces for the TMR outputs (which are slow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"
- note added: "NOTE: Place Rgate close to MCU, and Rpull close to N-MOSFET."
- note added: "NOTE: See page 42 (application example) and 52 (configuration 3) of npm1100 datasheet See Hardware Application Guidelines for inductor choices"
- note added: "NOTE: VIN must provide inrush current to charge 72 x 0.1 uF TMR decoupling capacitors (total 7.2 uF). For a 2.1 V step with 40 us slew: I_inrush = C * dV/dt = 7.2 uF * (2.1 V / 40 us) = 378 mA. This exceeds the nPM1100 buck current limit (150 mA), so local energy storage is required. Place a 10 uF to 22 uF X7R ceramic capacitor close to the TPS22902 VIN pin to supply the inrush current and preven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"
- note added: "PMIC"
- note removed: "ADC Expanders"
- moved on the sheet: C29, C30, C31, D1, D10, D11, D12, D13, D14, D15, D16, D17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

Commit message: A  notes/bypasscaps A  notes/keytravel M  notes/leds A  notes/muxadc M  notes/notes A  notes/pulldown M  notes/scan A  notes/swupdate M  pcb/LED.kicad_sch M  pcb/pcb.kicad_pcb M  pcb/pcb.kicad_prl M  pcb/pcb.kicad_pro M  pcb/pcb.kicad_sch M  pcb/switch.kicad_sch M  placefp.py A  tmr-footprints/C_0402_1005Metric.kicad_mod M  tmr-footprints/C_0603_1608Metric.kicad_mod D  tmr-footprints/C_1206_3216Metric.kicad_mod A  tmr-footprints/Ezurio_BL54L15_Module.kicad_mod A  tmr-footprints/LED_1206_3216Metric_ReverseMount_Hole2.1mm.kicad_mod A  tmr-footprints/Murata_DFE201210U.kicad_mod A  tmr-footprints/R_0402_1005Metric.kicad_mod M  tmr-footprints/SOT-23-3.kicad_mod M  tmr-symbols.kicad_sym
Parts:
- removed BT1: Battery_Cell, symbol Device:Battery_Cell
- removed C1, C10, C11, C12, C13, C14, C15, C16, C17, C18, C19, C2, C29, C3, C30, C31, C4, C5, C6, C7, C8, C9: C_Small, symbol Device:C_Small
- removed D1, D10, D11, D12, D13, D14, D15, D16, D17, D18, D19, D2, D20, D21, D22, D23, D24, D25, D26, D27, D28, D29, D3, D30, D31, D32, D33, D34, D35, D36, D37, D38, D39, D4, D40, D41, D42, D43, D44, D45, D46, D47, D48, D49, D5, D50, D51, D52, D53, D54, D55, D56, D57, D58, D59, D6, D60, D61, D62, D63, D64, D65, D66, D67, D68, D69, D7, D70, D71, D72, D8, D9: LED, symbol Device:LED
- removed F1: Polyfuse_Small, symbol Device:Polyfuse_Small
- removed H2, H3, H4, H5, H6, H7, H8: MountingHole, symbol Mechanical:MountingHole
- removed Hs1, Hs10, Hs2, Hs3, Hs4, Hs5, Hs6, Hs7, Hs8, Hs9: ~, tmr-lib:SMTSO_M1.6, symbol giri:MountingHoleSMD
- removed Q2: AO3401A, Package_TO_SOT_SMD:SOT-23, symbol Transistor_FET:AO3401A
- removed R1, R2, R3, R4, R5, R6, R7, R8: R, symbol Device:R
- removed R10, R11, R12, R13, R15, R16, R17, R18: R_Small, symbol Device:R_Small
- removed SW1, SW2: SW_DIP_x01_XKB_TS_2030, Button_Switch_SMD:SW_SPST_B3U-3000P, symbol RP2040_Minimal:SW_DIP_x01_XKB_TS_2030
- removed TH1: Thermistor_NTC, symbol Device:Thermistor_NTC
- removed U1: IS31FL3731-QF, Package_DFN_QFN:QFN-28-1EP_4x4mm_P0.4mm_EP2.3x2.3mm, symbol Driver_LED:IS31FL3731-QF
- removed U1: RP2040, rp2040:RP2040-QFN-56, symbol RP2040_Minimal:RP2040
- removed U2: Memory_Flash_W25Q64_XSON, rp2040:8-USON, symbol RP2040_Minimal:Memory_Flash_W25Q64_XSON
- removed U3: NCP114ASN330T1G, Package_SO:TSOP-5_1.65x3.05mm_P0.95mm, symbol RP2040_Minimal:Regulator_LDO_ONS_NCP114_TSOP5
- removed U8: ADG706BRU, Package_SO:TSSOP-28_4.4x9.7mm_P0.65mm, symbol tmr-lib:ADG706BRU
- removed USB1: USB_TYPE_C_Receptacle_16P, Connector_USB:USB_C_Receptacle_G-Switch_GT-USB-7025, symbol RP2040_Minimal:USB_TYPE_C_Receptacle_16P
- removed X1: 12.000MHz, rp2040:Crystal_SMD_2520-4Pin_2.5x2.0mm-Handsolder, symbol RP2040_Minimal:Crystal_P4
- added BAT1: Battery_Pack_PS5, Connector_JST:JST_EH_S3B-EH_1x03_P2.50mm_Horizontal, symbol tmr-lib:Battery_Pack_PS5
- added C10, C7, C8, C9: 0.1uF, Capacitor_SMD:C_0402_1005Metric, symbol Device:C_Small_US
- added Hs10, Hs11, Hs12, Hs2, Hs3, Hs4, Hs5, Hs6, Hs7, Hs8, Hs9: M2_Pad, MountingHole:MountingHole_2.2mm_M2_ISO7380_Pad_TopBottom, symbol Mechanical:MountingHole
- added J2: Conn_01x06_Socket, symbol Connector:Conn_01x06_Socket
- added M1: nRF54L15 module, tmr-lib:Ezurio_BL54L15_Module, symbol tmr-lib:Ezurio_BL54L15_TRACE ANT_SCH_Symbol
- added U2, U3, U4, U5, U6: ADG706BRU, Package_SO:TSSOP-28_4.4x9.7mm_P0.65mm, symbol tmr-lib:ADG706BRU
- C1: renamed from C36; value C_Small -> 2.2uF; footprint (none) -> Capacitor_SMD:C_0603_1608Metric
- C11: renamed from C86; value C_Small -> 10uF; footprint (none) -> Capacitor_SMD:C_0603_1608Metric
- C2: renamed from C34; value C_Small -> 10uF; footprint (none) -> Capacitor_SMD:C_0603_1608Metric
- C3: renamed from C37; value C_Small -> 1uF; footprint (none) -> Capacitor_SMD:C_0603_1608Metric
- C4: renamed from C35; value C_Small -> 10uF; footprint (none) -> Capacitor_SMD:C_0603_1608Metric
- C5: renamed from C33; value C_Small -> 10uF; footprint (none) -> Capacitor_SMD:C_0603_1608Metric
- C6: renamed from C60; footprint Capacitor_SMD:C_0603_1608Metric -> Capacitor_SMD:C_0402_1005Metric
- Hs1: renamed from H1; value MountingHole -> M2_Pad; footprint (none) -> MountingHole:MountingHole_2.2mm_M2_ISO7380_Pad_TopBottom
- L1: value L_Small -> 2.2uF; footprint (none) -> tmr-lib:Murata_DFE201210U
- R1: renamed from R20; value R_Small -> 1M0; footprint (none) -> Resistor_SMD:R_0603_1608Metric
- R10: renamed from R1; value R_Small -> 100k; footprint (none) -> Resistor_SMD:R_0603_1608Metric
- R2: renamed from R9; value R -> 5.1k; footprint (none) -> Resistor_SMD:R_0603_1608Metric
- R3: renamed from R14; value R -> 5.1k; footprint (none) -> Resistor_SMD:R_0603_1608Metric
- R4: renamed from R21; value R_Small -> 1M5; footprint (none) -> Resistor_SMD:R_0603_1608Metric
- R5: renamed from R19; value R_Small -> 1M0; footprint (none) -> Resistor_SMD:R_0603_1608Metric
- R6: renamed from R22; value R_Small -> 220k; footprint (none) -> Resistor_SMD:R_0603_1608Metric
- R7: renamed from R23; value R -> 100k; footprint (none) -> Resistor_SMD:R_0603_1608Metric
- R8: renamed from R?; value R_Small -> 220R; footprint (none) -> Resistor_SMD:R_0603_1608Metric
- R9: renamed from R?; value R_Small -> 10k; footprint (none) -> Resistor_SMD:R_0603_1608Metric
- SW1: renamed from SW3; footprint (none) -> TestPoint:TestPoint_Bridge_Pitch3.81mm_Drill1.3mm
- Stb1, Stb2: footprint tmr-lib:stabilizer_lowpro_2u -> tmr-lib:Stabilizer_Lowpro_2U
- renumbered Q3 to Q2, U4 to U1, U33 to U7
Connections:
- net +2V1_TMR: now also C10.1, C7.1, C8.1, C9.1, U2.1 (VDD), U2.18 (EN), U3.1 (VDD), U3.18 (EN), U4.1 (VDD), U4.18 (EN), U5.1 (VDD), U5.18 (EN), U6.1 (VDD), U6.18 (EN)
- net GND: now also BAT1.3 (GND), C10.2, C7.2, C8.2, C9.2, U2.12 (GND), U2.27 (VSS), U3.12 (GND), U3.27 (VSS), U4.12 (GND), U4.27 (VSS), U5.12 (GND), U5.27 (VSS), U6.12 (GND), U6.27 (VSS)
- net VBAT: now also BAT1.1 (VBAT)
- net at U1.14 (NTC): now also BAT1.2 (NTC)
- no-connect marks 6 -> 1
Other:
- removed sheet LED
- removed sheet LED73
- removed sheet Switch73
- added sheet LED29 (LED.kicad_sch)
- added sheet LED59 (LED.kicad_sch)
- added sheet Switch1 (switch.kicad_sch)
- added sheet Switch10 (switch.kicad_sch)
- added sheet Switch11 (switch.kicad_sch)
- added sheet Switch12 (switch.kicad_sch)
- added sheet Switch13 (switch.kicad_sch)
- added sheet Switch14 (switch.kicad_sch)
- added sheet Switch15 (switch.kicad_sch)
- added sheet Switch16 (switch.kicad_sch)
- added sheet Switch17 (switch.kicad_sch)
- added sheet Switch18 (switch.kicad_sch)
- added sheet Switch19 (switch.kicad_sch)
- added sheet Switch2 (switch.kicad_sch)
- added sheet Switch20 (switch.kicad_sch)
- added sheet Switch21 (switch.kicad_sch)
- added sheet Switch22 (switch.kicad_sch)
- added sheet Switch23 (switch.kicad_sch)
- added sheet Switch24 (switch.kicad_sch)
- added sheet Switch25 (switch.kicad_sch)
- added sheet Switch26 (switch.kicad_sch)
- added sheet Switch27 (switch.kicad_sch)
- added sheet Switch28 (switch.kicad_sch)
- added sheet Switch29 (switch.kicad_sch)
- added sheet Switch3 (switch.kicad_sch)
- added sheet Switch30 (switch.kicad_sch)
- added sheet Switch31 (switch.kicad_sch)
- added sheet Switch32 (switch.kicad_sch)
- added sheet Switch33 (switch.kicad_sch)
- added sheet Switch34 (switch.kicad_sch)
- added sheet Switch35 (switch.kicad_sch)
- added sheet Switch36 (switch.kicad_sch)
- added sheet Switch37 (switch.kicad_sch)
- added sheet Switch38 (switch.kicad_sch)
- added sheet Switch39 (switch.kicad_sch)
- added sheet Switch4 (switch.kicad_sch)
- added sheet Switch40 (switch.kicad_sch)
- added sheet Switch41 (switch.kicad_sch)
- added sheet Switch42 (switch.kicad_sch)
- added sheet Switch43 (switch.kicad_sch)
- added sheet Switch44 (switch.kicad_sch)
- added sheet Switch45 (switch.kicad_sch)
- added sheet Switch46 (switch.kicad_sch)
- added sheet Switch47 (switch.kicad_sch)
- added sheet Switch48 (switch.kicad_sch)
- added sheet Switch49 (switch.kicad_sch)
- added sheet Switch5 (switch.kicad_sch)
- added sheet Switch50 (switch.kicad_sch)
- added sheet Switch51 (switch.kicad_sch)
- added sheet Switch52 (switch.kicad_sch)
- added sheet Switch53 (switch.kicad_sch)
- added sheet Switch54 (switch.kicad_sch)
- added sheet Switch55 (switch.kicad_sch)
- added sheet Switch56 (switch.kicad_sch)
- added sheet Switch57 (switch.kicad_sch)
- added sheet Switch6 (switch.kicad_sch)
- added sheet Switch7 (switch.kicad_sch)
- added sheet Switch8 (switch.kicad_sch)
- added sheet Switch9 (switch.kicad_sch)
- sheet Switch58 ports: added VOUTS; removed Vout
- sheet Switch59 ports: added VOUTS; removed Vout
- sheet Switch60 ports: added VOUTS; removed Vout
- sheet Switch61 ports: added VOUTS; removed Vout
- sheet Switch62 ports: added VOUTS; removed Vout
- sheet Switch63 ports: added VOUTS; removed Vout
- sheet Switch64 ports: added VOUTS; removed Vout
- sheet Switch65 ports: added VOUTS; removed Vout
- sheet Switch66 ports: added VOUTS; removed Vout
- sheet Switch67 ports: added VOUTS; removed Vout
- sheet Switch68 ports: added VOUTS; removed Vout
- sheet Switch69 ports: added VOUTS; removed Vout
- sheet Switch70 ports: added VOUTS; removed Vout
- sheet Switch71 ports: added VOUTS; removed Vout
- sheet Switch72 ports: added VOUTS; removed Vout
- note added: "Analog MUXes"
- note added: "Load Switch to pulse TMR sensors"
- note added: "Low Side N-FET Switch for PWM"
- note added: "NOTE: See page 42 (application example) and 52 (configuration 3) of npm1100 datasheet Suggested inductors: Murata DFE201210U-2R2M Samsung CIGT201610EH2R2MNE Samsung CIGT252008LM2R2MNE Taiyo Yuden MDKK1616T2R2MM (See Hardware Application Guidelines for more inductor choices)"
- note removed: "3.3V/300mA LDO"
- note removed: "4-64Mbit Flash, Quad SPI, 100-133MHz, XIP (eXecute In Place), 3.3V: USON 2x3x.6 mm Winbond: W25Q16JVUXIQ (2MB, 133 MHz) GigaDevice: GD25Q40CEIGR (512kB, 120MHz) GigaDevice: GD25Q80CEIGR (1MB, 120 MHz) GigaDevice: GD25Q80EEIGR (1MB, 133MHz) ISSI: IS25LP080D-JULE (1MB, 133 MHz) WSON-8 5x6mm: Winbond W25Q128JV 16MB C190862 XSON-8 4x4mm: Winbond W25Q64JV 8MB C2940195"
- note removed: "BOM:"
- note removed: "Boot"
- note removed: "Crystal"
- note removed: "Crystal 12MHz, 2520 SMD package: JYJE: 2TJ412000NYGBC JGHC: S22120001210120 Yangxing Tech: X252012MMB4SI-24 Seiko Epson: Q24FA20H0068700 ECS: ECS-120-12-36-AGN-TR3"
- note removed: "Filter / VCC Cap"
- note removed: "LDO"
- note removed: "LDO 3.3V/300mA, TSOP5 package: On Semi NCP114ASN330T1G Richtek RT9078-33GJ5"
- note removed: "LED Driver"
- note removed: "Make sure these two R's are close to RP2040"
- note removed: "Make sure this C is close to pin 44 of RP2040"
- note removed: "Make sure this C is close to pin 45 of RP2040"
- note removed: "NCP114: Input Capacitor Selection (CIN) It is recommended to connect at least a 1uF Ceramic X5R or X7R capacitor as close as possible to the IN pin of the device. Output Decoupling (COUT) The NCP114 requires an output capacitor connected as close as possible to the output pin of the regulator. The recommended capacitor value is 1uF and X7R or X5R dielectric due to its low capacitance variations o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"
- note removed: "NOTE: See page 42 (application example) and 52 (configuration 3) of npm1100 datasheet See Hardware Application Guidelines for inductor choices"
- note removed: "Power"
- note removed: "Pull up / down"
- note removed: "QSPI Flash"
- note removed: "RP2040"
- note removed: "Reset"
- note removed: "Tactile switch: Alps: SKSF, SKSGACE010, side SKSCPBE010 Panasonic: EVPAL7A1AB24, EVPAF7B70, side mount EVPAVAA1A, EVPAEGE2A, EVPAEBB2A Omron: B3U-1000P, side B3U-3000P"
- note removed: "To Turn Power for Sensors MCU drives GPIO LOW. V_GS becomes -3.3V, turning the P-FET ON. Choose between AO3401A and Si2301."
- note removed: "USB TYPE C"
- moved on the sheet: C1, C11, C2, C3, C4, C5, C6, Hs1, J1, JLC1, L1, Q1A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

Commit message: D  notes/analog D  notes/bypasscaps D  notes/charging D  notes/fusion D  notes/is31fl3731 D  notes/keyfrequency D  notes/keytravel D  notes/leds D  notes/loadsw D  notes/muxadc D  notes/notes D  notes/nrf D  notes/nuts D  notes/parts D  notes/pulldown D  notes/scan D  notes/soldering D  notes/spi D  notes/swupdate D  notes/tmr M  pcb/pcb.kicad_pro M  pcb/pcb.kicad_sch M  pcb/switch.kicad_sch A  tmr-footprints/tps22997.kicad_mod M  tmr-symbols.kicad_sym
Parts:
- removed C10, C6, C7, C8, C9: 0.1uF, Capacitor_SMD:C_0402_1005Metric, symbol Device:C_Small_US
- removed C11: 10uF, Capacitor_SMD:C_0603_1608Metric, symbol Device:C_Small
- removed Q2: Si2302CDS, Package_TO_SOT_SMD:SOT-23-3, symbol tmr-lib:Si2302CDS
- removed R10: 100k, Resistor_SMD:R_0603_1608Metric, symbol Device:R_Small
- removed R8: 220R, Resistor_SMD:R_0603_1608Metric, symbol Device:R_Small
- removed R9: 10k, Resistor_SMD:R_0603_1608Metric, symbol Device:R_Small
- removed U2, U3, U4, U5, U6: ADG706BRU, Package_SO:TSSOP-28_4.4x9.7mm_P0.65mm, symbol tmr-lib:ADG706BRU
- removed U7: TPS22902, tmr-lib:Texas_DSBGA-4_0.8x0.8mm_Layout2x2_P0.4mm, symbol tmr-lib:TPS22902
- added Cbias?: 0.1uF, Capacitor_SMD:C_0603_1608Metric, symbol Device:C_Small
- added Cct?: 100pF, Capacitor_SMD:C_0603_1608Metric, symbol Device:C_Small
- added Cvin?: 10uF, Capacitor_SMD:C_0603_1608Metric, symbol Device:C_Small
- added JP?: SolderJumper_3_Bridged12, symbol Jumper:SolderJumper_3_Bridged12
- added Ron?: 100k, Resistor_SMD:R_0603_1608Metric, symbol Device:R_Small
- added Rpg?: 10k, Resistor_SMD:R_0603_1608Metric, symbol Device:R_Small
- added U?: TPS22997RYZR, tmr-lib:tps22997, symbol tmr-lib:TPS22997RYZR
Connections:
- net GND: now also Cbias?.2, Cct?.2, Cvin?.2, JP?.3 (B), Ron?.2, U?.5 (GND); no longer U1.2 (VOUTBSET1)
- net VSYS: now also U1.2 (VOUTBSET1), JP?.1 (A); no longer U1.3 (VOUTBSET0)
- net +2V1 renamed +3V0
- net +3V0: now also Cbias?.1, Cvin?.1, U?.1 (VBIAS), U?.2 (VIN), U?.3 (VIN)
- new net: Cct?.1, U?.9 (CT)
- new net: JP?.2 (C), U1.3 (VOUTBSET0)
- new net +3V0_SENSOR: Rpg?.2, U?.7 (VOUT), U?.8 (VOUT)
- new net SENSOR_PWR_EN: Ron?.1, U?.10 (ON)
- new net SENSOR_PWR_GOOD: Rpg?.1, U?.4 (PG)
- no-connect marks 1 -> 2
Other:
- removed sheet LED1
- removed sheet LED10
- removed sheet LED11
- removed sheet LED12
- removed sheet LED13
- removed sheet LED14
- removed sheet LED15
- removed sheet LED16
- removed sheet LED17
- removed sheet LED18
- removed sheet LED19
- removed sheet LED2
- removed sheet LED20
- removed sheet LED21
- removed sheet LED22
- removed sheet LED23
- removed sheet LED24
- removed sheet LED25
- removed sheet LED26
- removed sheet LED27
- removed sheet LED28
- removed sheet LED29
- removed sheet LED3
- removed sheet LED30
- removed sheet LED31
- removed sheet LED32
- removed sheet LED33
- removed sheet LED34
- removed sheet LED35
- removed sheet LED36
- removed sheet LED37
- removed sheet LED38
- removed sheet LED39
- removed sheet LED4
- removed sheet LED40
- removed sheet LED41
- removed sheet LED42
- removed sheet LED43
- removed sheet LED44
- removed sheet LED45
- removed sheet LED46
- removed sheet LED47
- removed sheet LED48
- removed sheet LED49
- removed sheet LED5
- removed sheet LED50
- removed sheet LED51
- removed sheet LED52
- removed sheet LED53
- removed sheet LED54
- removed sheet LED55
- removed sheet LED56
- removed sheet LED57
- removed sheet LED58
- removed sheet LED59
- removed sheet LED6
- removed sheet LED60
- removed sheet LED61
- removed sheet LED62
- removed sheet LED63
- removed sheet LED64
- removed sheet LED65
- removed sheet LED66
- removed sheet LED67
- removed sheet LED68
- removed sheet LED69
- removed sheet LED7
- removed sheet LED70
- removed sheet LED71
- removed sheet LED72
- removed sheet LED8
- removed sheet LED9
- note added: "NOTE: VIN must supply the inrush current needed to charge 72 x 0.1 uF TMR decoupling capacitors (7.2 uF total). For a 3 V step with a 40 us slew rate: I_inrush = C * dV/dt = 7.2 uF * (3 V / 40 us) = 540 mA This exceeds the nPM1100 buck current limit (150 mA). To mitigate this, either: * Add a reservoir capacitor for local energy storage, or * Use a load switch with a slower slew rate (>= 144 us),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"
- note removed: "Low Side N-FET Switch for PWM"
- note removed: "NOTE: Place Rgate close to MCU, and Rpull close to N-MOSFET."
- note removed: "NOTE: VIN must provide inrush current to charge 72 x 0.1 uF TMR decoupling capacitors (total 7.2 uF). For a 2.1 V step with 40 us slew: I_inrush = C * dV/dt = 7.2 uF * (2.1 V / 40 us) = 378 mA. This exceeds the nPM1100 buck current limit (150 mA), so local energy storage is required. Place a 10 uF to 22 uF X7R ceramic capacitor close to the TPS22902 VIN pin to supply the inrush current and preven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"

Commit message: M  pcb/pcb.kicad_sch A  tmr-footprints/L_Samsung_CIGT201610EH2R2MNE.kicad_mod D  tmr-footprints/Murata_DFE201210U.kicad_mod M  tmr-symbols.kicad_sym
Parts:
- added BAT?: Battery_Pack_PS5, Connector_JST:JST_EH_S3B-EH_1x03_P2.50mm_Horizontal, symbol tmr-lib:Battery_Pack_PS5
- added C? (x2): 2.2uF, Capacitor_SMD:C_0603_1608Metric, symbol Device:C_Small
- added C? (x5): 10uF, Capacitor_SMD:C_0603_1608Metric, symbol Device:C_Small
- added C?: 1uF, Capacitor_SMD:C_0603_1608Metric, symbol Device:C_Small
- added C?: 100nF, Capacitor_SMD:C_0603_1608Metric, symbol Device:C_Small
- added J?: USB_C_Receptacle_USB2.0_14P, symbol Connector:USB_C_Receptacle_USB2.0_14P
- added L? (x2): 2.2uH, tmr-lib:L_Samsung_CIGT201610EH2R2MNE, symbol Device:L_Small
- added PMIC?: nPM1300-QEXX, Package_DFN_QFN:QFN-32-1EP_5x5mm_P0.5mm_EP3.6x3.6mm_ThermalVias, symbol nordic-npm:nPM1300-QEXX
- added R? (x2): 47k, Resistor_SMD:R_0402_1005Metric, symbol Device:R
- added R? (x2): 10k, Resistor_SMD:R_0402_1005Metric, symbol Device:R_Small
- added SW?: SW_DIP_x01, symbol Switch:SW_DIP_x01
- C1: value 2.2uF -> 1uF
- L1: value 2.2uF -> 2.2uH; footprint tmr-lib:Murata_DFE201210U -> (none)
- M1: value nRF54L15 module -> Ezurio BL54L15 (nrf54L15) module
Connections:
- net GND: now also BAT?.3 (GND), C?.1, C?.2, C?.2, C?.2, C?.2, C?.2, C?.2, C?.2, C?.2, J?.A1 (GND), J?.A12 (GND), J?.B1 (GND), J?.B12 (GND), J?.S1 (SHIELD), PMIC?.2 (PVSS1), PMIC?.30 (LSIN2/VINLDO2), PMIC?.31 (LSOUT2/VOUTLDO2), PMIC?.33 (AVSS), PMIC?.6 (PVSS2), R?.1, R?.1, SW?.1
- net VSYS: now also C?.1, C?.1, C?.1, PMIC?.20 (VSYS), PMIC?.4 (PVDD)
- net at J1.A9 (VBUS), J1.B9 (VBUS), U1.17 (VBUS): no longer C1.1
- net VDDIO: now reaches M1.26 (VDD_nRF)
- net VDDIO: now also C?.1, C?.2, L?.1, PMIC?.1 (VOUT1), PMIC?.12 (VDDIO), R?.1, R?.1
- new net: PMIC?.16 (VSET2), R?.2
- new net: C?.1, PMIC?.22 (VBUSOUT)
- new net: PMIC?.17 (VSET1), R?.2
- new net: BAT?.1 (VBAT), C?.1, PMIC?.19 (VBAT)
- new net: C?.1, L?.1, PMIC?.28 (LSIN1/VINLDO1), PMIC?.32 (VOUT2)
- new net: PMIC?.15 (SHPHLD), SW?.2
- new net: L?.2, PMIC?.3 (SW1)
- new net: BAT?.2 (NTC), PMIC?.18 (NTC)
- new net: C1.1, J?.A4 (VBUS), J?.A9 (VBUS), J?.B4 (VBUS), J?.B9 (VBUS), PMIC?.21 (VBUS)
- new net: J?.A5 (CC1), PMIC?.23 (CC1)
- new net: J?.B5 (CC2), PMIC?.24 (CC2)
- new net: L?.2, PMIC?.5 (SW2)
- new net GPIOx: PMIC?.10 (GPIO3)
- new net INT: PMIC?.8 (GPIO1)
- new net LOADSW_CTRL: PMIC?.9 (GPIO2)
- new net SCL: PMIC?.14 (SCL), R?.2
- new net SDA: PMIC?.13 (SDA), R?.2
- new net VCC_tmr: C?.1, PMIC?.29 (LSOUT1/VOUTLDO1)
- no-connect marks 2 -> 11
Other:
- note added: "1.8V"
- moved on the sheet: BAT1, C1, C2, C3, C4, C5, Hs1, Hs10, Hs11, Hs12, Hs2, Hs3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
