File: pcb/pcb.kicad_sch (KiCad schematic)
At the start: 61 parts, among them J1 USB_C_Receptacle_PowerOnly_6P, J2 Conn_01x06_Socket, M1 Ezurio BL54L15 (nrf54L15) mod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, Q1 DMC2400UV, SW1 SW_DIP_x01, U1 nPM1100-QDXX

Commit message: M  pcb/pcb.kicad_pcb M  pcb/pcb.kicad_sch M  pcb/switch.kicad_sch M  placefp.py A  tmr-footprints/Texas_DYY0016A_TSOT-23-16_2x4.2mm_P0.5mm.kicad_mod M  tmr-symbols.kicad_sym
Parts:
- removed BAT1: Battery_Pack_PS5, Connector_JST:JST_EH_S3B-EH_1x03_P2.50mm_Horizontal, symbol tmr-lib:Battery_Pack_PS5
- removed C2, C4, C5, Cvin?: 10uF, Capacitor_SMD:C_0603_1608Metric, symbol Device:C_Small
- removed C3: 1uF, Capacitor_SMD:C_0603_1608Metric, symbol Device:C_Small
- removed Cbias?: 0.1uF, Capacitor_SMD:C_0603_1608Metric, symbol Device:C_Small
- removed Cct?: 100pF, Capacitor_SMD:C_0603_1608Metric, symbol Device:C_Small
- removed J1: USB_C_Receptacle_PowerOnly_6P, symbol Connector:USB_C_Receptacle_PowerOnly_6P
- removed JP?: SolderJumper_3_Bridged12, symbol Jumper:SolderJumper_3_Bridged12
- removed L1: 2.2uH, symbol Device:L_Small
- removed Q1: DMC2400UV, Package_TO_SOT_SMD:SOT-563, symbol tmr-lib:DMC2400UV
- removed R1, R5: 1M0, Resistor_SMD:R_0603_1608Metric, symbol Device:R_Small
- removed R2, R3: 5.1k, Resistor_SMD:R_0603_1608Metric, symbol Device:R
- removed R4: 1M5, Resistor_SMD:R_0603_1608Metric, symbol Device:R_Small
- removed R6: 220k, Resistor_SMD:R_0603_1608Metric, symbol Device:R_Small
- removed R7: 100k, Resistor_SMD:R_0603_1608Metric, symbol Device:R
- removed Ron?: 100k, Resistor_SMD:R_0603_1608Metric, symbol Device:R_Small
- removed Rpg?: 10k, Resistor_SMD:R_0603_1608Metric, symbol Device:R_Small
- removed U1: nPM1100-QDXX, Package_DFN_QFN:QFN-24-1EP_4x4mm_P0.5mm_EP2.6x2.6mm_ThermalVias, symbol nordic-npm:nPM1100-QDXX
- removed U?: TPS22997RYZR, tmr-lib:tps22997, symbol tmr-lib:TPS22997RYZR
- added C13, C17, C7, C8: .1uF, Capacitor_SMD:C_0402_1005Metric, symbol Device:C_Small
- added C14: 1nF, Capacitor_SMD:C_0603_1608Metric, symbol Device:C_Small
- added C15, C16, C18: 1uF, Capacitor_SMD:C_0603_1608Metric, symbol Device:C_Small
- added D1, D10, D11, D12, D13, D14, D15, D16, D17, D18, D19, D2, D20, D21, D22, D23, D24, D25, D26, D27, D28, D29, D3, D30, D31, D32, D33, D34, D35, D36, D37, D38, D39, D4, D40, D41, D42, D43, D44, D45, D46, D47, D48, D49, D5, D50, D51, D52, D53, D54, D55, D56, D57, D58, D59, D6, D60, D61, D62, D63, D64, D65, D66, D67, D68, D69, D7, D70, D71, D72, D8, D9: Green LED, tmr-lib:LED_1206_3216Metric_ReverseMount_Hole2.1mm, symbol Device:LED_Small_Filled
- added LEDDR1: LP5864, Package_DFN_QFN:VQFN-32-1EP_4x4mm_P0.4mm_EP2.8x2.8mm_ThermalVias, symbol tmr-lib:LP5864
- added MUXA1, MUXA2: TMUX1574DYY, tmr-lib:Texas_DYY0016A_TSOT-23-16_2x4.2mm_P0.5mm, symbol Analog_Switch:TMUX1574DYY
- added MUXB1: TMUX1108PW, Package_SO:TSSOP-16_4.4x5mm_P0.65mm, symbol Analog_Switch:TMUX1108PW
- added USB1: USB_C_Receptacle_PowerOnly_6P, Connector_USB:USB_C_Receptacle_GCT_USB4125-xx-x-0190_6P_TopMnt_Horizontal, symbol Connector:USB_C_Receptacle_PowerOnly_6P
- C4: renamed from C?; value 100nF -> 0.1uF; footprint Capacitor_SMD:C_0603_1608Metric -> Capacitor_SMD:C_0402_1005Metric
- L1: renamed from L?; Ex (none) -> Murata DFE201210U-2R2M Samsung CIGT201610EH2R2MNE Samsung C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
- SW1: footprint TestPoint:TestPoint_Bridge_Pitch3.81mm_Drill1.3mm -> (none)
- gave numbers to parts that had none: 17
- renumbered C1 to C6
Connections:
- net GND: now also C13.1, C14.2, C15.1, C16.2, C17.1, C17.2, C18.2, C7.1, C8.1, LEDDR1.26 (IFS), LEDDR1.27 (VSYNC), LEDDR1.30 (ADDR0_MISO), LEDDR1.31 (ADDR1_SS), LEDDR1.33 (GND), MUXA1.15 (~{EN}), MUXA1.8 (GND), MUXA2.15 (~{EN}), MUXA2.8 (GND), MUXB1.14 (GND), MUXB1.3 (VSS), USB1.A12 (GND), USB1.B12 (GND), USB1.S1 (SHIELD); no longer SW1.2
- net SCL: now also LEDDR1.28 (SCL_SCLK)
- net SDA: now also LEDDR1.29 (SDA_MOSI)
- net VSYS: now also C16.1, C18.1, LEDDR1.1 (VCC), LEDDR1.15 (VLED)
- net AIN3: now reaches M1.20 (P1.07/AIN3)
- net AIN3: now also MUXA1.12 (D4)
- net AIN2: now reaches M1.21 (P1.06/AIN2)
- net AIN2: now also MUXA1.9 (D3)
- net AIN1: now reaches M1.22 (P1.05/AIN1)
- net AIN1: now also MUXA1.7 (D2)
- net AIN0: now reaches M1.23 (P1.04/AIN0/CLK)
- net AIN0: now also MUXA1.4 (D1)
- net AIN7: now reaches M1.32 (P1.14/AIN7)
- net AIN7: now also MUXA2.12 (D4)
- net AIN6: now reaches M1.33 (P1.13/AIN6)
- net AIN6: now also MUXA2.9 (D3)
- net AIN5: now reaches M1.34 (P1.12/AIN5/CLK)
- net AIN5: now also MUXA2.7 (D2)
- net AIN4: now reaches M1.35 (P1.11/AIN4/CLK)
- net AIN4: now also MUXA2.4 (D1)
- net VCCS: now reaches C10.1, L2.1, PMIC1.28 (LSIN1/VINLDO1), PMIC1.32 (VOUT2)
- net VCCS: now also C13.2, C7.2, C8.2, MUXA1.16 (VDD), MUXA2.16 (VDD), MUXB1.13 (VDD), MUXB1.2 (EN)
- net at J1.A4 (VBUS), J1.A9 (VBUS), J1.B4 (VBUS)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: no longer C6.1, PMIC1.21 (VBUS)
- net at PMIC1.23 (CC1): now also USB1.A5 (CC1); no longer J1.A5 (CC1)
- net at PMIC1.24 (CC2): now also USB1.B5 (CC2); no longer J1.B5 (CC2)
- net GPIOx renamed GPIO_X
- new net: C6.1, PMIC1.21 (VBUS), USB1.A9 (VBUS), USB1.B9 (VBUS)
- new net: C15.2, LEDDR1.25 (VCAP)
- new net ANA_MUX_1: MUXA1.14 (S4A), MUXB1.8 (D)
- new net CS0: LEDDR1.2 (CS0)
- new net CS1: LEDDR1.3 (CS1)
- new net CS10: LEDDR1.17 (CS10)
- new net CS11: LEDDR1.18 (CS11)
- new net CS12: LEDDR1.19 (CS12)
- new net CS13: LEDDR1.20 (CS13)
- new net CS14: LEDDR1.21 (CS14)
- new net CS15: LEDDR1.22 (CS15)
- new net CS16: LEDDR1.23 (CS16)
- new net CS17: LEDDR1.24 (CS17)
- new net CS2: LEDDR1.4 (CS2)
- new net CS3: LEDDR1.5 (CS3)
- new net CS4: LEDDR1.6 (CS4)
- new net CS5: LEDDR1.7 (CS5)
- new net CS6: LEDDR1.8 (CS6)
- new net CS7: LEDDR1.9 (CS7)
- new net CS8: LEDDR1.10 (CS8)
- new net CS9: LEDDR1.16 (CS9)
- new net LED_DR_EN: C14.1, LEDDR1.32 (VIO_EN)
- new net MUX_A_SEL: MUXA1.1 (SEL), MUXA2.1 (SEL)
- new net SW0: LEDDR1.11 (SW0)
- new net SW1: LEDDR1.12 (SW1)
- new net SW2: LEDDR1.13 (SW2)
- new net SW3: LEDDR1.14 (SW3)
- no-connect marks 11 -> 9
Other:
- note added: "MCU Module"
- note removed: "Load Switch to pulse TMR sensors"
- note removed: "NOTE: See page 42 (application example) and 52 (configuration 3) of npm1100 datasheet Suggested inductors: Murata DFE201210U-2R2M Samsung CIGT201610EH2R2MNE Samsung CIGT252008LM2R2MNE Taiyo Yuden MDKK1616T2R2MM (See Hardware Application Guidelines for more inductor choices)"
- note removed: "NOTE: VIN must supply the inrush current needed to charge 72 x 0.1 uF TMR decoupling capacitors (7.2 uF total). For a 3 V step with a 40 us slew rate: I_inrush = C * dV/dt = 7.2 uF * (3 V / 40 us) = 540 mA This exceeds the nPM1100 buck current limit (150 mA). To mitigate this, either: * Add a reservoir capacitor for local energy storage, or * Use a load switch with a slower slew rate (>= 144 us),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"
- moved on the sheet: Hs1, Hs10, Hs11, Hs12, Hs2, Hs3, Hs4, Hs5, Hs6, Hs7, Hs8, Hs9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

Commit message: M  pcb/pcb.kicad_pcb M  pcb/pcb.kicad_prl M  pcb/pcb.kicad_pro M  pcb/pcb.kicad_sch M  pcb/switch.kicad_sch M  placefp.py M  tracks.py
Parts:
- added C10, C11, C16, C17, C18, C21, C22, C23, C24, C27, C28, C29, C30, C9: .1uF, Capacitor_SMD:C_0402_1005Metric, symbol Device:C_Small
- added MUXB2, MUXB3, MUXB4, MUXB5, MUXB6, MUXB7, MUXB8: TMUX1108PW, Package_SO:TSSOP-16_4.4x5mm_P0.65mm, symbol Analog_Switch:TMUX1108PW
- renumbered C9 to C12, C10 to C13, C11 to C14, C17 to C15, C12 to C19, C8 to C20, C14 to C25, C15 to C26, C16 to C31, C18 to C32, C7 to C6, C6 to C7, C13 to C8
Connections:
- net AIN4: now also M1.33 (P1.13/AIN6); no longer M1.35 (P1.11/AIN4/CLK)
- net AIN5: now also M1.32 (P1.14/AIN7); no longer M1.34 (P1.12/AIN5/CLK)
- net AIN6: now also M1.35 (P1.11/AIN4/CLK); no longer M1.33 (P1.13/AIN6)
- net AIN7: now also M1.34 (P1.12/AIN5/CLK); no longer M1.32 (P1.14/AIN7)
- net ANA_01: now also MUXB1.7 (S4)
- net ANA_02: now also MUXB1.6 (S3)
- net ANA_03: now also MUXB1.9 (S8)
- net ANA_04: now also MUXB1.10 (S7)
- net ANA_05: now also MUXB1.11 (S6)
- net ANA_06: now also MUXB1.12 (S5)
- net ANA_07: now also MUXB1.4 (S1)
- net ANA_08: now also MUXB1.5 (S2)
- net ANA_09: now also MUXA2.10 (S3B)
- net ANA_10: now also MUXB5.9 (S8)
- net ANA_11: now also MUXB5.10 (S7)
- net ANA_12: now also MUXB5.11 (S6)
- net ANA_13: now also MUXB5.12 (S5)
- net ANA_14: now also MUXB5.7 (S4)
- net ANA_15: now also MUXB5.6 (S3)
- net ANA_16: now also MUXB2.5 (S2)
- net ANA_17: now also MUXB2.9 (S8)
- net ANA_18: now also MUXB2.10 (S7)
- net ANA_19: now also MUXB2.11 (S6)
- net ANA_20: now also MUXB2.12 (S5)
- net ANA_21: now also MUXB2.4 (S1)
- net ANA_22: now also MUXA1.13 (S4B)
- net ANA_23: now also MUXA2.6 (S2B)
- net ANA_24: now also MUXA2.13 (S4B)
- net ANA_25: now also MUXB6.9 (S8)
- net ANA_26: now also MUXB6.10 (S7)
- net ANA_27: now also MUXB6.11 (S6)
- net ANA_28: now also MUXB6.12 (S5)
- net ANA_29: now also MUXB5.5 (S2)
- net ANA_30: now also MUXB2.6 (S3)
- net ANA_31: now also MUXB2.7 (S4)
- net ANA_32: now also MUXB3.9 (S8)
- net ANA_33: now also MUXB3.10 (S7)
- net ANA_34: now also MUXB3.11 (S6)
- net ANA_35: now also MUXB3.12 (S5)
- net ANA_36: now also MUXA1.6 (S2B)
- net ANA_37: now also MUXA1.10 (S3B)
- net ANA_38: now also MUXA2.3 (S1B)
- net ANA_39: now also MUXB7.4 (S1)
- net ANA_40: now also MUXB6.7 (S4)
- net ANA_41: now also MUXB6.6 (S3)
- net ANA_42: now also MUXB6.5 (S2)
- net ANA_43: now also MUXB6.4 (S1)
- net ANA_44: now also MUXB5.4 (S1)
- net ANA_45: now also MUXB3.4 (S1)
- net ANA_46: now also MUXB3.5 (S2)
- net ANA_47: now also MUXB4.9 (S8)
- net ANA_48: now also MUXB4.10 (S7)
- net ANA_49: now also MUXB4.11 (S6)
- net ANA_50: now also MUXB4.12 (S5)
- net ANA_51: now also MUXA1.3 (S1B)
- net ANA_52: now also MUXB8.4 (S1)
- net ANA_53: now also MUXB8.5 (S2)
- net ANA_54: now also MUXB8.6 (S3)
- net ANA_55: now also MUXB8.7 (S4)
- net ANA_56: now also MUXB7.12 (S5)
- net ANA_57: now also MUXB7.6 (S3)
- net ANA_58: now also MUXB7.5 (S2)
- net ANA_59: now also MUXB3.6 (S3)
- net ANA_60: now also MUXB3.7 (S4)
- net ANA_61: now also MUXB4.4 (S1)
- net ANA_62: now also MUXB4.7 (S4)
- net ANA_63: now also MUXB4.6 (S3)
- net ANA_64: now also MUXB4.5 (S2)
- net ANA_65: now also MUXB8.12 (S5)
- net ANA_66: now also MUXB8.11 (S6)
- net ANA_67: now also MUXB8.10 (S7)
- net ANA_68: now also MUXB8.9 (S8)
- net ANA_69: now also MUXB7.9 (S8)
- net ANA_70: now also MUXB7.10 (S7)
- net ANA_71: now also MUXB7.11 (S6)
- net ANA_72: now also MUXB7.7 (S4)
- net GND: now also C10.1, C11.1, C16.1, C16.2, C17.1, C17.2, C18.1, C18.2, C21.1, C22.1, C23.1, C24.1, C27.1, C27.2, C28.1, C28.2, C29.1, C29.2, C30.1, C30.2, C9.1, MUXB2.14 (GND), MUXB2.3 (VSS), MUXB3.14 (GND), MUXB3.3 (VSS), MUXB4.14 (GND), MUXB4.3 (VSS), MUXB5.14 (GND), MUXB5.3 (VSS), MUXB6.14 (GND), MUXB6.3 (VSS), MUXB7.14 (GND), MUXB7.3 (VSS), MUXB8.14 (GND), MUXB8.3 (VSS)
- net MUX_A_SEL: now also M1.24 (P1.01/XL2)
- net VCCS: now also C10.2, C11.2, C21.2, C22.2, C23.2, C24.2, C9.2, MUXB2.13 (VDD), MUXB2.2 (EN), MUXB3.13 (VDD), MUXB3.2 (EN), MUXB4.13 (VDD), MUXB4.2 (EN), MUXB5.13 (VDD), MUXB5.2 (EN), MUXB6.13 (VDD), MUXB6.2 (EN), MUXB7.13 (VDD), MUXB7.2 (EN), MUXB8.13 (VDD), MUXB8.2 (EN)
- net MUX_B_2: now reaches MUXA1.11 (S3A)
- net MUX_B_2: now also MUXB2.8 (D)
- net MUX_B_4: now reaches MUXA1.2 (S1A)
- net MUX_B_4: now also MUXB4.8 (D)
- net MUX_B_3: now reaches MUXA1.5 (S2A)
- net MUX_B_3: now also MUXB3.8 (D)
- net MUX_B_5: now reaches MUXA2.11 (S3A)
- net MUX_B_5: now also MUXB5.8 (D)
- net MUX_B_6: now reaches MUXA2.14 (S4A)
- net MUX_B_6: now also MUXB6.8 (D)
- net MUX_B_7: now reaches MUXA2.2 (S1A)
- net MUX_B_7: now also MUXB7.8 (D)
- net MUX_B_8: now reaches MUXA2.5 (S2A)
- net MUX_B_8: now also MUXB8.8 (D)
- net ANA_MUX_1 renamed MUX_B_1
Other:
- moved on the sheet: C15, C20, C6, C8, M1, MUXA1, MUXA2, MUXB1, SW1

Commit message: M  pcb/pcb.kicad_pcb M  pcb/pcb.kicad_prl M  pcb/pcb.kicad_pro M  pcb/pcb.kicad_sch M  placefp.py
Parts:
- removed SW1: SW_DIP_x01, symbol Switch:SW_DIP_x01
- renumbered SW2 to SW1
Connections:
- net AIN4: now also M1.35 (P1.11/AIN4/CLK), MUXA2.9 (D3); no longer M1.33 (P1.13/AIN6), MUXA2.4 (D1)
- net AIN5: now also M1.34 (P1.12/AIN5/CLK), MUXA2.12 (D4); no longer M1.32 (P1.14/AIN7), MUXA2.7 (D2)
- net AIN6: now also M1.33 (P1.13/AIN6), MUXA2.4 (D1); no longer M1.35 (P1.11/AIN4/CLK), MUXA2.9 (D3)
- net AIN7: now also M1.32 (P1.14/AIN7), MUXA2.7 (D2); no longer M1.34 (P1.12/AIN5/CLK), MUXA2.12 (D4)
- net ANA_30: now also MUXB2.7 (S4); no longer MUXB2.6 (S3)
- net ANA_31: now also MUXB2.6 (S3); no longer MUXB2.7 (S4)
- net ANA_45: now also MUXB3.5 (S2); no longer MUXB3.4 (S1)
- net ANA_46: now also MUXB3.4 (S1); no longer MUXB3.5 (S2)
- net ANA_57: now also MUXB7.5 (S2); no longer MUXB7.6 (S3)
- net ANA_58: now also MUXB7.6 (S3); no longer MUXB7.5 (S2)
- net CS0: now also D1.1 (K), D16.1 (K), D30.1 (K), D45.1 (K)
- net CS1: now also D17.1 (K), D2.1 (K), D31.1 (K), D46.1 (K)
- net CS10: now also D24.1 (K), D38.1 (K), D53.1 (K), D9.1 (K)
- net CS11: now also D10.1 (K), D25.1 (K), D39.1 (K), D54.1 (K)
- net CS12: now also D11.1 (K), D26.1 (K), D40.1 (K), D55.1 (K)
- net CS13: now also D12.1 (K), D27.1 (K), D41.1 (K), D56.1 (K)
- net CS14: now also D13.1 (K), D28.1 (K), D42.1 (K), D57.1 (K)
- net CS15: now also D14.1 (K), D29.1 (K), D43.1 (K), D58.1 (K)
- net CS16: now also D15.1 (K), D44.1 (K), D71.1 (K), D72.1 (K)
- net CS17: now also D67.1 (K), D68.1 (K), D69.1 (K), D70.1 (K)
- net CS2: now also D18.1 (K), D3.1 (K), D32.1 (K), D47.1 (K)
- net CS3: now also D19.1 (K), D33.1 (K), D4.1 (K), D48.1 (K)
- net CS4: now also D20.1 (K), D34.1 (K), D49.1 (K), D5.1 (K)
- net CS5: now also D21.1 (K), D35.1 (K), D50.1 (K), D6.1 (K)
- net CS6: now also D22.1 (K), D36.1 (K), D51.1 (K), D7.1 (K)
- net CS7: now also D23.1 (K), D37.1 (K), D52.1 (K), D8.1 (K)
- net CS8: now also D59.1 (K), D60.1 (K), D61.1 (K), D62.1 (K)
- net CS9: now also D63.1 (K), D64.1 (K), D65.1 (K), D66.1 (K)
- net SW0: now also D1.2 (A), D10.2 (A), D11.2 (A), D12.2 (A), D13.2 (A), D14.2 (A), D15.2 (A), D2.2 (A), D3.2 (A), D4.2 (A), D5.2 (A), D6.2 (A), D62.2 (A), D66.2 (A), D7.2 (A), D70.2 (A), D8.2 (A), D9.2 (A)
- net SW1: now also D16.2 (A), D17.2 (A), D18.2 (A), D19.2 (A), D20.2 (A), D21.2 (A), D22.2 (A), D23.2 (A), D24.2 (A), D25.2 (A), D26.2 (A), D27.2 (A), D28.2 (A), D29.2 (A), D61.2 (A), D65.2 (A), D69.2 (A), D72.2 (A)
- net SW2: now also D30.2 (A), D31.2 (A), D32.2 (A), D33.2 (A), D34.2 (A), D35.2 (A), D36.2 (A), D37.2 (A), D38.2 (A), D39.2 (A), D40.2 (A), D41.2 (A), D42.2 (A), D43.2 (A), D44.2 (A), D60.2 (A), D64.2 (A), D68.2 (A)
- net SW3: now also D45.2 (A), D46.2 (A), D47.2 (A), D48.2 (A), D49.2 (A), D50.2 (A), D51.2 (A), D52.2 (A), D53.2 (A), D54.2 (A), D55.2 (A), D56.2 (A), D57.2 (A), D58.2 (A), D59.2 (A), D63.2 (A), D67.2 (A), D71.2 (A)
- net MUXB_SEL_0: now reaches MUXB6.1 (A0)
- net MUXB_SEL_0: now also MUXB1.1 (A0), MUXB2.1 (A0), MUXB3.1 (A0), MUXB4.1 (A0), MUXB5.1 (A0), MUXB7.1 (A0), MUXB8.1 (A0)
- net MUXB_SEL_2: now reaches MUXB6.15 (A2)
- net MUXB_SEL_2: now also MUXB1.15 (A2), MUXB2.15 (A2), MUXB3.15 (A2), MUXB4.15 (A2), MUXB5.15 (A2), MUXB7.15 (A2), MUXB8.15 (A2)
- net MUXB_SEL_1: now reaches MUXB6.16 (A1)
- net MUXB_SEL_1: now also MUXB1.16 (A1), MUXB2.16 (A1), MUXB3.16 (A1), MUXB4.16 (A1), MUXB5.16 (A1), MUXB7.16 (A1), MUXB8.16 (A1)
- net MUX_A_SEL renamed MUXA_SEL
Other:
- moved on the sheet: C20, C6, D59, D60, D61, D62, D63, D64, D65, D66, D67, D68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
