File: ver1/pcb/pcb.kicad_sch (KiCad schematic)
At the start: 143 parts, among them M1 Ezurio BL54L15 (nrf54L15) mod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, SW1 SW_DIP_x01

Commit message: M  ver1/border.py M  ver1/pcb/fp-lib-table M  ver1/pcb/pcb.kicad_pcb M  ver1/pcb/pcb.kicad_pro M  ver1/pcb/pcb.kicad_sch M  ver1/placefp.py M  ver1/plate/fp-lib-table M  ver1/plate/plate.kicad_pcb M  ver1/plate/plate.kicad_sch A  ver1/tmr-footprints/Dummy.kicad_mod  M ver2/pcb/pcb.kicad_prl
Parts:
- added BAT2: ~, Connector_JST:JST_SH_SM03B-SRSS-TB_1x03-1MP_P1.00mm_Horizontal, symbol tmr-lib:Battery_Pack_PS5
Connections:
- net GND: now also BAT2.3 (GND)
- net VBAT: now reaches BAT1.1 (VBAT), C28.1, PMIC1.19 (VBAT)
- net VBAT: now also BAT2.1 (VBAT)
- no-connect marks 26 -> 27
Changed lines of the file:
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@@
 	)
 	(junction
+		(at 487.68 306.07)
+		(diameter 0)
+		(color 0 0 0 0)
+	)
+	(junction
 		(at 119.38 367.03)
 		(diameter 0)
@@
 	)
 	(junction
+		(at 499.11 313.69)
+		(diameter 0)
+		(color 0 0 0 0)
+	)
+	(junction
 		(at 52.07 355.6)
 		(diameter 0)
@@
 	)
 	(no_connect
+		(at 514.35 308.61)
+	)
+	(no_connect
 		(at 486.41 109.22)
 	)
@@
 	(wire
 		(pts
+			(xy 514.35 306.07) (xy 514.35 302.26)
+		)
+		(stroke
+			(width 0)
+			(type default)
+		)
+	)
+	(wire
+		(pts
 			(xy 185.42 304.8) (xy 185.42 307.34)
 		)
@@
 	(wire
 		(pts
-			(xy 482.6 306.07) (xy 488.95 306.07)
+			(xy 482.6 306.07) (xy 487.68 306.07)
 		)
 		(stroke
@@
 	(wire
 		(pts
+			(xy 487.68 302.26) (xy 487.68 306.07)
+		)
+		(stroke
+			(width 0)
+			(type default)
+		)
+	)
+	(wire
+		(pts
 			(xy 405.13 308.61) (xy 403.86 308.61)
 		)
@@
 		)
 	)
-	(polyline
-		(pts
-			(xy -259.08 556.26) (xy -161.29 556.26)
-		)
-		(stroke
-			(width 0.8128)
-			(type solid)
-		)
-	)
 	(wire
 		(pts
@@
 	(wire
 		(pts
+			(xy 514.35 302.26) (xy 487.68 302.26)
+		)
+		(stroke
+			(width 0)
+			(type default)
+		)
+	)
+	(wire
+		(pts
 			(xy 187.96 303.53) (xy 187.96 304.8)
 		)
@@
 	(wire
 		(pts
+			(xy 487.68 306.07) (xy 488.95 306.07)
+		)
+		(stroke
+			(width 0)
+			(type default)
+		)
+	)
+	(wire
+		(pts
 			(xy 201.93 384.81) (xy 207.01 384.81)
 		)
@@
 	(wire
 		(pts
+			(xy 499.11 313.69) (xy 524.51 313.69)
+		)
+		(stroke
+			(width 0)
+			(type default)
+		)
+	)
+	(wire
+		(pts
 			(xy 146.05 375.92) (xy 146.05 384.81)
 		)
@@
 		)
 	)
+	(label "VBAT"
+		(at 496.57 302.26 0)
+		(effects
+			(font
+				(size 1.27 1.27)
+			)
+			(justify left bottom)
+		)
+	)
 	(label "MUXB_SEL_1"
 		(at 83.82 266.7 180)
@@
 					(unit 1)
 				)
+			)
+		)
+	)
+	(symbol
+		(lib_name "Battery_Pack_PS5_1")
+		(lib_id "tmr-lib:Battery_Pack_PS5")
+		(at 523.24 307.34 0)
+		(unit 1)
+		(exclude_from_sim no)
+		(in_bom yes)
+		(on_board yes)
+		(dnp no)
+		(fields_autoplaced yes)
+		(property "Reference" "BAT2"
+			(at 529.59 307.3399 0)
+			(effects
+				(font
+					(size 1.27 1.27)
+				)
+				(justify left)
+			)
+		)
+		(property "Value" "~"
+			(at 529.59 308.6099 0)
+			(effects
+				(font
+					(size 1.27 1.27)
+				)
+				(justify left)
+				(hide yes)
+			)
+		)
+		(property "Footprint" "Connector_JST:JST_SH_SM03B-SRSS-TB_1x03-1MP_P1.00mm_Horizontal"
+			(at 502.412 332.994 0)
+			(effects
+				(font
+					(size 1.27 1.27)
+				)
+				(justify left)
+				(hide yes)
+			)
+		)
+		(property "Datasheet" ""
+			(at 527.558 330.708 0)
+			(effects
+				(font
+					(size 1.27 1.27)
+				)
+				(hide yes)
+			)
+		)
+		(property "Description" "PS5 battery pack (red->power, black->ground, white->ntc)"
+			(at 526.034 335.28 0)
+			(effects
+				(font
+					(size 1.27 1.27)
+				)
+				(hide yes)
+			)
+		)
+		(pin "3"
+		)
+		(pin "2"
+		)
+		(pin "1"
+		)
+		(instances
+			(project "pcb"
+				(path "/672ae9a0-2ac9-4023-9977-e9626ff99f32"
+					(reference "BAT2")
+					(unit 1)
+				)
