File: ver1/plate/plate.kicad_sch (KiCad schematic)
At the start: 73 parts

Commit message: M  ver1/border.py M  ver1/pcb/fp-lib-table M  ver1/pcb/pcb.kicad_pcb M  ver1/pcb/pcb.kicad_pro M  ver1/pcb/pcb.kicad_sch M  ver1/placefp.py M  ver1/plate/fp-lib-table M  ver1/plate/plate.kicad_pcb M  ver1/plate/plate.kicad_sch A  ver1/tmr-footprints/Dummy.kicad_mod  M ver2/pcb/pcb.kicad_prl
Parts:
- added BAT1, BAT2, USB1: TestPoint, tmr-lib:Dummy, symbol Connector:TestPoint
- added Hs1, Hs10, Hs11, Hs12, Hs2, Hs3, Hs4, Hs5, Hs6, Hs7, Hs8, Hs9: MountingHole, MountingHole:MountingHole_2.1mm, symbol Mechanical:MountingHole
Connections:
- no-connect marks 0 -> 3
