File: ver1/plate/plate.kicad_pcb (KiCad board)
At the start: 2 copper layers, 299.5 x 123 mm, 73 parts

Commit message: M  ver1/border.py M  ver1/pcb/fp-lib-table M  ver1/pcb/pcb.kicad_pcb M  ver1/pcb/pcb.kicad_pro M  ver1/pcb/pcb.kicad_sch M  ver1/placefp.py M  ver1/plate/fp-lib-table M  ver1/plate/plate.kicad_pcb M  ver1/plate/plate.kicad_sch A  ver1/tmr-footprints/Dummy.kicad_mod  M ver2/pcb/pcb.kicad_prl
Parts:
- added BAT1: TestPoint, tmr-lib:Dummy, F.Cu at (23.2, 80.0)
- added BAT2: TestPoint, tmr-lib:Dummy, F.Cu at (229.8, 80.0)
- added Hs1: MountingHole, MountingHole:MountingHole_2.1mm, F.Cu at (28.5, 8.93)
- added Hs10: MountingHole, MountingHole:MountingHole_2.1mm, F.Cu at (209.0, 27.9)
- added Hs11: MountingHole, MountingHole:MountingHole_2.1mm, F.Cu at (275.5, 65.9)
- added Hs12: MountingHole, MountingHole:MountingHole_2.1mm, F.Cu at (255.2, 38.0)
- added Hs2: MountingHole, MountingHole:MountingHole_2.1mm, F.Cu at (142.5, 8.93)
- added Hs3: MountingHole, MountingHole:MountingHole_2.1mm, F.Cu at (275.5, 8.93)
- added Hs4: MountingHole, MountingHole:MountingHole_2.1mm, F.Cu at (1.90, 73.0)
- added Hs5: MountingHole, MountingHole:MountingHole_2.1mm, F.Cu at (42.8, 46.9)
- added Hs6: MountingHole, MountingHole:MountingHole_2.1mm, F.Cu at (137.8, 46.9)
- added Hs7: MountingHole, MountingHole:MountingHole_2.1mm, F.Cu at (86.4, 83.6)
- added Hs8: MountingHole, MountingHole:MountingHole_2.1mm, F.Cu at (189.1, 83.6)
- added Hs9: MountingHole, MountingHole:MountingHole_2.1mm, F.Cu at (95.0, 27.9)
- added USB1: TestPoint, tmr-lib:Dummy, F.Cu at (12.6, 19.0)
Other:
- board size 299.5 x 123 mm -> 299.2 x 122.8 mm

Commit message: M  ver1/border.py M  ver1/pcb/pcb.kicad_pcb M  ver1/pcb/pcb.kicad_prl M  ver1/placefp.py A  ver1/plate/plate-Edge_Cuts.dxf M  ver1/plate/plate.kicad_pcb M  ver1/plate/plate.kicad_prl M  ver1/tmr-footprints/Dummy.kicad_mod M  ver1/tmr-footprints/Gateron_Switch_Lowpro.kicad_mod M  ver1/tmr-footprints/Switch_Cutout.kicad_mod A  ver1/tmr-footprints/USB_C_Receptacle_GCT_USB4515-xx-x_6P_MidMnt_Horizontal.kicad_mod M  ver2/pcb/pcb.kicad_prl
Parts:
- moved USB1 0.90 mm to (11.7, 19.0)
Other:
- outline, holes or cut-outs redrawn
