File: ver2/plate/plate.kicad_pcb (KiCad board)
At the start: 2 copper layers, 299.5 x 123 mm, 73 parts

Commit message: M  ver2/border.py M  ver2/pcb/dxf/pcb-Edge_Cuts.dxf D  ver2/pcb/dxf/pcb-Edge_Cuts.gbr D  ver2/pcb/dxf/pcb-job.gbrjob M  ver2/pcb/pcb.kicad_pcb M  ver2/placefp.py A  ver2/plate/dxf/plate-Edge_Cuts.dxf M  ver2/plate/fp-lib-table M  ver2/plate/plate.kicad_pcb M  ver2/plate/plate.kicad_prl M  ver2/plate/plate.kicad_sch M  ver2/plate/sym-lib-table A  ver2/tmr-footprints/MountingHole_1.6mm.kicad_mod
Parts:
- added BAT1: Battery_Pack_PS5, Connector_JST:JST_SH_SM03B-SRSS-TB_1x03-1MP_P1.00mm_Horizontal, F.Cu at (25.0, 82.2)
- added Hs1: MountingHole, tmr-lib:MountingHole_1.6mm, F.Cu at (-5.00, -3.00)
- added Hs10: MountingHole, tmr-lib:MountingHole_1.6mm, F.Cu at (228.0, 27.9)
- added Hs11: MountingHole, tmr-lib:MountingHole_1.6mm, F.Cu at (290.8, 80.0)
- added Hs2: MountingHole, tmr-lib:MountingHole_1.6mm, F.Cu at (142.5, 8.93)
- added Hs3: MountingHole, tmr-lib:MountingHole_1.6mm, F.Cu at (290.8, 8.93)
- added Hs4: MountingHole, tmr-lib:MountingHole_1.6mm, F.Cu at (-5.00, 80.0)
- added Hs5: MountingHole, tmr-lib:MountingHole_1.6mm, F.Cu at (42.8, 46.9)
- added Hs6: MountingHole, tmr-lib:MountingHole_1.6mm, F.Cu at (137.8, 46.9)
- added Hs7: MountingHole, tmr-lib:MountingHole_1.6mm, F.Cu at (86.4, 83.6)
- added Hs8: MountingHole, tmr-lib:MountingHole_1.6mm, F.Cu at (189.1, 83.6)
- added Hs9: MountingHole, tmr-lib:MountingHole_1.6mm, F.Cu at (95.0, 27.9)
- added USB1: USB_C_Receptacle_PowerOnly_6P, Connector_USB:USB_C_Receptacle_GCT_USB4125-xx-x-0190_6P_TopMnt_Horizontal, F.Cu at (-7.80, 19.0)
Other:
- board size 299.5 x 123 mm -> 305.8 x 122.8 mm

Commit message: A  bak/README.md R  ver2/RP2040_Minimal.kicad_sym -> bak/RP2040_Minimal.kicad_sym A  bak/border.py A  bak/dumploc.py A  bak/nordic-lib-kicad-npm.kicad_sym A  bak/pcb/LED.kicad_sch R  ver2/pcb/dxf/pcb-Edge_Cuts.dxf -> bak/pcb/dxf/pcb-Edge_Cuts.dxf A  bak/pcb/fp-lib-table A  bak/pcb/pcb.kicad_pcb A  bak/pcb/pcb.kicad_prl A  bak/pcb/pcb.kicad_pro A  bak/pcb/pcb.kicad_sch A  bak/pcb/switch.kicad_sch A  bak/pcb/sym-lib-table A  bak/placefp.py R  ver2/plate/dxf/plate-Edge_Cuts.dxf -> bak/plate/dxf/plate-Edge_Cuts.dxf A  bak/plate/fp-lib-table A  bak/plate/plate.kicad_pcb A  bak/plate/plate.kicad_prl A  bak/plate/plate.kicad_pro A  bak/plate/plate.kicad_sch A  bak/plate/sym-lib-table A  bak/rmtracks.py A  bak/tmr-footprints/Button_Switch_3x4x2.5.kicad_mod A  bak/tmr-footprints/C_0402_1005Metric.kicad_mod A  bak/tmr-footprints/C_0603_1608Metric.kicad_mod A  bak/tmr-footprints/DFN-3L-1.6x1.6.kicad_mod A  bak/tmr-footprints/Ezurio_BL54L15_Module.kicad_mod A  bak/tmr-footprints/Gateron_Switch_Lowpro.kicad_mod A  bak/tmr-footprints/IS31FL3731-RECESSED-SSOP-28_5.3x10.2mm_P0.65mm.kicad_mod A  bak/tmr-footprints/IS31FL3731-SSOP-28_5.3x10.2mm_P0.65mm.kicad_mod A  bak/tmr-footprints/JLC_Order_Num.kicad_mod A  bak/tmr-footprints/LED-6028.kicad_mod A  bak/tmr-footprints/LED_1206_3216Metric_ReverseMount_Hole2.1mm.kicad_mod A  bak/tmr-footprints/LED_1206_3216Metric_ReverseMount_Hole2.2x1.8mm.kicad_mod A  bak/tmr-footprints/L_Samsung_CIGT201610EH2R2MNE.kicad_mod A  bak/tmr-footprints/MCP3208-RECESSED-SOIC-16_3.9x9.9mm_P1.27mm.kicad_mod A  bak/tmr-footprints/MCP3208-SOIC-16_3.9x9.9mm_P1.27mm.kicad_mod R  ver2/tmr-footprints/MountingHole_1.6mm.kicad_mod -> bak/tmr-footprints/MountingHole_1.6mm.kicad_mod A  bak/tmr-footprints/MountingHole_2.1mm_M2_NoPad.kicad_mod A  bak/tmr-footprints/MountingHole_2.2mm_M2_NoPad.kicad_mod A  bak/tmr-footprints/MountingHole_5.3mm_M5_ISO14580_Pad_TopBottom.kicad_mod A  bak/tmr-footprints/Panasonic_EVPAE.kicad_mod A  bak/tmr-footprints/R_0402_1005Metric.kicad_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
Parts:
- added BAT2: TestPoint, tmr-lib:Dummy, F.Cu at (229.8, 80.0)
- added Hs12: MountingHole, MountingHole:MountingHole_2.1mm, F.Cu at (255.2, 38.0)
- BAT1: value Battery_Pack_PS5 -> TestPoint; footprint Connector_JST:JST_SH_SM03B-SRSS-TB_1x03-1MP_P1.00mm_Horizontal -> tmr-lib:Dummy
- Hs1, Hs10, Hs11, Hs2, Hs3, Hs4, Hs5, Hs6, Hs7, Hs8, Hs9: footprint tmr-lib:MountingHole_1.6mm -> MountingHole:MountingHole_2.1mm
- USB1: value USB_C_Receptacle_PowerOnly_6P -> TestPoint; footprint Connector_USB:USB_C_Receptacle_GCT_USB4125-xx-x-0190_6P_TopMnt_Horizontal -> tmr-lib:Dummy
- moved Hs1 35.6 mm to (28.5, 8.93)
- moved Hs11 20.7 mm to (275.5, 65.9)
- moved USB1 19.5 mm to (11.7, 19.0)
- moved Hs10 19.0 mm to (209.0, 27.9)
- moved Hs3 15.2 mm to (275.5, 8.93)
- moved Hs4 9.83 mm to (1.90, 73.0)
- moved BAT1 2.87 mm to (23.2, 80.0)
Other:
- board size 305.8 x 122.8 mm -> 299.2 x 122.8 mm
