File: ver2/plate/plate.kicad_sch (KiCad schematic)
At the start: 73 parts

Commit message: M  ver2/border.py M  ver2/pcb/dxf/pcb-Edge_Cuts.dxf D  ver2/pcb/dxf/pcb-Edge_Cuts.gbr D  ver2/pcb/dxf/pcb-job.gbrjob M  ver2/pcb/pcb.kicad_pcb M  ver2/placefp.py A  ver2/plate/dxf/plate-Edge_Cuts.dxf M  ver2/plate/fp-lib-table M  ver2/plate/plate.kicad_pcb M  ver2/plate/plate.kicad_prl M  ver2/plate/plate.kicad_sch M  ver2/plate/sym-lib-table A  ver2/tmr-footprints/MountingHole_1.6mm.kicad_mod
Parts:
- added BAT1: Battery_Pack_PS5, Connector_JST:JST_SH_SM03B-SRSS-TB_1x03-1MP_P1.00mm_Horizontal, symbol tmr-lib:Battery_Pack_PS5
- added Hs1, Hs10, Hs11, Hs2, Hs3, Hs4, Hs5, Hs6, Hs7, Hs8, Hs9: MountingHole, tmr-lib:MountingHole_1.6mm, symbol Mechanical:MountingHole
- added USB1: USB_C_Receptacle_PowerOnly_6P, Connector_USB:USB_C_Receptacle_GCT_USB4125-xx-x-0190_6P_TopMnt_Horizontal, symbol Connector:USB_C_Receptacle_PowerOnly_6P
Connections:
- new net: USB1.A12 (GND), USB1.B12 (GND)
- new net: USB1.A9 (VBUS), USB1.B9 (VBUS)

Commit message: A  bak/README.md R  ver2/RP2040_Minimal.kicad_sym -> bak/RP2040_Minimal.kicad_sym A  bak/border.py A  bak/dumploc.py A  bak/nordic-lib-kicad-npm.kicad_sym A  bak/pcb/LED.kicad_sch R  ver2/pcb/dxf/pcb-Edge_Cuts.dxf -> bak/pcb/dxf/pcb-Edge_Cuts.dxf A  bak/pcb/fp-lib-table A  bak/pcb/pcb.kicad_pcb A  bak/pcb/pcb.kicad_prl A  bak/pcb/pcb.kicad_pro A  bak/pcb/pcb.kicad_sch A  bak/pcb/switch.kicad_sch A  bak/pcb/sym-lib-table A  bak/placefp.py R  ver2/plate/dxf/plate-Edge_Cuts.dxf -> bak/plate/dxf/plate-Edge_Cuts.dxf A  bak/plate/fp-lib-table A  bak/plate/plate.kicad_pcb A  bak/plate/plate.kicad_prl A  bak/plate/plate.kicad_pro A  bak/plate/plate.kicad_sch A  bak/plate/sym-lib-table A  bak/rmtracks.py A  bak/tmr-footprints/Button_Switch_3x4x2.5.kicad_mod A  bak/tmr-footprints/C_0402_1005Metric.kicad_mod A  bak/tmr-footprints/C_0603_1608Metric.kicad_mod A  bak/tmr-footprints/DFN-3L-1.6x1.6.kicad_mod A  bak/tmr-footprints/Ezurio_BL54L15_Module.kicad_mod A  bak/tmr-footprints/Gateron_Switch_Lowpro.kicad_mod A  bak/tmr-footprints/IS31FL3731-RECESSED-SSOP-28_5.3x10.2mm_P0.65mm.kicad_mod A  bak/tmr-footprints/IS31FL3731-SSOP-28_5.3x10.2mm_P0.65mm.kicad_mod A  bak/tmr-footprints/JLC_Order_Num.kicad_mod A  bak/tmr-footprints/LED-6028.kicad_mod A  bak/tmr-footprints/LED_1206_3216Metric_ReverseMount_Hole2.1mm.kicad_mod A  bak/tmr-footprints/LED_1206_3216Metric_ReverseMount_Hole2.2x1.8mm.kicad_mod A  bak/tmr-footprints/L_Samsung_CIGT201610EH2R2MNE.kicad_mod A  bak/tmr-footprints/MCP3208-RECESSED-SOIC-16_3.9x9.9mm_P1.27mm.kicad_mod A  bak/tmr-footprints/MCP3208-SOIC-16_3.9x9.9mm_P1.27mm.kicad_mod R  ver2/tmr-footprints/MountingHole_1.6mm.kicad_mod -> bak/tmr-footprints/MountingHole_1.6mm.kicad_mod A  bak/tmr-footprints/MountingHole_2.1mm_M2_NoPad.kicad_mod A  bak/tmr-footprints/MountingHole_2.2mm_M2_NoPad.kicad_mod A  bak/tmr-footprints/MountingHole_5.3mm_M5_ISO14580_Pad_TopBottom.kicad_mod A  bak/tmr-footprints/Panasonic_EVPAE.kicad_mod A  bak/tmr-footprints/R_0402_1005Metric.kicad_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
Parts:
- removed BAT1: Battery_Pack_PS5, Connector_JST:JST_SH_SM03B-SRSS-TB_1x03-1MP_P1.00mm_Horizontal, symbol tmr-lib:Battery_Pack_PS5
- removed USB1: USB_C_Receptacle_PowerOnly_6P, Connector_USB:USB_C_Receptacle_GCT_USB4125-xx-x-0190_6P_TopMnt_Horizontal, symbol Connector:USB_C_Receptacle_PowerOnly_6P
- added BAT1, BAT2, USB1: TestPoint, tmr-lib:Dummy, symbol Connector:TestPoint
- added Hs12: MountingHole, MountingHole:MountingHole_2.1mm, symbol Mechanical:MountingHole
- Hs1, Hs10, Hs11, Hs2, Hs3, Hs4, Hs5, Hs6, Hs7, Hs8, Hs9: footprint tmr-lib:MountingHole_1.6mm -> MountingHole:MountingHole_2.1mm
Connections:
- no-connect marks 0 -> 3
