File: ver3/pcb/pcb.kicad_sch (KiCad schematic)
At the start: 151 parts, among them SW1 SW_DIP_x01, Y1 32.768 kHz

Commit message: M  ver3/border.py M  ver3/pcb/pcb.kicad_pcb M  ver3/pcb/pcb.kicad_sch M  ver3/placefp.py M  ver3/tmr-footprints/Gateron_Switch_Lowpro.kicad_mod A  ver3/tmr-footprints/Gateron_Switch_Lowpro_2.kicad_mod A  ver3/tmr-footprints/MountingHole_2.2mm_M2_ISO7380_Pad_TopBottom.kicad_mod
Parts:
- Hs1, Hs10, Hs11, Hs12, Hs2, Hs3, Hs4, Hs5, Hs6, Hs7, Hs8, Hs9: footprint MountingHole:MountingHole_2.2mm_M2_ISO7380_Pad_TopBottom -> tmr-lib:MountingHole_2.2mm_M2_ISO7380_Pad_TopBottom
Changed lines of the file:
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@@
 			)
 		)
-		(property "Footprint" "MountingHole:MountingHole_2.2mm_M2_ISO7380_Pad_TopBottom"
+		(property "Footprint" "tmr-lib:MountingHole_2.2mm_M2_ISO7380_Pad_TopBottom"
 			(at 359.41 364.49 0)
 			(effects
@@
 			)
 		)
-		(property "Footprint" "MountingHole:MountingHole_2.2mm_M2_ISO7380_Pad_TopBottom"
+		(property "Footprint" "tmr-lib:MountingHole_2.2mm_M2_ISO7380_Pad_TopBottom"
 			(at 359.41 372.11 0)
 			(effects
@@
 			)
 		)
-		(property "Footprint" "MountingHole:MountingHole_2.2mm_M2_ISO7380_Pad_TopBottom"
+		(property "Footprint" "tmr-lib:MountingHole_2.2mm_M2_ISO7380_Pad_TopBottom"
 			(at 384.81 364.49 0)
 			(effects
@@
 			)
 		)
-		(property "Footprint" "MountingHole:MountingHole_2.2mm_M2_ISO7380_Pad_TopBottom"
+		(property "Footprint" "tmr-lib:MountingHole_2.2mm_M2_ISO7380_Pad_TopBottom"
 			(at 372.11 364.49 0)
 			(effects
@@
 			)
 		)
-		(property "Footprint" "MountingHole:MountingHole_2.2mm_M2_ISO7380_Pad_TopBottom"
+		(property "Footprint" "tmr-lib:MountingHole_2.2mm_M2_ISO7380_Pad_TopBottom"
 			(at 397.51 372.11 0)
 			(effects
@@
 			)
 		)
-		(property "Footprint" "MountingHole:MountingHole_2.2mm_M2_ISO7380_Pad_TopBottom"
+		(property "Footprint" "tmr-lib:MountingHole_2.2mm_M2_ISO7380_Pad_TopBottom"
 			(at 372.11 372.11 0)
 			(effects
@@
 			)
 		)
-		(property "Footprint" "MountingHole:MountingHole_2.2mm_M2_ISO7380_Pad_TopBottom"
+		(property "Footprint" "tmr-lib:MountingHole_2.2mm_M2_ISO7380_Pad_TopBottom"
 			(at 359.41 379.73 0)
 			(effects
@@
 			)
 		)
-		(property "Footprint" "MountingHole:MountingHole_2.2mm_M2_ISO7380_Pad_TopBottom"
+		(property "Footprint" "tmr-lib:MountingHole_2.2mm_M2_ISO7380_Pad_TopBottom"
 			(at 397.51 379.73 0)
 			(effects
@@
 			)
 		)
-		(property "Footprint" "MountingHole:MountingHole_2.2mm_M2_ISO7380_Pad_TopBottom"
+		(property "Footprint" "tmr-lib:MountingHole_2.2mm_M2_ISO7380_Pad_TopBottom"
 			(at 384.81 372.11 0)
 			(effects
@@
 			)
 		)
-		(property "Footprint" "MountingHole:MountingHole_2.2mm_M2_ISO7380_Pad_TopBottom"
+		(property "Footprint" "tmr-lib:MountingHole_2.2mm_M2_ISO7380_Pad_TopBottom"
 			(at 372.11 379.73 0)
 			(effects
@@
 			)
 		)
-		(property "Footprint" "MountingHole:MountingHole_2.2mm_M2_ISO7380_Pad_TopBottom"
+		(property "Footprint" "tmr-lib:MountingHole_2.2mm_M2_ISO7380_Pad_TopBottom"
 			(at 384.81 379.73 0)
 			(effects
@@
 			)
 		)
-		(property "Footprint" "MountingHole:MountingHole_2.2mm_M2_ISO7380_Pad_TopBottom"
+		(property "Footprint" "tmr-lib:MountingHole_2.2mm_M2_ISO7380_Pad_TopBottom"
 			(at 397.51 364.49 0)
 			(effects
