File: hardware/nRF52840_v1/plate/plate.kicad_pcb (KiCad board)
At the start: 2 copper layers, 299.2 x 122.8 mm, 88 parts

Commit message: M  hardware/nRF52840_v1/border.py M  hardware/nRF52840_v1/pcb/pcb.kicad_pcb M  hardware/nRF52840_v1/placefp.py D  hardware/nRF52840_v1/plate/plate-Edge_Cuts.dxf M  hardware/nRF52840_v1/plate/plate.kicad_pcb M  hardware/nRF52840_v1/plate/plate.kicad_pro M  hardware/nRF52840_v1/plate/plate.kicad_sch
Parts:
- moved Jusb1 31.0 mm to (15.6, -11.8), turned to 180 degrees
- renumbered USB1 to Jusb1
Other:
- outline, holes or cut-outs redrawn
