File: hardware/nRF52840_v1/plate/plate.kicad_sch (KiCad schematic)
At the start: 88 parts

Commit message: M  hardware/nRF52840_v1/border.py M  hardware/nRF52840_v1/pcb/pcb.kicad_pcb M  hardware/nRF52840_v1/placefp.py D  hardware/nRF52840_v1/plate/plate-Edge_Cuts.dxf M  hardware/nRF52840_v1/plate/plate.kicad_pcb M  hardware/nRF52840_v1/plate/plate.kicad_pro M  hardware/nRF52840_v1/plate/plate.kicad_sch
Parts:
- renumbered USB1 to Jusb1
Changed lines of the file:
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@@
 		(dnp no)
 		(fields_autoplaced yes)
-		(property "Reference" "USB1"
+		(property "Reference" "Jusb1"
 			(at 41.91 108.4579 0)
 			(effects
@@
 			(project ""
 				(path "/4c67809e-1748-4898-89f6-ff92314048f2"
-					(reference "USB1")
+					(reference "Jusb1")
 					(unit 1)
 				)
