File: hardware/nRF52840_v2/plate/plate.kicad_pcb (KiCad board)
At the start: 2 copper layers, 299.2 x 122.8 mm, 88 parts

Commit message: M  hardware/nRF52840_v1/placefp.py M  hardware/nRF52840_v2/placefp.py M  hardware/nRF52840_v2/plate/plate.kicad_pcb M  hardware/nRF52840_v2/plate/plate.kicad_prl M  hardware/nRF52840_v2/plate/plate.kicad_sch A  hardware/nRF52840_v3/README.md A  hardware/nRF52840_v3/border.py A  hardware/nRF52840_v3/dumploc.py A  hardware/nRF52840_v3/nordic-lib-kicad-npm.kicad_sym A  hardware/nRF52840_v3/pcb/LED.kicad_sch A  hardware/nRF52840_v3/pcb/fp-lib-table A  hardware/nRF52840_v3/pcb/pcb-eagle-import.kicad_sym A  hardware/nRF52840_v3/pcb/pcb.kicad_pcb A  hardware/nRF52840_v3/pcb/pcb.kicad_prl A  hardware/nRF52840_v3/pcb/pcb.kicad_pro A  hardware/nRF52840_v3/pcb/pcb.kicad_sch A  hardware/nRF52840_v3/pcb/switch.kicad_sch A  hardware/nRF52840_v3/pcb/sym-lib-table A  hardware/nRF52840_v3/placefp.py A  hardware/nRF52840_v3/plate/fp-lib-table A  hardware/nRF52840_v3/plate/plate.kicad_pcb A  hardware/nRF52840_v3/plate/plate.kicad_prl A  hardware/nRF52840_v3/plate/plate.kicad_pro A  hardware/nRF52840_v3/plate/plate.kicad_sch A  hardware/nRF52840_v3/plate/sym-lib-table A  hardware/nRF52840_v3/rmtracks.py A  hardware/nRF52840_v3/tmr-footprints/Aliexpress_SW_DIP_3.6x7.3mm.kicad_mod A  hardware/nRF52840_v3/tmr-footprints/Aliexpress_SW_DIP_TS_1136W_3x6x5mm.kicad_mod A  hardware/nRF52840_v3/tmr-footprints/Aliexpress_SW_DIP_TS_1292V_4x6.2x1.8mm.kicad_mod A  hardware/nRF52840_v3/tmr-footprints/Button_Switch_3x4x2.5.kicad_mod A  hardware/nRF52840_v3/tmr-footprints/C_0402_1005Metric.kicad_mod A  hardware/nRF52840_v3/tmr-footprints/C_0603_1608Metric.kicad_mod A  hardware/nRF52840_v3/tmr-footprints/DFN-3L-1.6x1.6.kicad_mod A  hardware/nRF52840_v3/tmr-footprints/Dummy.kicad_mod A  hardware/nRF52840_v3/tmr-footprints/Ezurio_BL54L15_Module.kicad_mod A  hardware/nRF52840_v3/tmr-footprints/GCT_USB4215-03-A_REVA.kicad_mod A  hardware/nRF52840_v3/tmr-footprints/Gateron_Switch_Lowpro.kicad_mod A  hardware/nRF52840_v3/tmr-footprints/IS31FL3731-RECESSED-SSOP-28_5.3x10.2mm_P0.65mm.kicad_mod A  hardware/nRF52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
Parts:
- moved S62 0.75 mm to (78.4, 79.5), turned to 0 degrees
- renumbered USB1 to Jusb1
Changed lines of the file:
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@@
 			)
 		)
-		(property "Datasheet" ""
+		(property "Datasheet" "~"
 			(at 0 0 0)
 			(unlocked yes)
@@
 			)
 		)
-		(property "Description" ""
+		(property "Description" "test point"
 			(at 0 0 0)
 			(unlocked yes)
@@
 	(footprint "tmr-lib:Switch_Cutout"
 		(layer "F.Cu")
-		(at 77.625 79.5 -20)
+		(at 78.375 79.5)
 		(descr "Cherry MX keyswitch PCB Mount with 1.00u keycap")
 		(tags "Cherry MX Keyboard Keyswitch Switch PCB Cutout 1.00u")
 		(property "Reference" "S62"
-			(at 0.1 -6.1 340)
+			(at 0.1 -6.1 0)
 			(layer "F.SilkS")
 			(hide yes)
@@
 		)
 		(property "Value" "SWHole"
-			(at 0.1 8.5 340)
+			(at 0.1 8.5 0)
 			(layer "F.Fab")
 			(effects
@@
 		)
 		(property "Datasheet" ""
-			(at 0 0 340)
+			(at 0 0 0)
 			(layer "F.Fab")
 			(hide yes)
@@
 		)
 		(property "Description" ""
-			(at 0 0 340)
+			(at 0 0 0)
 			(layer "F.Fab")
 			(hide yes)
@@
 		(attr through_hole)
 		(fp_line
-			(start -6.6 7)
-			(end 6.6 7)
-			(stroke
-				(width 0.12)
-				(type solid)
-			)
-			(layer "Edge.Cuts")
-		)
-		(fp_line
 			(start -7 -6.6)
 			(end -7 6.6)
@@
 		)
 		(fp_line
-			(start 7 -6.6)
-			(end 7 6.6)
+			(start -6.6 7)
+			(end 6.6 7)
 			(stroke
 				(width 0.12)
@@
 			(layer "Edge.Cuts")
 		)
-		(fp_arc
-			(start -6.6 7)
-			(mid -6.882843 6.882843)
-			(end -7 6.6)
+		(fp_line
+			(start 7 -6.6)
+			(end 7 6.6)
 			(stroke
 				(width 0.12)
@@
 		)
 		(fp_arc
-			(start 7 6.6)
-			(mid 6.882843 6.882843)
-			(end 6.6 7)
+			(start -6.6 7)
+			(mid -6.882843 6.882843)
+			(end -7 6.6)
 			(stroke
 				(width 0.12)
@@
 			(layer "Edge.Cuts")
 		)
+		(fp_arc
+			(start 7 6.6)
+			(mid 6.882843 6.882843)
+			(end 6.6 7)
+			(stroke
+				(width 0.12)
+				(type solid)
+			)
+			(layer "Edge.Cuts")
+		)
 		(fp_poly
 			(pts
@@
 		)
 		(fp_text user "${REFERENCE}"
-			(at 0 -8.199999 340)
+			(at 0 -8.199999 0)
 			(layer "F.Fab")
 			(effects
@@
 		(layer "F.Cu")
 		(at 11.7 19 -90)
-		(property "Reference" "USB1"
+		(property "Reference" "Jusb1"
 			(at 0 -0.5 270)
 			(unlocked yes)
@@
 			)
 		)
-		(property "Datasheet" ""
+		(property "Datasheet" "~"
 			(at 0 0 270)
 			(unlocked yes)
@@
 			)
 		)
-		(property "Description" ""
+		(property "Description" "test point"
 			(at 0 0 270)
 			(unlocked yes)
@@
 			)
 		)
-		(property "Datasheet" ""
+		(property "Datasheet" "~"
 			(at 0 0 0)
 			(unlocked yes)
@@
 			)
 		)
-		(property "Description" ""
+		(property "Description" "test point"
 			(at 0 0 0)
 			(unlocked yes)

Commit message: M  hardware/nRF52840_v2/plate/plate.kicad_pcb M  hardware/nRF52840_v2/plate/plate.kicad_prl M  hardware/nRF52840_v2/plate/plate.kicad_pro A  hardware/nRF52840_v2/tmr-footprints/MountingHole_1.8mm_M1.6_NoPad.kicad_mod A  hardware/nRF52840_v2/tmr-footprints/MountingHole_2.2mm_M2.kicad_mod A  hardware/nRF52840_v2/tmr-footprints/SMTSO_M2.kicad_mod M  hardware/nRF52840_v3/border.py M  hardware/nRF52840_v3/pcb/pcb.kicad_pcb M  hardware/nRF52840_v3/pcb/pcb.kicad_prl M  hardware/nRF52840_v3/pcb/pcb.kicad_sch M  hardware/nRF52840_v3/placefp.py R  hardware/nRF52840_v2/plate/plate-Edge_Cuts.dxf -> hardware/nRF52840_v3/plate/plate-Edge_Cuts.dxf M  hardware/nRF52840_v3/plate/plate.kicad_pcb M  hardware/nRF52840_v3/plate/plate.kicad_prl M  hardware/nRF52840_v3/plate/plate.kicad_pro M  hardware/nRF52840_v3/plate/plate.kicad_sch A  hardware/nRF52840_v3/tmr-footprints/Aliexpress_SW_TACT_4x4x1.5mm.kicad_mod A  hardware/nRF52840_v3/tmr-footprints/MountingHole_1.8mm_M1.6_NoPad.kicad_mod A  hardware/nRF52840_v3/tmr-footprints/SMTSO_M2.kicad_mod M  hardware/nRF52840_v3/tmr-footprints/Stabilizer_Lowpro_2U.kicad_mod A  hardware/nRF52840_v3/tmr-footprints/USB_C_Receptacle_GCT_USB4085.kicad_mod
Parts:
- moved Jusb1 31.0 mm to (15.6, -11.8), turned to 180 degrees
- moved S62 0.75 mm to (77.6, 79.5), turned to -20 degrees
Other:
- outline, holes or cut-outs redrawn
