File: hardware/nRF52840_v3/plate/plate.kicad_pcb (KiCad board)
At the start: 2 copper layers, 299.2 x 122.8 mm, 88 parts

Commit message: M  hardware/nRF52840_v2/plate/plate.kicad_pcb M  hardware/nRF52840_v2/plate/plate.kicad_prl M  hardware/nRF52840_v2/plate/plate.kicad_pro A  hardware/nRF52840_v2/tmr-footprints/MountingHole_1.8mm_M1.6_NoPad.kicad_mod A  hardware/nRF52840_v2/tmr-footprints/MountingHole_2.2mm_M2.kicad_mod A  hardware/nRF52840_v2/tmr-footprints/SMTSO_M2.kicad_mod M  hardware/nRF52840_v3/border.py M  hardware/nRF52840_v3/pcb/pcb.kicad_pcb M  hardware/nRF52840_v3/pcb/pcb.kicad_prl M  hardware/nRF52840_v3/pcb/pcb.kicad_sch M  hardware/nRF52840_v3/placefp.py R  hardware/nRF52840_v2/plate/plate-Edge_Cuts.dxf -> hardware/nRF52840_v3/plate/plate-Edge_Cuts.dxf M  hardware/nRF52840_v3/plate/plate.kicad_pcb M  hardware/nRF52840_v3/plate/plate.kicad_prl M  hardware/nRF52840_v3/plate/plate.kicad_pro M  hardware/nRF52840_v3/plate/plate.kicad_sch A  hardware/nRF52840_v3/tmr-footprints/Aliexpress_SW_TACT_4x4x1.5mm.kicad_mod A  hardware/nRF52840_v3/tmr-footprints/MountingHole_1.8mm_M1.6_NoPad.kicad_mod A  hardware/nRF52840_v3/tmr-footprints/SMTSO_M2.kicad_mod M  hardware/nRF52840_v3/tmr-footprints/Stabilizer_Lowpro_2U.kicad_mod A  hardware/nRF52840_v3/tmr-footprints/USB_C_Receptacle_GCT_USB4085.kicad_mod
Parts:
- removed Hs11, Hs12: MountingHole, MountingHole:MountingHole_2.1mm
- Hs1, Hs10, Hs2, Hs3, Hs4, Hs5, Hs6, Hs7, Hs8, Hs9: footprint MountingHole:MountingHole_2.1mm -> tmr-lib:MountingHole_1.8mm_M1.6_NoPad
- S57: footprint tmr-lib:Switch_Cutout_1.75u -> tmr-lib:Switch_Cutout
- S70: footprint tmr-lib:Switch_Cutout_1.25u -> tmr-lib:Switch_Cutout
- moved Hs9 114.0 mm to (209.0, 27.9)
- moved Hs8 109.4 mm to (95.0, 27.9)
- moved Hs7 102.8 mm to (189.1, 83.6)
- moved Hs5 95.0 mm to (137.8, 46.9)
- moved Hs10 69.8 mm to (268.4, 64.6)
- moved Hs6 63.1 mm to (86.4, 83.6)
- moved Hs4 17.1 mm to (19.0, 74.0)
- moved S58 4.75 mm to (280.2, 57.0)
- moved S69 4.15 mm to (223.2, 76.0)
- moved S59 4.15 mm to (7.12, 76.0)
- moved S60 4.15 mm to (30.9, 76.0)
- moved S61 4.15 mm to (52.2, 76.0)
- moved S57 2.38 mm to (256.5, 57.0)
- moved S70 1.78 mm to (242.2, 76.0)
- moved Jusb1 1.66 mm to (15.8, -13.4)
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Other:
- board size 299.2 x 122.8 mm -> 315.2 x 194.5 mm
