File: hardware/nRF52840_bakelite_cnc/pcb/pcb.kicad_sch (KiCad schematic)
At the start: 149 parts, among them SW1 SW_DIP_x01, SW2 SW_DIP_x01, Y1 32.768 kHz

Commit message: M  hardware/nRF52840_bakelite_cnc/border.py M  hardware/nRF52840_bakelite_cnc/pcb/pcb.kicad_pcb M  hardware/nRF52840_bakelite_cnc/pcb/pcb.kicad_prl M  hardware/nRF52840_bakelite_cnc/pcb/pcb.kicad_sch A  hardware/nRF52840_bakelite_cnc/tmr-footprints/Molex_Pico_Lock_CONN_5037630000-SD_02.kicad_mod A  hardware/nRF52840_bakelite_cnc/tmr-footprints/Molex_Pico_Lock_CONN_5037630000-SD_04.kicad_mod M  hardware/nRF52840_bakelite_cnc/tmr-symbols.kicad_sym
Parts:
- BAT1: footprint Connector_JST:JST_SH_SM03B-SRSS-TB_1x03-1MP_P1.00mm_Horizontal -> tmr-lib:Molex_Pico_Lock_CONN_5037630000-SD_04
- BAT2: footprint Connector_JST:JST_SH_SM03B-SRSS-TB_1x03-1MP_P1.00mm_Horizontal -> tmr-lib:Molex_Pico_Lock_CONN_5037630000-SD_02
Connections:
- net GND: now also BAT2.2 (GND); no longer BAT2.3 (GND)
Changed lines of the file:
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@@
 	)
 	(junction
-		(at 501.65 313.69)
-		(diameter 0)
-		(color 0 0 0 0)
-	)
-	(junction
 		(at 105.41 373.38)
 		(diameter 0)
@@
 	)
 	(junction
+		(at 499.11 316.23)
+		(diameter 0)
+		(color 0 0 0 0)
+	)
+	(junction
 		(at 137.16 375.92)
 		(diameter 0)
@@
 	)
 	(junction
+		(at 524.51 313.69)
+		(diameter 0)
+		(color 0 0 0 0)
+	)
+	(junction
 		(at 154.94 375.92)
 		(diameter 0)
@@
 	)
 	(junction
-		(at 524.51 313.69)
-		(diameter 0)
-		(color 0 0 0 0)
-	)
-	(junction
 		(at 215.9 344.17)
 		(diameter 0)
@@
 	)
 	(no_connect
-		(at 514.35 308.61)
-	)
-	(no_connect
 		(at 359.41 152.4)
 	)
@@
 	)
 	(no_connect
+		(at 496.57 313.69)
+	)
+	(no_connect
 		(at 405.13 267.97)
 	)
@@
 	(wire
 		(pts
+			(xy 524.51 316.23) (xy 499.11 316.23)
+		)
+		(stroke
+			(width 0)
+			(type default)
+		)
+	)
+	(wire
+		(pts
 			(xy 356.87 152.4) (xy 356.87 158.75)
 		)
@@
 	(wire
 		(pts
-			(xy 524.51 313.69) (xy 527.05 313.69)
-		)
-		(stroke
-			(width 0)
-			(type default)
-		)
-	)
-	(wire
-		(pts
 			(xy 34.29 389.89) (xy 34.29 396.24)
 		)
@@
 	(wire
 		(pts
-			(xy 501.65 313.69) (xy 524.51 313.69)
-		)
-		(stroke
-			(width 0)
-			(type default)
-		)
-	)
-	(wire
-		(pts
 			(xy 374.65 287.02) (xy 374.65 290.83)
 		)
@@
 	(wire
 		(pts
+			(xy 524.51 313.69) (xy 527.05 313.69)
+		)
+		(stroke
+			(width 0)
+			(type default)
+		)
+	)
+	(wire
+		(pts
 			(xy 87.63 373.38) (xy 87.63 375.92)
 		)
@@
 	(wire
 		(pts
+			(xy 524.51 313.69) (xy 524.51 316.23)
+		)
+		(stroke
+			(width 0)
+			(type default)
+		)
+	)
+	(wire
+		(pts
 			(xy 289.56 246.38) (xy 298.45 246.38)
 		)
@@
 	)
 	(symbol
-		(lib_name "Battery_Pack_PS5_1")
-		(lib_id "tmr-lib:Battery_Pack_PS5")
-		(at 523.24 307.34 0)
-		(unit 1)
-		(exclude_from_sim no)
-		(in_bom yes)
-		(on_board yes)
-		(dnp no)
-		(fields_autoplaced yes)
-		(property "Reference" "BAT2"
-			(at 529.59 307.3399 0)
-			(effects
-				(font
-					(size 1.27 1.27)
-				)
-				(justify left)
-			)
-		)
-		(property "Value" "~"
-			(at 529.59 308.6099 0)
-			(effects
-				(font
-					(size 1.27 1.27)
-				)
-				(justify left)
-				(hide yes)
-			)
-		)
-		(property "Footprint" "Connector_JST:JST_SH_SM03B-SRSS-TB_1x03-1MP_P1.00mm_Horizontal"
-			(at 502.412 332.994 0)
-			(effects
-				(font
-					(size 1.27 1.27)
-				)
-				(justify left)
-				(hide yes)
-			)
-		)
-		(property "Datasheet" ""
-			(at 527.558 330.708 0)
-			(effects
-				(font
-					(size 1.27 1.27)
-				)
-				(hide yes)
-			)
-		)
-		(property "Description" "PS5 battery pack (red->power, black->ground, white->ntc)"
-			(at 526.034 335.28 0)
-			(effects
-				(font
-					(size 1.27 1.27)
-				)
-				(hide yes)
-			)
-		)
-		(pin "3"
-		)
-		(pin "2"
-		)
-		(pin "1"
-		)
-		(pin "MP"
-		)
-		(instances
-			(project "pcb"
-				(path "/672ae9a0-2ac9-4023-9977-e9626ff99f32"
-					(reference "BAT2")
-					(unit 1)
-				)
-			)
-		)
-	)
-	(symbol
 		(lib_id "power:GND")
 		(at 33.02 299.72 0)
@@
 	)
 	(symbol
+		(lib_name "Battery_Pack_PS5_1")
+		(lib_id "tmr-lib:Battery_Pack_PS5")
+		(at 523.24 307.34 0)
+		(unit 1)
+		(exclude_from_sim no)
+		(in_bom yes)
+		(on_board yes)
+		(dnp no)
+		(fields_autoplaced yes)
+		(property "Reference" "BAT2"
+			(at 529.59 307.3399 0)
+			(effects
+				(font
+					(size 1.27 1.27)
+				)
+				(justify left)
+			)
+		)
+		(property "Value" "~"
+			(at 529.59 308.6099 0)
+			(effects
+				(font
+					(size 1.27 1.27)
+				)
+				(justify left)
+				(hide yes)
+			)
+		)
+		(property "Footprint" "tmr-lib:Molex_Pico_Lock_CONN_5037630000-SD_02"
+			(at 502.412 332.994 0)
+			(effects
+				(font
+					(size 1.27 1.27)
+				)
+				(justify left)
+				(hide yes)
+			)
+		)
+		(property "Datasheet" ""
+			(at 527.558 330.708 0)
+			(effects
+				(font
+					(size 1.27 1.27)
+				)
+				(hide yes)
+			)
+		)
+		(property "Description" "PS5 battery pack (red->power, black->ground, white->ntc)"
+			(at 526.034 335.28 0)
+			(effects
+				(font
+					(size 1.27 1.27)
+				)
+				(hide yes)
+			)
+		)
+		(pin "2"
+		)
+		(pin "1"
+		)
+		(pin "MP"
+		)
+		(instances
+			(project "pcb"
+				(path "/672ae9a0-2ac9-4023-9977-e9626ff99f32"
+					(reference "BAT2")
+					(unit 1)
+				)
+			)
+		)
+	)
+	(symbol
 		(lib_id "Device:LED_Small_Filled")
 		(at 36.83 349.25 180)
@@
 			)
 		)
-		(property "Footprint" "Connector_JST:JST_SH_SM03B-SRSS-TB_1x03-1MP_P1.00mm_Horizontal"
+		(property "Footprint" "tmr-lib:Molex_Pico_Lock_CONN_5037630000-SD_04"
 			(at 477.012 332.994 0)
 			(effects
@@
 		(pin "MP"
 		)
+		(pin "4"
+		)
 		(instances

Commit message: M  hardware/nRF52840_bakelite_cnc/border.py M  hardware/nRF52840_bakelite_cnc/pcb/pcb.kicad_pcb M  hardware/nRF52840_bakelite_cnc/pcb/pcb.kicad_prl M  hardware/nRF52840_bakelite_cnc/pcb/pcb.kicad_pro M  hardware/nRF52840_bakelite_cnc/pcb/pcb.kicad_sch M  hardware/nRF52840_bakelite_cnc/pcb/switch.kicad_sch M  hardware/nRF52840_bakelite_cnc/placefp.py M  hardware/nRF52840_bakelite_cnc/plate/plate.kicad_pcb M  hardware/nRF52840_bakelite_cnc/plate/plate.kicad_sch A  hardware/nRF52840_bakelite_cnc/tmr-footprints/C_0402_1005Metric_Cvcc.kicad_mod A  hardware/nRF52840_bakelite_cnc/tmr-footprints/C_0402_1005Metric_Cvout.kicad_mod M  hardware/nRF52840_bakelite_cnc/tmr-footprints/Gateron_Switch_Lowpro.kicad_mod A  hardware/nRF52840_bakelite_cnc/tmr-footprints/PCB_Wire_Solder_3p_Connector.kicad_mod
Parts:
- BAT1: footprint tmr-lib:Molex_Pico_Lock_CONN_5037630000-SD_04 -> tmr-lib:PCB_Wire_Solder_3p_Connector
- BAT2: footprint tmr-lib:Molex_Pico_Lock_CONN_5037630000-SD_02 -> tmr-lib:PCB_Wire_Solder_3p_Connector
Connections:
- net ANA_57: now also MUXB7.6 (S3); no longer MUXB7.5 (S2)
- net ANA_58: now also MUXB7.7 (S4); no longer MUXB7.6 (S3)
- net ANA_72: now also MUXB7.5 (S2); no longer MUXB7.7 (S4)
- net GND: now also BAT2.3 (GND); no longer BAT1.MP, BAT2.2 (GND), BAT2.MP
- net at BAT1.2 (NTC), PMIC1.18 (NTC): now also BAT2.2 (NTC)
- no-connect marks 38 -> 37
Other:
- note added: "NOTE: - The Mux Placement: Place the 5 muxes as close to the nRF54L15 as possible. It is better to have long traces for the TMR outputs (which are slow DC signals) than long traces for the Mux-to-ADC lines (which carry the "chosen" signal). - Route the analog traces far away from PWM traces. - If aluminum plates are used for case, place 2 dowels to align them."
- note added: "NOTE: Only one of the batteries should be connected to NTC"
- note removed: "NOTE: - The Mux Placement: Place the 5 muxes as close to the nRF54L15 as possible. It is better to have long traces for the TMR outputs (which are slow DC signals) than long traces for the Mux-to-ADC lines (which carry the "chosen" signal). - Route the analog traces far away from PWM traces."
- moved on the sheet: C33, C34, C35, C36, LEDDR1
