File: hardware/nRF52840_bakelite_cnc/pcb/switch.kicad_sch (KiCad schematic)
At the start: 4 parts

Commit message: M  hardware/nRF52840_bakelite_cnc/border.py M  hardware/nRF52840_bakelite_cnc/pcb/pcb.kicad_pcb M  hardware/nRF52840_bakelite_cnc/pcb/pcb.kicad_prl M  hardware/nRF52840_bakelite_cnc/pcb/pcb.kicad_pro M  hardware/nRF52840_bakelite_cnc/pcb/pcb.kicad_sch M  hardware/nRF52840_bakelite_cnc/pcb/switch.kicad_sch M  hardware/nRF52840_bakelite_cnc/placefp.py M  hardware/nRF52840_bakelite_cnc/plate/plate.kicad_pcb M  hardware/nRF52840_bakelite_cnc/plate/plate.kicad_sch A  hardware/nRF52840_bakelite_cnc/tmr-footprints/C_0402_1005Metric_Cvcc.kicad_mod A  hardware/nRF52840_bakelite_cnc/tmr-footprints/C_0402_1005Metric_Cvout.kicad_mod M  hardware/nRF52840_bakelite_cnc/tmr-footprints/Gateron_Switch_Lowpro.kicad_mod A  hardware/nRF52840_bakelite_cnc/tmr-footprints/PCB_Wire_Solder_3p_Connector.kicad_mod
Parts:
- Cvcc1: footprint tmr-lib:C_0402_1005Metric -> tmr-lib:C_0402_1005Metric_Cvcc
- Cvout1: footprint tmr-lib:C_0402_1005Metric -> tmr-lib:C_0402_1005Metric_Cvout
Changed lines of the file:
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@@
 			)
 		)
-		(property "Footprint" "tmr-lib:C_0402_1005Metric"
+		(property "Footprint" "tmr-lib:C_0402_1005Metric_Cvout"
 			(at 140.97 69.85 0)
 			(effects
@@
 			)
 		)
-		(property "Footprint" "tmr-lib:C_0402_1005Metric"
+		(property "Footprint" "tmr-lib:C_0402_1005Metric_Cvcc"
 			(at 111.76 59.69 0)
 			(effects
