File: hardware/nRF52840_bakelite_cnc/plate/plate.kicad_sch (KiCad schematic)
At the start: 88 parts

Commit message: M  hardware/nRF52840_bakelite_cnc/border.py M  hardware/nRF52840_bakelite_cnc/pcb/pcb.kicad_prl M  hardware/nRF52840_bakelite_cnc/plate/plate.kicad_pcb M  hardware/nRF52840_bakelite_cnc/plate/plate.kicad_sch M  hardware/nRF52840_bakelite_cnc/plate/sym-lib-table
Parts:
- removed Hs11, Hs12: MountingHole, MountingHole:MountingHole_2.1mm, symbol Mechanical:MountingHole
- removed JLC1: JLC_Order_Num, tmr-lib:JLC_Order_Num, symbol Giri:JLC_Order_Num
- added JLC1: JLC_Order_Num, tmr-lib:JLC_Order_Num, symbol tmr-lib:JLC_Order_Num
- S42, S70: footprint tmr-lib:Switch_Cutout_1.25u -> tmr-lib:Switch_Cutout
- S46: footprint tmr-lib:Switch_Cutout_1.75u -> tmr-lib:Switch_Cutout
- S57: footprint tmr-lib:Switch_Cutout_1.75u -> tmr-lib:Switch_Cutout_1.25u
Changed lines of the file:
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@@
 	)
 	(symbol
-		(lib_id "Giri:JLC_Order_Num")
-		(at 191.77 104.14 0)
-		(unit 1)
-		(exclude_from_sim no)
-		(in_bom yes)
-		(on_board yes)
-		(dnp no)
-		(fields_autoplaced yes)
-		(property "Reference" "JLC1"
-			(at 195.58 102.87 0)
-			(effects
-				(font
-					(size 1.27 1.27)
-				)
-				(justify left)
-			)
-		)
-		(property "Value" "JLC_Order_Num"
-			(at 195.58 105.41 0)
-			(effects
-				(font
-					(size 1.27 1.27)
-				)
-				(justify left)
-				(hide yes)
-			)
-		)
-		(property "Footprint" "tmr-lib:JLC_Order_Num"
-			(at 191.77 104.14 0)
-			(effects
-				(font
-					(size 1.27 1.27)
-				)
-				(hide yes)
-			)
-		)
-		(property "Datasheet" ""
-			(at 191.77 104.14 0)
-			(effects
-				(font
-					(size 1.27 1.27)
-				)
-				(hide yes)
-			)
-		)
-		(property "Description" ""
-			(at 191.77 104.14 0)
-			(effects
-				(font
-					(size 1.27 1.27)
-				)
-			)
-		)
-		(instances
-			(project "plate"
-				(path "/4c67809e-1748-4898-89f6-ff92314048f2"
-					(reference "JLC1")
-					(unit 1)
-				)
-			)
-		)
-	)
-	(symbol
 		(lib_id "tmr-lib:SWHole")
 		(at 80.01 78.74 0)
@@
 			)
 		)
-		(property "Footprint" "tmr-lib:Switch_Cutout_1.75u"
+		(property "Footprint" "tmr-lib:Switch_Cutout_1.25u"
 			(at 194.31 78.74 0)
 			(effects
@@
 			)
 		)
-		(property "Footprint" "tmr-lib:Switch_Cutout_1.25u"
+		(property "Footprint" "tmr-lib:Switch_Cutout"
 			(at 194.31 66.04 0)
 			(effects
@@
 			)
 		)
-		(property "Footprint" "tmr-lib:Switch_Cutout_1.75u"
+		(property "Footprint" "tmr-lib:Switch_Cutout"
 			(at 68.58 78.74 0)
 			(effects
@@
 	)
 	(symbol
+		(lib_id "tmr-lib:JLC_Order_Num")
+		(at 198.12 119.38 0)
+		(unit 1)
+		(exclude_from_sim no)
+		(in_bom yes)
+		(on_board yes)
+		(dnp no)
+		(fields_autoplaced yes)
+		(property "Reference" "JLC1"
+			(at 201.93 118.1099 0)
+			(effects
+				(font
+					(size 1.27 1.27)
+				)
+				(justify left)
+			)
+		)
+		(property "Value" "JLC_Order_Num"
+			(at 201.93 120.6499 0)
+			(effects
+				(font
+					(size 1.27 1.27)
+				)
+				(justify left)
+			)
+		)
+		(property "Footprint" "tmr-lib:JLC_Order_Num"
+			(at 198.12 119.38 0)
+			(effects
+				(font
+					(size 1.27 1.27)
+				)
+				(hide yes)
+			)
+		)
+		(property "Datasheet" ""
+			(at 198.12 119.38 0)
+			(effects
+				(font
+					(size 1.27 1.27)
+				)
+				(hide yes)
+			)
+		)
+		(property "Description" ""
+			(at 198.12 119.38 0)
+			(effects
+				(font
+					(size 1.27 1.27)
+				)
+				(hide yes)
+			)
+		)
+		(instances
+			(project ""
+				(path "/4c67809e-1748-4898-89f6-ff92314048f2"
+					(reference "JLC1")
+					(unit 1)
+				)
+			)
+		)
+	)
+	(symbol
 		(lib_id "tmr-lib:SWHole")
 		(at 91.44 53.34 0)
@@
 			)
 		)
-		(property "Footprint" "tmr-lib:Switch_Cutout_1.25u"
+		(property "Footprint" "tmr-lib:Switch_Cutout"
 			(at 182.88 91.44 0)
 			(effects
@@
 					(unit 1)
 				)
-			)
-		)
-	)
-	(symbol
-		(lib_id "Mechanical:MountingHole")
-		(at 138.43 143.51 0)
-		(unit 1)
-		(exclude_from_sim no)
-		(in_bom no)
-		(on_board yes)
-		(dnp no)
-		(fields_autoplaced yes)
-		(property "Reference" "Hs11"
-			(at 140.97 142.2399 0)
-			(effects
-				(font
-					(size 1.27 1.27)
-				)
-				(justify left)
-			)
-		)
-		(property "Value" "MountingHole"
-			(at 140.97 144.7799 0)
-			(effects
-				(font
-					(size 1.27 1.27)
-				)
-				(justify left)
-			)
-		)
-		(property "Footprint" "MountingHole:MountingHole_2.1mm"
-			(at 138.43 143.51 0)
-			(effects
-				(font
-					(size 1.27 1.27)
-				)
-				(hide yes)
-			)
-		)
-		(property "Datasheet" "~"
-			(at 138.43 143.51 0)
-			(effects
-				(font
-					(size 1.27 1.27)
-				)
-				(hide yes)
-			)
-		)
-		(property "Description" "Mounting Hole without connection"
-			(at 138.43 143.51 0)
-			(effects
-				(font
-					(size 1.27 1.27)
-				)
-				(hide yes)
-			)
-		)
-		(instances
-			(project "plate"
-				(path "/4c67809e-1748-4898-89f6-ff92314048f2"
-					(reference "Hs11")
-					(unit 1)
-				)
-			)
-		)
-	)
-	(symbol
-		(lib_id "Mechanical:MountingHole")
-		(at 161.29 143.51 0)
-		(unit 1)
-		(exclude_from_sim no)
-		(in_bom no)
-		(on_board yes)
-		(dnp no)
-		(fields_autoplaced yes)
-		(property "Reference" "Hs12"
-			(at 163.83 142.2399 0)
-			(effects
-				(font
-					(size 1.27 1.27)
-				)
-				(justify left)
-			)
-		)
-		(property "Value" "MountingHole"
-			(at 163.83 144.7799 0)
-			(effects
-				(font
-					(size 1.27 1.27)
-				)
-				(justify left)
-			)
-		)
-		(property "Footprint" "MountingHole:MountingHole_2.1mm"
-			(at 161.29 143.51 0)
-			(effects
-				(font
-					(size 1.27 1.27)
-				)
-				(hide yes)
-			)
-		)
-		(property "Datasheet" "~"
-			(at 161.29 143.51 0)
-			(effects
-				(font
-					(size 1.27 1.27)
-				)
-				(hide yes)
-			)
-		)
-		(property "Description" "Mounting Hole without connection"
-			(at 161.29 143.51 0)
-			(effects
-				(font
-					(size 1.27 1.27)
-				)
-				(hide yes)
-			)
-		)
-		(instances
-			(project "plate"
-				(path "/4c67809e-1748-4898-89f6-ff92314048f2"
-					(reference "Hs12")
-					(unit 1)
-				)

Commit message: M  hardware/nRF52840_bakelite_cnc/border.py M  hardware/nRF52840_bakelite_cnc/pcb/pcb.kicad_pcb M  hardware/nRF52840_bakelite_cnc/pcb/pcb.kicad_prl M  hardware/nRF52840_bakelite_cnc/pcb/pcb.kicad_pro M  hardware/nRF52840_bakelite_cnc/pcb/pcb.kicad_sch M  hardware/nRF52840_bakelite_cnc/pcb/switch.kicad_sch M  hardware/nRF52840_bakelite_cnc/placefp.py M  hardware/nRF52840_bakelite_cnc/plate/plate.kicad_pcb M  hardware/nRF52840_bakelite_cnc/plate/plate.kicad_sch A  hardware/nRF52840_bakelite_cnc/tmr-footprints/C_0402_1005Metric_Cvcc.kicad_mod A  hardware/nRF52840_bakelite_cnc/tmr-footprints/C_0402_1005Metric_Cvout.kicad_mod M  hardware/nRF52840_bakelite_cnc/tmr-footprints/Gateron_Switch_Lowpro.kicad_mod A  hardware/nRF52840_bakelite_cnc/tmr-footprints/PCB_Wire_Solder_3p_Connector.kicad_mod
Parts:
- S70: footprint tmr-lib:Switch_Cutout -> tmr-lib:Switch_Cutout_1.25u
Changed lines of the file:
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@@
 			)
 		)
-		(property "Footprint" "tmr-lib:Switch_Cutout"
+		(property "Footprint" "tmr-lib:Switch_Cutout_1.25u"
 			(at 182.88 91.44 0)
 			(effects
