File: hardware/nRF52840_plastic_cnc/pcb/pcb.kicad_sch (KiCad schematic)
At the start: 149 parts, among them SW1 SW_DIP_x01, SW2 SW_DIP_x01, Y1 32.768 kHz

Commit message: M  hardware/nRF52840_plastic_cnc/border.py M  hardware/nRF52840_plastic_cnc/pcb/pcb-Edge_Cuts.dxf M  hardware/nRF52840_plastic_cnc/pcb/pcb.kicad_pcb M  hardware/nRF52840_plastic_cnc/pcb/pcb.kicad_prl M  hardware/nRF52840_plastic_cnc/pcb/pcb.kicad_sch M  hardware/nRF52840_plastic_cnc/placefp.py M  hardware/nRF52840_plastic_cnc/plate/plate.kicad_pcb M  hardware/nRF52840_plastic_cnc/plate/plate.kicad_sch
Parts:
- renumbered Hs1 to H1
Other:
- moved on the sheet: JLC1
Changed lines of the file:
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@@
 		(dnp no)
 		(fields_autoplaced yes)
-		(property "Reference" "Hs1"
+		(property "Reference" "H1"
 			(at 361.95 363.2199 0)
 			(effects
@@
 			(project "pcb"
 				(path "/672ae9a0-2ac9-4023-9977-e9626ff99f32"
-					(reference "Hs1")
+					(reference "H1")
 					(unit 1)
 				)
@@
 	(symbol
 		(lib_id "tmr-lib:JLC_Order_Num")
-		(at 391.16 392.43 0)
+		(at 392.43 410.21 0)
 		(unit 1)
 		(exclude_from_sim no)
@@
 		(fields_autoplaced yes)
 		(property "Reference" "JLC1"
-			(at 394.97 391.1599 0)
+			(at 396.24 408.9399 0)
 			(effects
 				(font
@@
 		)
 		(property "Value" "JLC_Order_Num"
-			(at 394.97 393.6999 0)
+			(at 396.24 411.4799 0)
 			(effects
 				(font
@@
 		)
 		(property "Footprint" "tmr-lib:JLC_Order_Num"
-			(at 391.16 392.43 0)
+			(at 392.43 410.21 0)
 			(effects
 				(font
@@
 		)
 		(property "Datasheet" ""
-			(at 391.16 392.43 0)
+			(at 392.43 410.21 0)
 			(effects
 				(font
@@
 		)
 		(property "Description" ""
-			(at 391.16 392.43 0)
-			(effects
-				(font
+			(at 392.43 410.21 0)
+			(effects
+				(font
