File: hardware/nRF52840_plastic_cnc/plate/plate.kicad_pcb (KiCad board)
At the start: 2 copper layers, 308.8 x 122.8 mm, 86 parts

Commit message: M  hardware/nRF52840_plastic_cnc/border.py M  hardware/nRF52840_plastic_cnc/pcb/pcb-Edge_Cuts.dxf M  hardware/nRF52840_plastic_cnc/pcb/pcb.kicad_pcb M  hardware/nRF52840_plastic_cnc/pcb/pcb.kicad_prl M  hardware/nRF52840_plastic_cnc/pcb/pcb.kicad_sch M  hardware/nRF52840_plastic_cnc/placefp.py M  hardware/nRF52840_plastic_cnc/plate/plate.kicad_pcb M  hardware/nRF52840_plastic_cnc/plate/plate.kicad_sch
Parts:
- S46: footprint tmr-lib:Switch_Cutout -> tmr-lib:Switch_Cutout_1.75u
- moved BAT2 20.4 mm to (230.2, 78.5)
- moved S45 4.75 mm to (7.12, 57.0)
- moved Hs4 3.62 mm to (21.4, 61.0)
- moved S46 2.38 mm to (35.6, 57.0)
- moved S59 1.00 mm to (10.9, 76.0)
- moved S60 0.80 mm to (34.6, 76.0)
- moved BAT1 0.60 mm to (23.0, 80.0)
- moved S61 0.60 mm to (56.0, 76.0)
- moved S69 0.60 mm to (219.5, 76.0)
- moved S70 0.60 mm to (240.9, 76.0)
Other:
- board size 308.8 x 122.8 mm -> 313.5 x 122.8 mm

Commit message: M  hardware/nRF52840_plastic_cnc/border.py A  hardware/nRF52840_plastic_cnc/pcb/pcb-User_1.dxf A  hardware/nRF52840_plastic_cnc/pcb/pcb-User_2.dxf A  hardware/nRF52840_plastic_cnc/pcb/pcb-User_3.dxf M  hardware/nRF52840_plastic_cnc/pcb/pcb.kicad_pcb M  hardware/nRF52840_plastic_cnc/pcb/pcb.kicad_prl M  hardware/nRF52840_plastic_cnc/placefp.py M  hardware/nRF52840_plastic_cnc/plate/plate.kicad_pcb M  hardware/nRF52840_plastic_cnc/plate/plate.kicad_sch M  hardware/nRF52840_plastic_cnc/tmr-footprints/Gateron_Switch_Lowpro.kicad_mod A  hardware/nRF52840_plastic_cnc/tmr-footprints/M2_HeatSinkNut_Flanged.kicad_mod
Parts:
- added H1: M2 Heat Sink Nut Marker (3.2mm,4.6mm flange), tmr-lib:M2_HeatSinkNut_Flanged, F.Cu at (28.5, 8.93)
- added H10: M2 Heat Sink Nut Marker (3.2mm,4.6mm flange), tmr-lib:M2_HeatSinkNut_Flanged, F.Cu at (264.8, 57.0)
- added H2: M2 Heat Sink Nut Marker (3.2mm,4.6mm flange), tmr-lib:M2_HeatSinkNut_Flanged, F.Cu at (142.5, 8.93)
- added H3: M2 Heat Sink Nut Marker (3.2mm,4.6mm flange), tmr-lib:M2_HeatSinkNut_Flanged, F.Cu at (275.5, 8.93)
- added H4: M2 Heat Sink Nut Marker (3.2mm,4.6mm flange), tmr-lib:M2_HeatSinkNut_Flanged, F.Cu at (21.4, 61.0)
- added H5: M2 Heat Sink Nut Marker (3.2mm,4.6mm flange), tmr-lib:M2_HeatSinkNut_Flanged, F.Cu at (137.8, 46.9)
- added H6: M2 Heat Sink Nut Marker (3.2mm,4.6mm flange), tmr-lib:M2_HeatSinkNut_Flanged, F.Cu at (86.4, 83.6)
- added H7: M2 Heat Sink Nut Marker (3.2mm,4.6mm flange), tmr-lib:M2_HeatSinkNut_Flanged, F.Cu at (189.1, 83.6)
- added H8: M2 Heat Sink Nut Marker (3.2mm,4.6mm flange), tmr-lib:M2_HeatSinkNut_Flanged, F.Cu at (95.0, 27.9)
- added H9: M2 Heat Sink Nut Marker (3.2mm,4.6mm flange), tmr-lib:M2_HeatSinkNut_Flanged, F.Cu at (209.0, 27.9)
Other:
- outline, holes or cut-outs redrawn
