File: hardware/nRF52840_fr4_cnc/pcb/pcb.kicad_sch (KiCad schematic)
At the start: 149 parts, among them SW1 SW_DIP_x01, SW2 SW_DIP_x01, Y1 32.768 kHz

Commit message: R  hardware/nRF52840_plastic_cnc/README.md -> hardware/nRF52840_abs_cnc/README.md R  hardware/nRF52840_plastic_cnc/border.py -> hardware/nRF52840_abs_cnc/border.py R  hardware/nRF52840_plastic_cnc/curves.py -> hardware/nRF52840_abs_cnc/curves.py R  hardware/nRF52840_plastic_cnc/dumploc.py -> hardware/nRF52840_abs_cnc/dumploc.py R  hardware/nRF52840_plastic_cnc/nordic-lib-kicad-npm.kicad_sym -> hardware/nRF52840_abs_cnc/nordic-lib-kicad-npm.kicad_sym R  hardware/nRF52840_plastic_cnc/pcb/LED.kicad_sch -> hardware/nRF52840_abs_cnc/pcb/LED.kicad_sch R  hardware/nRF52840_plastic_cnc/pcb/fp-lib-table -> hardware/nRF52840_abs_cnc/pcb/fp-lib-table R  hardware/nRF52840_fr4_cnc/pcb/pcb-Edge_Cuts.dxf -> hardware/nRF52840_abs_cnc/pcb/pcb-Edge_Cuts.dxf R  hardware/nRF52840_fr4_cnc/pcb/pcb-User_1.dxf -> hardware/nRF52840_abs_cnc/pcb/pcb-User_1.dxf R  hardware/nRF52840_fr4_cnc/pcb/pcb-User_2.dxf -> hardware/nRF52840_abs_cnc/pcb/pcb-User_2.dxf R  hardware/nRF52840_fr4_cnc/pcb/pcb-User_3.dxf -> hardware/nRF52840_abs_cnc/pcb/pcb-User_3.dxf R  hardware/nRF52840_plastic_cnc/pcb/pcb-eagle-import.kicad_sym -> hardware/nRF52840_abs_cnc/pcb/pcb-eagle-import.kicad_sym R  hardware/nRF52840_plastic_cnc/pcb/pcb.kicad_pcb -> hardware/nRF52840_abs_cnc/pcb/pcb.kicad_pcb R  hardware/nRF52840_plastic_cnc/pcb/pcb.kicad_prl -> hardware/nRF52840_abs_cnc/pcb/pcb.kicad_prl R  hardware/nRF52840_plastic_cnc/pcb/pcb.kicad_pro -> hardware/nRF52840_abs_cnc/pcb/pcb.kicad_pro R  hardware/nRF52840_plastic_cnc/pcb/pcb.kicad_sch -> hardware/nRF52840_abs_cnc/pcb/pcb.kicad_sch R  hardware/nRF52840_plastic_cnc/pcb/switch.kicad_sch -> hardware/nRF52840_abs_cnc/pcb/switch.kicad_sch R  hardware/nRF52840_plastic_cnc/pcb/sym-lib-table -> hardware/nRF52840_abs_cnc/pcb/sym-lib-table R  hardware/nRF52840_plastic_cnc/placefp.py -> hardware/nRF52840_abs_cnc/placefp.py R  hardware/nRF52840_plastic_cnc/plate/fp-lib-table -> hardware/nRF52840_abs_cnc/plate/fp-lib-table R  hardware/nRF52840_plastic_cnc/plate/plate.kicad_pcb -> ha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
Parts:
- SW1, SW2: footprint tmr-lib:Aliexpress_SW_DIP_TS_1292V_4x6.2x1.8mm -> tmr-lib:Aliexpress_SW_TACT_4x4x1.5mm
Changed lines of the file:
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@@
 			)
 		)
-		(property "Footprint" "tmr-lib:Aliexpress_SW_DIP_TS_1292V_4x6.2x1.8mm"
+		(property "Footprint" "tmr-lib:Aliexpress_SW_TACT_4x4x1.5mm"
 			(at 397.51 303.53 0)
 			(effects
@@
 			)
 		)
-		(property "Footprint" "tmr-lib:Aliexpress_SW_DIP_TS_1292V_4x6.2x1.8mm"
+		(property "Footprint" "tmr-lib:Aliexpress_SW_TACT_4x4x1.5mm"
 			(at 499.11 113.03 0)
 			(effects
