File: hardware/nRF52840_fr4_cnc/pcb/switch.kicad_sch (KiCad schematic)
At the start: 4 parts

Commit message: R  hardware/nRF52840_plastic_cnc/README.md -> hardware/nRF52840_abs_cnc/README.md R  hardware/nRF52840_plastic_cnc/border.py -> hardware/nRF52840_abs_cnc/border.py R  hardware/nRF52840_plastic_cnc/curves.py -> hardware/nRF52840_abs_cnc/curves.py R  hardware/nRF52840_plastic_cnc/dumploc.py -> hardware/nRF52840_abs_cnc/dumploc.py R  hardware/nRF52840_plastic_cnc/nordic-lib-kicad-npm.kicad_sym -> hardware/nRF52840_abs_cnc/nordic-lib-kicad-npm.kicad_sym R  hardware/nRF52840_plastic_cnc/pcb/LED.kicad_sch -> hardware/nRF52840_abs_cnc/pcb/LED.kicad_sch R  hardware/nRF52840_plastic_cnc/pcb/fp-lib-table -> hardware/nRF52840_abs_cnc/pcb/fp-lib-table R  hardware/nRF52840_fr4_cnc/pcb/pcb-Edge_Cuts.dxf -> hardware/nRF52840_abs_cnc/pcb/pcb-Edge_Cuts.dxf R  hardware/nRF52840_fr4_cnc/pcb/pcb-User_1.dxf -> hardware/nRF52840_abs_cnc/pcb/pcb-User_1.dxf R  hardware/nRF52840_fr4_cnc/pcb/pcb-User_2.dxf -> hardware/nRF52840_abs_cnc/pcb/pcb-User_2.dxf R  hardware/nRF52840_fr4_cnc/pcb/pcb-User_3.dxf -> hardware/nRF52840_abs_cnc/pcb/pcb-User_3.dxf R  hardware/nRF52840_plastic_cnc/pcb/pcb-eagle-import.kicad_sym -> hardware/nRF52840_abs_cnc/pcb/pcb-eagle-import.kicad_sym R  hardware/nRF52840_plastic_cnc/pcb/pcb.kicad_pcb -> hardware/nRF52840_abs_cnc/pcb/pcb.kicad_pcb R  hardware/nRF52840_plastic_cnc/pcb/pcb.kicad_prl -> hardware/nRF52840_abs_cnc/pcb/pcb.kicad_prl R  hardware/nRF52840_plastic_cnc/pcb/pcb.kicad_pro -> hardware/nRF52840_abs_cnc/pcb/pcb.kicad_pro R  hardware/nRF52840_plastic_cnc/pcb/pcb.kicad_sch -> hardware/nRF52840_abs_cnc/pcb/pcb.kicad_sch R  hardware/nRF52840_plastic_cnc/pcb/switch.kicad_sch -> hardware/nRF52840_abs_cnc/pcb/switch.kicad_sch R  hardware/nRF52840_plastic_cnc/pcb/sym-lib-table -> hardware/nRF52840_abs_cnc/pcb/sym-lib-table R  hardware/nRF52840_plastic_cnc/placefp.py -> hardware/nRF52840_abs_cnc/placefp.py R  hardware/nRF52840_plastic_cnc/plate/fp-lib-table -> hardware/nRF52840_abs_cnc/plate/fp-lib-table R  hardware/nRF52840_plastic_cnc/plate/plate.kicad_pcb -> ha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
Parts:
- S1: footprint tmr-lib:Gateron_Kailh_Lowpro_Switch -> tmr-lib:Gateron_Lowpro_Switch
Changed lines of the file:
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@@
 			)
 		)
-		(property "Footprint" "tmr-lib:Gateron_Kailh_Lowpro_Switch"
+		(property "Footprint" "tmr-lib:Gateron_Lowpro_Switch"
 			(at 97.79 64.77 0)
 			(effects
