File: hardware/nRF52840_fr4_cnc/plate/plate.kicad_pcb (KiCad board)
At the start: 2 copper layers, 313.5 x 122.8 mm, 96 parts

Commit message: M  hardware/nRF52840_fr4_cnc/plate/plate.kicad_pcb
Parts:
- moved Jusb1 20.5 mm to (4.50, -1.00), turned to -90 degrees
Other:
- outline, holes or cut-outs redrawn
