File: hardware/nRF54L15_kailh/plate/plate.kicad_pcb (KiCad board)
At the start: 2 copper layers, 313.5 x 122.8 mm, 96 parts

Commit message: M  hardware/nRF54L15_kailh/border.py A  hardware/nRF54L15_kailh/pcb/pcb-F_Fab.dxf M  hardware/nRF54L15_kailh/pcb/pcb.kicad_pcb M  hardware/nRF54L15_kailh/pcb/pcb.kicad_prl M  hardware/nRF54L15_kailh/pcb/pcb.kicad_sch M  hardware/nRF54L15_kailh/placefp.py A  hardware/nRF54L15_kailh/plate/plate-User_5.dxf M  hardware/nRF54L15_kailh/plate/plate.kicad_pcb M  hardware/nRF54L15_kailh/plate/plate.kicad_sch A  hardware/nRF54L15_kailh/tmr-footprints/MountingHole_1.7mm_M1.6_NoPad.kicad_mod M  hardware/nRF54L15_kailh/tmr-footprints/MountingHole_2.1mm_M2_NoPad.kicad_mod M  hardware/nRF54L15_kailh/tmr-footprints/Stabilizer_Lowpro_2U.kicad_mod R  hardware/nRF54L15_kailh/tmr-footprints/Switch_Cutout_1.25u.kicad_mod -> hardware/nRF54L15_kailh/tmr-footprints/Switch_Cutout_1.25u_powdercoat.kicad_mod R  hardware/nRF54L15_kailh/tmr-footprints/Switch_Cutout_1.75u.kicad_mod -> hardware/nRF54L15_kailh/tmr-footprints/Switch_Cutout_1.75u_powdercoat.kicad_mod R  hardware/nRF54L15_kailh/tmr-footprints/Switch_Cutout_2u.kicad_mod -> hardware/nRF54L15_kailh/tmr-footprints/Switch_Cutout_2u_powdercoat.kicad_mod R  hardware/nRF54L15_kailh/tmr-footprints/Switch_Cutout.kicad_mod -> hardware/nRF54L15_kailh/tmr-footprints/Switch_Cutout_powdercoat.kicad_mod A  hardware/nRF54L15_kailh/tmr-footprints/USB_C_Receptacle_GCT_USB4125-xx-x_6P_TopMnt_Horizontal.kicad_mod
Parts:
- removed H1, H10, H2, H3, H4, H5, H6, H7, H8, H9: M2 Heat Sink Nut Marker (3.2mm,4.6mm flange), tmr-lib:M2_HeatSinkNut_Flanged
- Hs6, Hs7, Hs8, Hs9: footprint MountingHole:MountingHole_2.1mm -> tmr-lib:MountingHole_1.7mm_M1.6_NoPad
- S1, S10, S11, S12, S13, S14, S15, S16, S17, S18, S19, S2, S20, S21, S22, S23, S24, S25, S26, S27, S28, S29, S3, S31, S32, S33, S34, S35, S36, S37, S38, S39, S4, S40, S41, S42, S43, S44, S47, S48, S49, S5, S50, S51, S52, S53, S54, S55, S56, S58, S6, S61, S62, S63, S65, S67, S68, S69, S7, S71, S72, S8, S9: footprint tmr-lib:Switch_Cutout -> tmr-lib:Switch_Cutout_powdercoat
- S30, S45, S57, S59, S60, S70: footprint tmr-lib:Switch_Cutout_1.25u -> tmr-lib:Switch_Cutout_1.25u_powdercoat
- S46: footprint tmr-lib:Switch_Cutout_1.75u -> tmr-lib:Switch_Cutout_1.75u_powdercoat
- S64, S66: footprint tmr-lib:Switch_Cutout_2u -> tmr-lib:Switch_Cutout_2u_powdercoat
- moved Jusb1 4.91 mm to (8.40, -3.98)
- moved BAT1 4.75 mm to (18.2, 80.0)
- moved S59 3.75 mm to (7.12, 76.0)
- moved S60 3.75 mm to (30.9, 76.0)
- moved S61 3.75 mm to (52.2, 76.0)
- moved S69 3.75 mm to (223.2, 76.0)
- moved BAT2 3.62 mm to (232.7, 81.1)
- moved S70 1.38 mm to (242.2, 76.0)
- moved S63 1.35 mm to (95.1, 87.2)
- moved S67 1.35 mm to (180.4, 87.2)
- moved S68 1.34 mm to (198.3, 80.7)
- moved S62 1.26 mm to (77.2, 80.7)
Other:
- outline, holes or cut-outs redrawn

Commit message: M  hardware/nRF54L15_kailh/plate/plate.kicad_pcb
Parts:
- moved Jusb1 13.3 mm to (19.0, -12.0), turned to 180 degrees
