File: hardware/nRF54L15_kailh/swplate/swplate.kicad_sch (KiCad schematic)
At the start: 102 parts

Commit message: M .gitignore M  hardware/nRF54L15_kailh/border.py M  hardware/nRF54L15_kailh/swplate/swplate.kicad_pcb M  hardware/nRF54L15_kailh/swplate/swplate.kicad_sch ?? hardware/resources/
Parts:
- Hd1, Hd2: footprint tmr-lib:DowelHole_3.0mm_M3_powdercoat -> tmr-lib:DowelHole_3.2mm_M3_powdercoat
Changed lines of the file:
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@@
 			)
 		)
-		(property "Footprint" "tmr-lib:DowelHole_3.0mm_M3_powdercoat"
+		(property "Footprint" "tmr-lib:DowelHole_3.2mm_M3_powdercoat"
 			(at 184.15 151.13 0)
 			(effects
@@
 			)
 		)
-		(property "Footprint" "tmr-lib:DowelHole_3.0mm_M3_powdercoat"
+		(property "Footprint" "tmr-lib:DowelHole_3.2mm_M3_powdercoat"
 			(at 163.83 151.13 0)
 			(effects
