File: hardware/nRF54L15_kailh/swplate/swplate.kicad_sch (KiCad schematic)
At the start: 102 parts

Commit message: M  .gitignore A  hardware/nRF54L15_gateron_kailh_TMR2615/LED.kicad_sch A  hardware/nRF54L15_gateron_kailh_TMR2615/fp-lib-table A  hardware/nRF54L15_gateron_kailh_TMR2615/nRF54L15_gateron_kailh_TMR2615.kicad_pcb A  hardware/nRF54L15_gateron_kailh_TMR2615/nRF54L15_gateron_kailh_TMR2615.kicad_prl A  hardware/nRF54L15_gateron_kailh_TMR2615/nRF54L15_gateron_kailh_TMR2615.kicad_pro A  hardware/nRF54L15_gateron_kailh_TMR2615/nRF54L15_gateron_kailh_TMR2615.kicad_sch A  hardware/nRF54L15_gateron_kailh_TMR2615/pcb-eagle-import.kicad_sym A  hardware/nRF54L15_gateron_kailh_TMR2615/switch.kicad_sch A  hardware/nRF54L15_gateron_kailh_TMR2615/sym-lib-table M  hardware/nRF54L15_kailh/border.py A  hardware/nRF54L15_kailh/botcase/botcase-Edge_Cuts.pdf M  hardware/nRF54L15_kailh/botcase/botcase.kicad_pcb M  hardware/nRF54L15_kailh/botcase/botcase.kicad_sch M  hardware/nRF54L15_kailh/botcover/botcover.kicad_pcb M  hardware/nRF54L15_kailh/botcover/botcover.kicad_sch M  hardware/nRF54L15_kailh/placefp.py A  hardware/nRF54L15_kailh/rebuild_board.py A  hardware/nRF54L15_kailh/run.sh M  hardware/nRF54L15_kailh/swplate/swplate.kicad_pcb M  hardware/nRF54L15_kailh/swplate/swplate.kicad_sch A  hardware/nRF54L15_kailh/tmr-footprints/Kailh_gateron_sw_lowpro.kicad_mod M  hardware/nRF54L15_kailh/tmr-footprints/Kailh_sw_lowpro.kicad_mod A  hardware/nRF54L15_kailh/tmr-footprints/M1.4_tap.kicad_mod A  hardware/nRF54L15_kailh/tmr-footprints/M2.5_tap.kicad_mod A  hardware/nRF54L15_kailh/tmr-footprints/MountingHole_1.6mm_M1.4_NoPad.kicad_mod M  hardware/nRF54L15_kailh/topcase/topcase.kicad_pcb A  hardware/nRF54L15_kailh/wristrest/fp-lib-table A  hardware/nRF54L15_kailh/wristrest/sym-lib-table A  hardware/nRF54L15_kailh/wristrest/wristrest.kicad_pcb A  hardware/nRF54L15_kailh/wristrest/wristrest.kicad_prl A  hardware/nRF54L15_kailh/wristrest/wristrest.kicad_pro A  hardware/nRF54L15_kailh/wristrest/wristrest.kicad_sch
Parts:
- H16: footprint tmr-lib:DowelHole_3.1mm_M3_powdercoat -> tmr-lib:MountingHole_2.7mm_M2.5
- Hd2: footprint tmr-lib:DowelHole_3.2mm_M3_powdercoat -> tmr-lib:DowelHole_3.1mm_M3_powdercoat
- Hs1, Hs10, Hs2, Hs3, Hs4, Hs5: footprint MountingHole:MountingHole_2.1mm -> MountingHole:MountingHole_2.2mm_M2
- Hs6, Hs7, Hs8, Hs9: footprint tmr-lib:MountingHole_1.7mm_M1.6_NoPad -> tmr-lib:MountingHole_1.6mm_M1.4_NoPad
Changed lines of the file:
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@@
 			)
 		)
-		(property "Footprint" "tmr-lib:MountingHole_1.7mm_M1.6_NoPad"
+		(property "Footprint" "tmr-lib:MountingHole_1.6mm_M1.4_NoPad"
 			(at 118.11 124.46 0)
 			(effects
@@
 			)
 		)
-		(property "Footprint" "tmr-lib:MountingHole_1.7mm_M1.6_NoPad"
+		(property "Footprint" "tmr-lib:MountingHole_1.6mm_M1.4_NoPad"
 			(at 163.83 124.46 0)
 			(effects
@@
 			)
 		)
-		(property "Footprint" "MountingHole:MountingHole_2.1mm"
+		(property "Footprint" "MountingHole:MountingHole_2.2mm_M2"
 			(at 96.52 114.3 0)
 			(effects
@@
 			)
 		)
-		(property "Footprint" "tmr-lib:DowelHole_3.2mm_M3_powdercoat"
+		(property "Footprint" "tmr-lib:DowelHole_3.1mm_M3_powdercoat"
 			(at 184.15 151.13 0)
 			(effects
@@
 			)
 		)
-		(property "Footprint" "tmr-lib:DowelHole_3.1mm_M3_powdercoat"
+		(property "Footprint" "tmr-lib:MountingHole_2.7mm_M2.5"
 			(at 110.49 185.42 0)
 			(effects
@@
 			)
 		)
-		(property "Footprint" "tmr-lib:MountingHole_1.7mm_M1.6_NoPad"
+		(property "Footprint" "tmr-lib:MountingHole_1.6mm_M1.4_NoPad"
 			(at 140.97 124.46 0)
 			(effects
@@
 			)
 		)
-		(property "Footprint" "MountingHole:MountingHole_2.1mm"
+		(property "Footprint" "MountingHole:MountingHole_2.2mm_M2"
 			(at 118.11 134.62 0)
 			(effects
@@
 			)
 		)
-		(property "Footprint" "MountingHole:MountingHole_2.1mm"
+		(property "Footprint" "MountingHole:MountingHole_2.2mm_M2"
 			(at 118.11 114.3 0)
 			(effects
@@
 			)
 		)
-		(property "Footprint" "MountingHole:MountingHole_2.1mm"
+		(property "Footprint" "MountingHole:MountingHole_2.2mm_M2"
 			(at 140.97 114.3 0)
 			(effects
@@
 			)
 		)
-		(property "Footprint" "tmr-lib:MountingHole_1.7mm_M1.6_NoPad"
+		(property "Footprint" "tmr-lib:MountingHole_1.6mm_M1.4_NoPad"
 			(at 96.52 134.62 0)
 			(effects
@@
 			)
 		)
-		(property "Footprint" "MountingHole:MountingHole_2.1mm"
+		(property "Footprint" "MountingHole:MountingHole_2.2mm_M2"
 			(at 96.52 124.46 0)
 			(effects
@@
 			)
 		)
-		(property "Footprint" "MountingHole:MountingHole_2.1mm"
+		(property "Footprint" "MountingHole:MountingHole_2.2mm_M2"
 			(at 163.83 114.3 0)
 			(effects
