File: hardware/nRF54L15_kailh/swplate/swplate.kicad_pcb (KiCad board)
At the start: 2 copper layers, 328.5 x 199 mm, 102 parts

Commit message: M .gitignore M  hardware/nRF54L15_kailh/border.py M  hardware/nRF54L15_kailh/swplate/swplate.kicad_pcb M  hardware/nRF54L15_kailh/swplate/swplate.kicad_sch ?? hardware/resources/
Parts:
- Hd1, Hd2: footprint tmr-lib:DowelHole_3.0mm_M3_powdercoat -> tmr-lib:DowelHole_3.2mm_M3_powdercoat
Other:
- board size 328.5 x 199 mm -> 328.1 x 198.6 mm

Commit message: M .gitignore M  hardware/nRF54L15_kailh/border.py A  hardware/nRF54L15_kailh/pat1.kicad_mod A  hardware/nRF54L15_kailh/pat1.kicad_sym A  hardware/nRF54L15_kailh/pat2.kicad_mod A  hardware/nRF54L15_kailh/pat3.kicad_mod A  hardware/nRF54L15_kailh/pat4.kicad_mod A  hardware/nRF54L15_kailh/pat5.kicad_mod M  hardware/nRF54L15_kailh/swplate/swplate.kicad_pcb M  hardware/nRF54L15_kailh/swplate/swplate.kicad_prl A  hardware/nRF54L15_kailh/tmr-footprints/pat1.kicad_mod A  hardware/nRF54L15_kailh/tmr-footprints/pat2.kicad_mod A  hardware/nRF54L15_kailh/tmr-footprints/pat3.kicad_mod A  hardware/nRF54L15_kailh/tmr-footprints/pat4.kicad_mod A  hardware/nRF54L15_kailh/tmr-footprints/pat5.kicad_mod
Other:
- outline, holes or cut-outs redrawn
