File: hardware/nRF54L15_kailh/swplate/swplate.kicad_pcb (KiCad board)
At the start: 2 copper layers, 328.1 x 198.6 mm, 102 parts

Commit message: M  .gitignore A  hardware/nRF54L15_gateron_kailh_TMR2615/LED.kicad_sch A  hardware/nRF54L15_gateron_kailh_TMR2615/fp-lib-table A  hardware/nRF54L15_gateron_kailh_TMR2615/nRF54L15_gateron_kailh_TMR2615.kicad_pcb A  hardware/nRF54L15_gateron_kailh_TMR2615/nRF54L15_gateron_kailh_TMR2615.kicad_prl A  hardware/nRF54L15_gateron_kailh_TMR2615/nRF54L15_gateron_kailh_TMR2615.kicad_pro A  hardware/nRF54L15_gateron_kailh_TMR2615/nRF54L15_gateron_kailh_TMR2615.kicad_sch A  hardware/nRF54L15_gateron_kailh_TMR2615/pcb-eagle-import.kicad_sym A  hardware/nRF54L15_gateron_kailh_TMR2615/switch.kicad_sch A  hardware/nRF54L15_gateron_kailh_TMR2615/sym-lib-table M  hardware/nRF54L15_kailh/border.py A  hardware/nRF54L15_kailh/botcase/botcase-Edge_Cuts.pdf M  hardware/nRF54L15_kailh/botcase/botcase.kicad_pcb M  hardware/nRF54L15_kailh/botcase/botcase.kicad_sch M  hardware/nRF54L15_kailh/botcover/botcover.kicad_pcb M  hardware/nRF54L15_kailh/botcover/botcover.kicad_sch M  hardware/nRF54L15_kailh/placefp.py A  hardware/nRF54L15_kailh/rebuild_board.py A  hardware/nRF54L15_kailh/run.sh M  hardware/nRF54L15_kailh/swplate/swplate.kicad_pcb M  hardware/nRF54L15_kailh/swplate/swplate.kicad_sch A  hardware/nRF54L15_kailh/tmr-footprints/Kailh_gateron_sw_lowpro.kicad_mod M  hardware/nRF54L15_kailh/tmr-footprints/Kailh_sw_lowpro.kicad_mod A  hardware/nRF54L15_kailh/tmr-footprints/M1.4_tap.kicad_mod A  hardware/nRF54L15_kailh/tmr-footprints/M2.5_tap.kicad_mod A  hardware/nRF54L15_kailh/tmr-footprints/MountingHole_1.6mm_M1.4_NoPad.kicad_mod M  hardware/nRF54L15_kailh/topcase/topcase.kicad_pcb A  hardware/nRF54L15_kailh/wristrest/fp-lib-table A  hardware/nRF54L15_kailh/wristrest/sym-lib-table A  hardware/nRF54L15_kailh/wristrest/wristrest.kicad_pcb A  hardware/nRF54L15_kailh/wristrest/wristrest.kicad_prl A  hardware/nRF54L15_kailh/wristrest/wristrest.kicad_pro A  hardware/nRF54L15_kailh/wristrest/wristrest.kicad_sch
Parts:
- H16: footprint tmr-lib:DowelHole_3.1mm_M3_powdercoat -> tmr-lib:MountingHole_2.7mm_M2.5
- Hd2: footprint tmr-lib:DowelHole_3.2mm_M3_powdercoat -> tmr-lib:DowelHole_3.1mm_M3_powdercoat
- Hs1, Hs10, Hs2, Hs3, Hs4, Hs5: footprint MountingHole:MountingHole_2.1mm -> MountingHole:MountingHole_2.2mm_M2
- Hs6, Hs7, Hs8, Hs9: footprint tmr-lib:MountingHole_1.7mm_M1.6_NoPad -> tmr-lib:MountingHole_1.6mm_M1.4_NoPad
