File: hardware/nRF54L15_kailh/botcover/botcover.kicad_pcb (KiCad board)
At the start: 2 copper layers, 328.1 x 198.6 mm, 143 parts

Commit message: M  hardware/nRF54L15_kailh/border.py M  hardware/nRF54L15_kailh/botcover/botcover.kicad_pcb M  hardware/nRF54L15_kailh/botcover/botcover.kicad_sch M  hardware/nRF54L15_kailh/pcb/pcb.kicad_pcb M  hardware/nRF54L15_kailh/pcb/pcb.kicad_sch M  hardware/nRF54L15_kailh/placefp.py A  hardware/nRF54L15_kailh/tmr-footprints/MountingHole_1.5mm_M1.4_NoPad.kicad_mod R  hardware/nRF54L15_kailh/tmr-footprints/SMTSO_M1.6.kicad_mod -> hardware/nRF54L15_kailh/tmr-footprints/SMTSO_M1.4_M1.6.kicad_mod
Parts:
- removed Hr30, Hr31, Hr32, Hr33, Hr34, Hr35, Hr36, Hr37, Hr38, Hr39, Hr40, Hr41, Hr42, Hr43, Hr44, Hr45, Hr46, Hr47, Hr48, Hr49, Hr50, Hr51, Hr52, Hr53: Rivet, tmr-lib:RivetClearanceHole_1.5mm
- added Hm1: M1.4, tmr-lib:MountingHole_1.5mm_M1.4_NoPad, F.Cu at (99.8, 40.5)
- added Hm2: M1.4, tmr-lib:MountingHole_1.5mm_M1.4_NoPad, F.Cu at (213.8, 40.5)
- Hr1, Hr10, Hr11, Hr12, Hr13, Hr14, Hr15, Hr16, Hr17, Hr18, Hr19, Hr2, Hr20, Hr21, Hr22, Hr23, Hr24, Hr25, Hr26, Hr27, Hr28, Hr29, Hr3, Hr4, Hr5, Hr6, Hr7, Hr8, Hr9: value Rivet -> M1.4; footprint tmr-lib:RivetClearanceHole_1.5mm -> tmr-lib:MountingHole_1.5mm_M1.4_NoPad
- moved Hr11 318.3 mm to (-9.00, 85.0)
- moved Hr10 278.8 mm to (-8.00, 39.0)
- moved Hr25 253.0 mm to (290.5, 130.5)
- moved Hr17 248.2 mm to (265.0, 83.0)
- moved Hr24 244.8 mm to (253.0, 113.0)
- moved Hr26 232.3 mm to (291.0, 165.0)
- moved Hr16 222.0 mm to (213.0, 88.5)
- moved Hr27 178.5 mm to (246.0, 177.0)
- moved Hr29 177.7 mm to (220.0, 122.0)
- moved Hr15 177.0 mm to (159.0, 115.5)
- moved Hr28 163.8 mm to (205.5, 165.5)
- moved Hr14 153.8 mm to (137.8, 88.0)
- moved Hr13 146.1 mm to (116.5, 115.5)
- moved Hr8 106.6 mm to (309.5, 23.0)
- moved Hr9 105.5 mm to (308.5, 65.5)
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Other:
- outline, holes or cut-outs redrawn
- board text added: "NOTE: - Use FreeCAD to generate STEP file to preserve Bezier curves. KiCad facets the Bezier curves."
- board text removed: "NOTE: - M1.4 rivets should be driven sub-flush and covered in paint or enamel to prevent scratching of laptop. - Use FreeCAD to generate STEP file to preserve Bezier curves. KiCad facets the Bezier curves. - Cut away a slot 30mm x 2mm in front of BLE antenna"
