File: hardware/nRF54LM20_TMR2615/pcb/.history/pcb.kicad_pcb (KiCad board)
At the start: 2 copper layers, 299.2 x 119.8 mm, 426 parts, among them M1 Minew_ME54BS13_V1.0, SW1 SW_DIP_x01, SW2 SW_DIP_x01

Commit message: M  hardware/nRF54LM20_TMR2615/pcb/.history/pcb.kicad_pcb M  hardware/nRF54LM20_TMR2615/pcb/pcb.kicad_pcb M  hardware/nRF54LM20_TMR2615/pcb/pcb.kicad_prl
Routing:
- net /MUXB_SEL_2: track 272.1 -> 269.3 mm
- net /ANA_16: track 106.3 -> 104.4 mm
- net /ANA_18: track 57.2 -> 55.5 mm
- net /ANA_17: track 78.7 -> 77.0 mm
- net /SCL: track 184.8 -> 183.3 mm
- net /SW0: track 842.4 -> 841.2 mm
- net /ANA_60: track 120.8 -> 119.9 mm
- net /ANA_59: track 141.0 -> 140.1 mm
- net /ANA_45: track 130.0 -> 129.1 mm
- net /ANA_46: track 99.9 -> 99.1 mm
- net VCCS: track 2756.2 -> 2755.5 mm
- net /SDA: track 182.6 -> 181.9 mm
- net GND: track 622.5 -> 622.0 mm
