File: hardware/nRF54LM20_TMR2615/swplate/swplate.kicad_pcb (KiCad board)
At the start: 2 copper layers, 313.9 x 198.7 mm, 103 parts, among them M1 Minew_ME54BS13_V1.0

Commit message: A  hardware/nRF54LM20_TMR2615/cohr M  hardware/nRF54LM20_TMR2615/pcb/pcb.kicad_pcb M  hardware/nRF54LM20_TMR2615/pcb/pcb.kicad_prl M  hardware/nRF54LM20_TMR2615/placefp.py M  hardware/nRF54LM20_TMR2615/swplate/swplate.kicad_pcb M  hardware/nRF54LM20_TMR2615/swplate/swplate.kicad_sch
Parts:
- S63: footprint tmr-lib:Switch_Cutout -> tmr-lib:Switch_Cutout_1.25u
- moved S63 2.42 mm to (95.9, 85.0), turned to 70 degrees
- moved S42 2.38 mm to (244.6, 38.0)
- moved S43 2.38 mm to (266.0, 38.0)
- moved Hs6 1.00 mm to (104.5, 75.0)
Changed lines of the file:
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@@
 		)
 	)
-	(footprint "tmr-lib:Switch_Cutout"
+	(footprint "tmr-lib:Switch_Cutout_1.25u"
 		(layer "F.Cu")
-		(at 95.1 87.25 -20)
+		(at 95.88 84.96 70)
 		(descr "Cherry MX keyswitch PCB Mount with 1.00u keycap")
 		(tags "Cherry MX Keyboard Keyswitch Switch PCB Cutout 1.00u")
 		(property "Reference" "S63"
-			(at 0.1 -6.1 340)
+			(at 0.1 -6.1 70)
 			(layer "F.SilkS")
 			(hide yes)
@@
 		)
 		(property "Value" "SWHole"
-			(at 0.1 8.5 340)
+			(at 0.1 8.5 70)
 			(layer "F.Fab")
 			(effects
@@
 		)
 		(property "Datasheet" ""
-			(at 0 0 340)
+			(at 0 0 70)
 			(layer "F.Fab")
 			(hide yes)
@@
 		)
 		(property "Description" ""
-			(at 0 0 340)
+			(at 0 0 70)
 			(layer "F.Fab")
 			(hide yes)
@@
 		(duplicate_pad_numbers_are_jumpers no)
 		(fp_line
-			(start -6.6 7)
-			(end 6.6 7)
+			(start -6.6 -7)
+			(end 6.6 -7)
 			(stroke
 				(width 0.12)
@@
 		)
 		(fp_line
-			(start -6.6 -7)
-			(end 6.6 -7)
+			(start 7 -6.6)
+			(end 7 6.6)
 			(stroke
 				(width 0.12)
@@
 		)
 		(fp_line
-			(start 7 -6.6)
-			(end 7 6.6)
+			(start -6.6 7)
+			(end 6.6 7)
 			(stroke
 				(width 0.12)
@@
 		)
 		(fp_arc
-			(start -6.6 7)
-			(mid -6.882843 6.882843)
-			(end -7 6.6)
+			(start -7 -6.6)
+			(mid -6.882843 -6.882843)
+			(end -6.6 -7)
 			(stroke
 				(width 0.12)
@@
 		)
 		(fp_arc
-			(start -7 -6.6)
-			(mid -6.882843 -6.882843)
-			(end -6.6 -7)
+			(start 6.6 -7)
+			(mid 6.882843 -6.882843)
+			(end 7 -6.6)
+			(stroke
+				(width 0.12)
+				(type solid)
+			)
+			(layer "Edge.Cuts")
+		)
+		(fp_arc
+			(start -6.6 7)
+			(mid -6.882843 6.882843)
+			(end -7 6.6)
 			(stroke
 				(width 0.12)
@@
 			(layer "Edge.Cuts")
 		)
-		(fp_arc
-			(start 6.6 -7)
-			(mid 6.882843 -6.882843)
-			(end 7 -6.6)
+		(fp_poly
+			(pts
+				(xy -11.875 -9.5) (xy 11.875 -9.5) (xy 11.875 9.5) (xy -11.875 9.5)
+			)
 			(stroke
 				(width 0.12)
 				(type solid)
 			)
-			(layer "Edge.Cuts")
+			(fill no)
+			(layer "User.2")
 		)
 		(fp_poly
@@
 		)
 		(fp_text user "${REFERENCE}"
-			(at 0 -8.199999 340)
+			(at 0 -8.199999 70)
 			(layer "F.Fab")
 			(effects
@@
 		)
 		(embedded_fonts no)
-		(model "/Users/gp/Downloads/KS33-low profile switch and stabilzier.stp"
-			(hide yes)
-			(offset
-				(xyz 0 0 -3)
-			)
-			(scale
-				(xyz 1 1 1)
-			)
-			(rotate
-				(xyz -0 -0 -0)
-			)
-		)
 	)
 	(footprint "tmr-lib:Switch_Cutout"
@@
 		(tags "Cherry MX Keyboard Keyswitch Switch PCB Cutout 1.00u")
 		(property "Reference" "S62"
-			(at 0.1 -6.1 340)
+			(at 0.100001 -6.1 340)
 			(layer "F.SilkS")
 			(hide yes)
@@
 	(footprint "tmr-lib:MountingHole_1.8mm_M1.6"
 		(layer "F.Cu")
-		(at 104.5 76)
+		(at 104.5 75)
 		(descr "Mounting Hole 2.2mm, no annular, M2")
 		(tags "mounting hole 2.2mm no annular m2")
@@
 		(tags "Cherry MX Keyboard Keyswitch Switch PCB Cutout 1.00u")
 		(property "Reference" "S30"
-			(at 0.1 -6.1 0)
+			(at 0.099999 -6.099999 0)
 			(layer "F.SilkS")
 			(hide yes)
@@
 		)
 		(property "Value" "SWHole"
-			(at 0.1 8.5 0)
+			(at 0.099999 8.5 0)
 			(layer "F.Fab")
 			(effects
@@
 		(duplicate_pad_numbers_are_jumpers no)
 		(fp_line
-			(start -7 -6.6)
+			(start -7 -6.600001)
 			(end -7 6.6)
 			(stroke
@@
 		)
 		(fp_line
-			(start -6.6 -7)
-			(end 6.6 -7)
+			(start -6.600001 7)
+			(end 6.6 7)
 			(stroke
 				(width 0.12)
@@
 		)
 		(fp_line
-			(start -6.6 7)
-			(end 6.6 7)
+			(start -6.6 -7)
+			(end 6.600001 -7)
 			(stroke
 				(width 0.12)
@@
 		(fp_line
 			(start 7 -6.6)
-			(end 7 6.6)
+			(end 7 6.600001)
 			(stroke
 				(width 0.12)
@@
 		)
 		(fp_arc
-			(start -7 -6.6)
-			(mid -6.882843 -6.882843)
+			(start -7 -6.600001)
+			(mid -6.882844 -6.882843)
 			(end -6.6 -7)
 			(stroke
@@
 		)
 		(fp_arc
-			(start -6.6 7)
-			(mid -6.882843 6.882843)
+			(start -6.600001 7)
+			(mid -6.882843 6.882844)
 			(end -7 6.6)
 			(stroke
@@
 		)
 		(fp_arc
-			(start 6.6 -7)
-			(mid 6.882843 -6.882843)
+			(start 6.600001 -7)
+			(mid 6.882843 -6.882844)
 			(end 7 -6.6)
 			(stroke
@@
 		)
 		(fp_arc
-			(start 7 6.6)
-			(mid 6.882843 6.882843)
+			(start 7 6.600001)
+			(mid 6.882844 6.882843)
 			(end 6.6 7)
 			(stroke
@@
 			(layer "Edge.Cuts")
 		)
-		(fp_rect
-			(start 11.875 -9.5)
-			(end -11.875 9.5)
+		(fp_poly
+			(pts
+				(xy -11.875001 -9.5) (xy 11.875 -9.5) (xy 11.875001 9.5) (xy -11.875 9.5)
+			)
 			(stroke
 				(width 0.12)
@@
 			(layer "User.2")
 		)
-		(fp_rect
-			(start 9.5 -9.5)
-			(end -9.5 9.5)
+		(fp_poly
+			(pts
+				(xy -9.499998 -9.500001) (xy 9.500001 -9.499998) (xy 9.499998 9.500001) (xy -9.500001 9.499998)
+			)
 			(stroke
 				(width 0.12)
@@
 		)
 		(fp_text user "${REFERENCE}"
-			(at 0 -8.2 0)
+			(at -0.000001 -8.200001 0)
 			(layer "F.Fab")
 			(effects
@@
 	(footprint "tmr-lib:Switch_Cutout"
 		(layer "F.Cu")
-		(at 242.25 38)
+		(at 244.625 38)
 		(descr "Cherry MX keyswitch PCB Mount with 1.00u keycap")
 		(tags "Cherry MX Keyboard Keyswitch Switch PCB Cutout 1.00u")
@@
 	(footprint "tmr-lib:Switch_Cutout"
 		(layer "F.Cu")
-		(at 263.625 38)
+		(at 266 38)
 		(descr "Cherry MX keyswitch PCB Mount with 1.00u keycap")
 		(tags "Cherry MX Keyboard Keyswitch Switch PCB Cutout 1.00u")

Commit message: M  hardware/nRF54LM20_TMR2615/border.py M  hardware/nRF54LM20_TMR2615/pcb/pcb.kicad_pcb M  hardware/nRF54LM20_TMR2615/pcb/pcb.kicad_prl M  hardware/nRF54LM20_TMR2615/placefp.py M  hardware/nRF54LM20_TMR2615/swplate/swplate.kicad_pcb
Parts:
- moved Hs7 5.00 mm to (174.0, 72.0)
- moved Hs6 4.53 mm to (104.0, 70.5)
