File: hardware/nRF54LM20_TMR2615/swplate/swplate.kicad_pcb (KiCad board)
At the start: 2 copper layers, 316.4 x 200.6 mm, 105 parts, among them M1 Minew_ME54BS13_V1.0, SW1 SW_Hole, SW2 SW_Hole

Commit message: M  hardware/nRF54LM20_TMR2615/layout_tools/border.py M  hardware/nRF54LM20_TMR2615/layout_tools/placefp.py M  hardware/nRF54LM20_TMR2615/pcb/pcb.kicad_pcb M  hardware/nRF54LM20_TMR2615/pcb/pcb.kicad_prl M  hardware/nRF54LM20_TMR2615/pcb/pcb.kicad_pro M  hardware/nRF54LM20_TMR2615/pcb/pcb.kicad_sch M  hardware/nRF54LM20_TMR2615/pcb/switch.kicad_sch M  hardware/nRF54LM20_TMR2615/swplate/swplate.kicad_pcb M  hardware/nRF54LM20_TMR2615/swplate/swplate.kicad_sch
Parts:
- removed H16: MountingHole, tmr-lib:MountingHole_3.2mm_M3_Heatsink_3.6mm
- moved H8 308.7 mm to (-6.95, 122.8)
- moved H12 298.7 mm to (287.4, 122.8)
- moved H7 120.9 mm to (295.5, 61.0)
- moved H13 78.5 mm to (209.1, 127.5)
- moved H15 78.4 mm to (287.4, 173.2)
- moved H9 73.6 mm to (66.5, 127.5)
- moved H11 73.4 mm to (-6.95, 173.2)
- moved H6 45.7 mm to (137.8, 91.2)
- moved H10 45.7 mm to (66.5, 173.2)
- moved H14 45.7 mm to (209.1, 173.2)
Other:
- outline, holes or cut-outs redrawn

Commit message: M  hardware/nRF54LM20_TMR2615/layout_tools/border.py M  hardware/nRF54LM20_TMR2615/layout_tools/placefp.py M  hardware/nRF54LM20_TMR2615/pcb/pcb.kicad_pcb M  hardware/nRF54LM20_TMR2615/pcb/pcb.kicad_prl M  hardware/nRF54LM20_TMR2615/pcb/pcb.kicad_pro M  hardware/nRF54LM20_TMR2615/pcb/pcb.kicad_sch M  hardware/nRF54LM20_TMR2615/swplate/swplate.kicad_pcb M  hardware/nRF54LM20_TMR2615/swplate/swplate.kicad_pro M  hardware/nRF54LM20_TMR2615/swplate/swplate.kicad_sch M  hardware/nRF54LM20_TMR2615/tmr-footprints/SMTSO_M1.6.kicad_mod
Parts:
- added JTAG1: Conn_ARM_JTAG_SWD_10, tmr-lib:SAMTEC-CLP-105-02-X-D-A, F.Cu at (180.5, -12.0)
Other:
- outline, holes or cut-outs redrawn
