File: hardware/nRF54LM20_TMR2615/swplate/swplate.kicad_sch (KiCad schematic)
At the start: 103 parts, among them M1 Minew_ME54BS13_V1.0

Commit message: A  hardware/nRF54LM20_TMR2615/cohr M  hardware/nRF54LM20_TMR2615/pcb/pcb.kicad_pcb M  hardware/nRF54LM20_TMR2615/pcb/pcb.kicad_prl M  hardware/nRF54LM20_TMR2615/placefp.py M  hardware/nRF54LM20_TMR2615/swplate/swplate.kicad_pcb M  hardware/nRF54LM20_TMR2615/swplate/swplate.kicad_sch
Parts:
- S63: footprint tmr-lib:Switch_Cutout -> tmr-lib:Switch_Cutout_1.25u
Changed lines of the file:
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@@
 			)
 		)
-		(property "Footprint" "tmr-lib:Switch_Cutout"
+		(property "Footprint" "tmr-lib:Switch_Cutout_1.25u"
 			(at 67.31 76.2 0)
 			(hide yes)

Commit message: M  hardware/nRF54LM20_TMR2615/pcb/pcb.kicad_pcb M  hardware/nRF54LM20_TMR2615/pcb/pcb.kicad_prl M  hardware/nRF54LM20_TMR2615/swplate/swplate.kicad_pcb M  hardware/nRF54LM20_TMR2615/swplate/swplate.kicad_pro M  hardware/nRF54LM20_TMR2615/swplate/swplate.kicad_sch A  hardware/nRF54LM20_TMR2615/tmr-footprints/SW_CK_PTS530_4.5x4.5x0.55mm_holeonly.kicad_mod
Parts:
- added SW1, SW2: SW_Hole, tmr-lib:SW_CK_PTS530_4.5x4.5x0.55mm_holeonly, symbol tmr-lib:JLC_Order_Num
Changed lines of the file:
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@@
+	)
+	(symbol
+		(lib_name "JLC_Order_Num_2")
+		(lib_id "tmr-lib:JLC_Order_Num")
+		(at 124.46 101.6 0)
+		(unit 1)
+		(body_style 1)
+		(exclude_from_sim no)
+		(in_bom yes)
+		(on_board yes)
+		(in_pos_files yes)
+		(dnp no)
+		(fields_autoplaced yes)
+		(property "Reference" "SW1"
+			(at 128.27 100.3299 0)
+			(show_name no)
+			(do_not_autoplace no)
+			(effects
+				(font
+					(size 1.27 1.27)
+				)
+				(justify left)
+			)
+		)
+		(property "Value" "SW_Hole"
+			(at 128.27 102.8699 0)
+			(show_name no)
+			(do_not_autoplace no)
+			(effects
+				(font
+					(size 1.27 1.27)
+				)
+				(justify left)
+			)
+		)
+		(property "Footprint" "tmr-lib:SW_CK_PTS530_4.5x4.5x0.55mm_holeonly"
+			(at 124.46 101.6 0)
+			(hide yes)
+			(show_name no)
+			(do_not_autoplace no)
+			(effects
+				(font
+					(size 1.27 1.27)
+				)
+			)
+		)
+		(property "Datasheet" ""
+			(at 124.46 101.6 0)
+			(hide yes)
+			(show_name no)
+			(do_not_autoplace no)
+			(effects
+				(font
+					(size 1.27 1.27)
+				)
+			)
+		)
+		(property "Description" ""
+			(at 124.46 101.6 0)
+			(hide yes)
+			(show_name no)
+			(do_not_autoplace no)
+			(effects
+				(font
+					(size 1.27 1.27)
+				)
+			)
+		)
+		(instances
+			(project "swplate"
+				(path "/4c67809e-1748-4898-89f6-ff92314048f2"
+					(reference "SW1")
+					(unit 1)
+				)
+			)
+		)
 	)
 	(symbol
@@
 					(unit 1)
 				)
+			)
+		)
+	)
+	(symbol
+		(lib_name "JLC_Order_Num_2")
+		(lib_id "tmr-lib:JLC_Order_Num")
+		(at 143.51 101.6 0)
+		(unit 1)
+		(body_style 1)
+		(exclude_from_sim no)
+		(in_bom yes)
+		(on_board yes)
+		(in_pos_files yes)
+		(dnp no)
+		(fields_autoplaced yes)
+		(property "Reference" "SW2"
+			(at 147.32 100.3299 0)
+			(show_name no)
+			(do_not_autoplace no)
+			(effects
+				(font
+					(size 1.27 1.27)
+				)
+				(justify left)
+			)
+		)
+		(property "Value" "SW_Hole"
+			(at 147.32 102.8699 0)
+			(show_name no)
+			(do_not_autoplace no)
+			(effects
+				(font
+					(size 1.27 1.27)
+				)
+				(justify left)
+			)
+		)
+		(property "Footprint" "tmr-lib:SW_CK_PTS530_4.5x4.5x0.55mm_holeonly"
+			(at 143.51 101.6 0)
+			(hide yes)
+			(show_name no)
+			(do_not_autoplace no)
+			(effects
+				(font
+					(size 1.27 1.27)
+				)
+			)
+		)
+		(property "Datasheet" ""
+			(at 143.51 101.6 0)
+			(hide yes)
+			(show_name no)
+			(do_not_autoplace no)
+			(effects
+				(font
+					(size 1.27 1.27)
+				)
+			)
+		)
+		(property "Description" ""
+			(at 143.51 101.6 0)
+			(hide yes)
+			(show_name no)
+			(do_not_autoplace no)
+			(effects
+				(font
+					(size 1.27 1.27)
+				)
+			)
+		)
+		(instances
+			(project "swplate"
+				(path "/4c67809e-1748-4898-89f6-ff92314048f2"
+					(reference "SW2")
+					(unit 1)
+				)

Commit message: M  hardware/nRF54LM20_TMR2615/swplate/swplate.kicad_pcb M  hardware/nRF54LM20_TMR2615/swplate/swplate.kicad_sch A  hardware/nRF54LM20_TMR2615/tmr-footprints/MountingHole_3.2mm_M3_Heatsink_3.6mm.kicad_mod
Parts:
- H1, H10, H11, H12, H13, H14, H15, H16, H2, H3, H4, H5, H6, H7, H8, H9: footprint tmr-lib:MountingHole_2.7mm_M2.5 -> tmr-lib:MountingHole_3.2mm_M3_Heatsink_3.6mm
Changed lines of the file:
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@@
 			)
 		)
-		(property "Footprint" "tmr-lib:MountingHole_2.7mm_M2.5"
+		(property "Footprint" "tmr-lib:MountingHole_3.2mm_M3_Heatsink_3.6mm"
 			(at 76.2 171.45 0)
 			(hide yes)
@@
 			)
 		)
-		(property "Footprint" "tmr-lib:MountingHole_2.7mm_M2.5"
+		(property "Footprint" "tmr-lib:MountingHole_3.2mm_M3_Heatsink_3.6mm"
 			(at 38.1 160.02 0)
 			(hide yes)
@@
 			)
 		)
-		(property "Footprint" "tmr-lib:MountingHole_2.7mm_M2.5"
+		(property "Footprint" "tmr-lib:MountingHole_3.2mm_M3_Heatsink_3.6mm"
 			(at 19.05 181.61 0)
 			(hide yes)
@@
 			)
 		)
-		(property "Footprint" "tmr-lib:MountingHole_2.7mm_M2.5"
+		(property "Footprint" "tmr-lib:MountingHole_3.2mm_M3_Heatsink_3.6mm"
 			(at 38.1 171.45 0)
 			(hide yes)
@@
 			)
 		)
-		(property "Footprint" "tmr-lib:MountingHole_2.7mm_M2.5"
+		(property "Footprint" "tmr-lib:MountingHole_3.2mm_M3_Heatsink_3.6mm"
 			(at 76.2 191.77 0)
 			(hide yes)
@@
 			)
 		)
-		(property "Footprint" "tmr-lib:MountingHole_2.7mm_M2.5"
+		(property "Footprint" "tmr-lib:MountingHole_3.2mm_M3_Heatsink_3.6mm"
 			(at 19.05 191.77 0)
 			(hide yes)
@@
 			)
 		)
-		(property "Footprint" "tmr-lib:MountingHole_2.7mm_M2.5"
+		(property "Footprint" "tmr-lib:MountingHole_3.2mm_M3_Heatsink_3.6mm"
 			(at 57.15 191.77 0)
 			(hide yes)
@@
 			)
 		)
-		(property "Footprint" "tmr-lib:MountingHole_2.7mm_M2.5"
+		(property "Footprint" "tmr-lib:MountingHole_3.2mm_M3_Heatsink_3.6mm"
 			(at 38.1 181.61 0)
 			(hide yes)
@@
 			)
 		)
-		(property "Footprint" "tmr-lib:MountingHole_2.7mm_M2.5"
+		(property "Footprint" "tmr-lib:MountingHole_3.2mm_M3_Heatsink_3.6mm"
 			(at 19.05 160.02 0)
 			(hide yes)
@@
 			)
 		)
-		(property "Footprint" "tmr-lib:MountingHole_2.7mm_M2.5"
+		(property "Footprint" "tmr-lib:MountingHole_3.2mm_M3_Heatsink_3.6mm"
 			(at 57.15 171.45 0)
 			(hide yes)
@@
 			)
 		)
-		(property "Footprint" "tmr-lib:MountingHole_2.7mm_M2.5"
+		(property "Footprint" "tmr-lib:MountingHole_3.2mm_M3_Heatsink_3.6mm"
 			(at 57.15 160.02 0)
 			(hide yes)
@@
 			)
 		)
-		(property "Footprint" "tmr-lib:MountingHole_2.7mm_M2.5"
+		(property "Footprint" "tmr-lib:MountingHole_3.2mm_M3_Heatsink_3.6mm"
 			(at 38.1 191.77 0)
 			(hide yes)
@@
 			)
 		)
-		(property "Footprint" "tmr-lib:MountingHole_2.7mm_M2.5"
+		(property "Footprint" "tmr-lib:MountingHole_3.2mm_M3_Heatsink_3.6mm"
 			(at 76.2 181.61 0)
 			(hide yes)
@@
 			)
 		)
-		(property "Footprint" "tmr-lib:MountingHole_2.7mm_M2.5"
+		(property "Footprint" "tmr-lib:MountingHole_3.2mm_M3_Heatsink_3.6mm"
 			(at 57.15 181.61 0)
 			(hide yes)
@@
 			)
 		)
-		(property "Footprint" "tmr-lib:MountingHole_2.7mm_M2.5"
+		(property "Footprint" "tmr-lib:MountingHole_3.2mm_M3_Heatsink_3.6mm"
 			(at 19.05 171.45 0)
 			(hide yes)
@@
 			)
 		)
-		(property "Footprint" "tmr-lib:MountingHole_2.7mm_M2.5"
+		(property "Footprint" "tmr-lib:MountingHole_3.2mm_M3_Heatsink_3.6mm"
 			(at 76.2 160.02 0)
 			(hide yes)

Commit message: M  hardware/nRF54LM20_TMR2615/layout_tools/border.py M  hardware/nRF54LM20_TMR2615/layout_tools/placefp.py M  hardware/nRF54LM20_TMR2615/pcb/pcb.kicad_pcb M  hardware/nRF54LM20_TMR2615/pcb/pcb.kicad_prl M  hardware/nRF54LM20_TMR2615/pcb/pcb.kicad_pro M  hardware/nRF54LM20_TMR2615/pcb/pcb.kicad_sch M  hardware/nRF54LM20_TMR2615/pcb/switch.kicad_sch M  hardware/nRF54LM20_TMR2615/swplate/swplate.kicad_pcb M  hardware/nRF54LM20_TMR2615/swplate/swplate.kicad_sch
Parts:
- removed H16: MountingHole, tmr-lib:MountingHole_3.2mm_M3_Heatsink_3.6mm, symbol Mechanical:MountingHole
Changed lines of the file:
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@@
-	)
-	(symbol
-		(lib_id "Mechanical:MountingHole")
-		(at 76.2 191.77 0)
-		(unit 1)
-		(body_style 1)
-		(exclude_from_sim no)
-		(in_bom no)
-		(on_board yes)
-		(in_pos_files yes)
-		(dnp no)
-		(fields_autoplaced yes)
-		(property "Reference" "H16"
-			(at 78.74 190.4999 0)
-			(show_name no)
-			(do_not_autoplace no)
-			(effects
-				(font
-					(size 1.27 1.27)
-				)
-				(justify left)
-			)
-		)
-		(property "Value" "MountingHole"
-			(at 78.74 193.0399 0)
-			(show_name no)
-			(do_not_autoplace no)
-			(effects
-				(font
-					(size 1.27 1.27)
-				)
-				(justify left)
-			)
-		)
-		(property "Footprint" "tmr-lib:MountingHole_3.2mm_M3_Heatsink_3.6mm"
-			(at 76.2 191.77 0)
-			(hide yes)
-			(show_name no)
-			(do_not_autoplace no)
-			(effects
-				(font
-					(size 1.27 1.27)
-				)
-			)
-		)
-		(property "Datasheet" ""
-			(at 76.2 191.77 0)
-			(hide yes)
-			(show_name no)
-			(do_not_autoplace no)
-			(effects
-				(font
-					(size 1.27 1.27)
-				)
-			)
-		)
-		(property "Description" "Mounting Hole without connection"
-			(at 76.2 191.77 0)
-			(hide yes)
-			(show_name no)
-			(do_not_autoplace no)
-			(effects
-				(font
-					(size 1.27 1.27)
-				)
-			)
-		)
-		(instances
-			(project "swplate"
-				(path "/4c67809e-1748-4898-89f6-ff92314048f2"
-					(reference "H16")
-					(unit 1)
-				)
-			)
-		)
 	)
 	(symbol

Commit message: M  hardware/nRF54LM20_TMR2615/layout_tools/border.py M  hardware/nRF54LM20_TMR2615/layout_tools/placefp.py M  hardware/nRF54LM20_TMR2615/pcb/pcb.kicad_pcb M  hardware/nRF54LM20_TMR2615/pcb/pcb.kicad_prl M  hardware/nRF54LM20_TMR2615/pcb/pcb.kicad_pro M  hardware/nRF54LM20_TMR2615/pcb/pcb.kicad_sch M  hardware/nRF54LM20_TMR2615/swplate/swplate.kicad_pcb M  hardware/nRF54LM20_TMR2615/swplate/swplate.kicad_pro M  hardware/nRF54LM20_TMR2615/swplate/swplate.kicad_sch M  hardware/nRF54LM20_TMR2615/tmr-footprints/SMTSO_M1.6.kicad_mod
Parts:
- added JTAG1: Conn_ARM_JTAG_SWD_10, tmr-lib:SAMTEC-CLP-105-02-X-D-A, symbol Connector:Conn_ARM_JTAG_SWD_10
Connections:
- new net: JTAG1.3 (GND), JTAG1.5 (GND)
- new net VDD_nRF: JTAG1.1 (VTref)
- no-connect marks 97 -> 104
Changed lines of the file:
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@@
 	)
 	(no_connect
+		(at 254 39.37)
+	)
+	(no_connect
 		(at 182.88 121.92)
 	)
@@
 	)
 	(no_connect
+		(at 254 29.21)
+	)
+	(no_connect
 		(at 149.86 160.02)
 	)
@@
 	)
 	(no_connect
+		(at 254 41.91)
+	)
+	(no_connect
 		(at 281.94 124.46)
 	)
@@
 	)
 	(no_connect
+		(at 241.3 52.07)
+	)
+	(no_connect
 		(at 251.46 162.56)
 	)
@@
 	)
 	(no_connect
+		(at 254 34.29)
+	)
+	(no_connect
 		(at 182.88 119.38)
 	)
@@
 	)
 	(no_connect
+		(at 238.76 52.07)
+	)
+	(no_connect
 		(at 269.24 162.56)
 	)
@@
 	)
 	(no_connect
+		(at 254 36.83)
+	)
+	(no_connect
 		(at 210.82 76.2)
 	)
@@
 		(at 149.86 147.32)
 	)
+	(label "VDD_nRF"
+		(at 241.3 21.59 180)
+		(effects
+			(font
+				(size 1.27 1.27)
+			)
+			(justify right bottom)
+		)
+	)
 	(symbol
 		(lib_id "tmr-lib:SWHole")
@@
 					(unit 1)
 				)
+			)
+		)
+	)
+	(symbol
+		(lib_id "Connector:Conn_ARM_JTAG_SWD_10")
+		(at 241.3 36.83 0)
+		(unit 1)
+		(body_style 1)
+		(exclude_from_sim no)
+		(in_bom yes)
+		(on_board yes)
+		(in_pos_files yes)
+		(dnp no)
+		(fields_autoplaced yes)
+		(property "Reference" "JTAG1"
+			(at 229.87 35.5599 0)
+			(show_name no)
+			(do_not_autoplace no)
+			(effects
+				(font
+					(size 1.27 1.27)
+				)
+				(justify right)
+			)
+		)
+		(property "Value" "Conn_ARM_JTAG_SWD_10"
+			(at 229.87 38.0999 0)
+			(show_name no)
+			(do_not_autoplace no)
+			(effects
+				(font
+					(size 1.27 1.27)
+				)
+				(justify right)
+			)
+		)
+		(property "Footprint" "tmr-lib:SAMTEC-CLP-105-02-X-D-A"
+			(at 241.3 36.83 0)
+			(hide yes)
+			(show_name no)
+			(do_not_autoplace no)
+			(effects
+				(font
+					(size 1.27 1.27)
+				)
+			)
+		)
+		(property "Datasheet" "http://infocenter.arm.com/help/topic/com.arm.doc.ddi0314h/DDI0314H_coresight_components_trm.pdf"
+			(at 232.41 68.58 90)
+			(hide yes)
+			(show_name no)
+			(do_not_autoplace no)
+			(effects
+				(font
+					(size 1.27 1.27)
+				)
+			)
+		)
+		(property "Description" "Cortex Debug Connector, standard ARM Cortex-M SWD and JTAG interface"
+			(at 241.3 36.83 0)
+			(hide yes)
+			(show_name no)
+			(do_not_autoplace no)
+			(effects
+				(font
+					(size 1.27 1.27)
+				)
+			)
+		)
+		(property "LCSC" "C6882278"
+			(at 241.3 36.83 0)
+			(hide yes)
+			(show_name no)
+			(do_not_autoplace no)
+			(effects
+				(font
+					(size 1.27 1.27)
+				)
+			)
+		)
+		(pin "7"
+		)
+		(pin "9"
+		)
+		(pin "1"
+		)
+		(pin "3"
+		)
+		(pin "5"
+		)
+		(pin "10"
+		)
+		(pin "4"
+		)
+		(pin "2"
+		)
+		(pin "6"
+		)
+		(pin "8"
+		)
+		(instances
+			(project "swplate"
+				(path "/4c67809e-1748-4898-89f6-ff92314048f2"
+					(reference "JTAG1")
+					(unit 1)
+				)
