File: hardware/nRF54LM20_TMR2615/pcb/pcb.kicad_pcb (KiCad board)
At the start: 2 copper layers, 299.2 x 119.9 mm, 426 parts, among them M1 Minew_ME54BS13_V1.0, SW1 SW_DIP_x01, SW2 SW_DIP_x01

Commit message: A  hardware/nRF54LM20_TMR2615/Bezier.py D  hardware/nRF54LM20_TMR2615/border.py M  hardware/nRF54LM20_TMR2615/layout_tools/placefp.py A  hardware/nRF54LM20_TMR2615/pcb/pcb-unsaved-export-VXg1D0.kicad_prl M  hardware/nRF54LM20_TMR2615/pcb/pcb.kicad_pcb M  hardware/nRF54LM20_TMR2615/pcb/pcb.kicad_prl M  hardware/nRF54LM20_TMR2615/pcb/pcb.kicad_pro M  hardware/nRF54LM20_TMR2615/pcb/pcb.kicad_sch D  hardware/nRF54LM20_TMR2615/placefp.py A  hardware/nRF54LM20_TMR2615/swplate/swplate-unsaved-export-pUvE8F.kicad_prl M  hardware/nRF54LM20_TMR2615/swplate/swplate.kicad_pcb M  hardware/nRF54LM20_TMR2615/swplate/swplate.kicad_pro A  hardware/nRF54LM20_TMR2615/tmr-footprints/SW_CK_PTS530_4.5x4.5x0.55mm.kicad_mod M  hardware/nRF54LM20_TMR2615/tmr-symbols.kicad_sym
Parts:
- SW1, SW2: value SW_DIP_x01 -> SW_CK_PTS530; footprint tmr-lib:Aliexpress_SW_TACT_4x4x1.5mm -> tmr-lib:SW_CK_PTS530_4.5x4.5x0.55mm; moved to F.Cu
- moved SW1 187.3 mm to (45.6, 103.3), turned to 0 degrees
- moved SW2 154.2 mm to (140.4, 114.9), turned to 0 degrees
Connections:
- SW1 pad 2: /NRESET -> GND
- SW2 pad 2: Net-(PMIC1-SHPHLD) -> GND
