File: hardware/nRF54LM20_TMR2615/pcb/pcb.kicad_pcb (KiCad board)
At the start: 2 copper layers, 297.2 x 119.5 mm, 426 parts, among them M1 Minew_ME54BS13_V1.0, SW1 SW_CK_PTS530, SW2 SW_CK_PTS530

Commit message: M  hardware/nRF54LM20_TMR2615/layout_tools/border.py M  hardware/nRF54LM20_TMR2615/layout_tools/placefp.py M  hardware/nRF54LM20_TMR2615/pcb/pcb.kicad_pcb M  hardware/nRF54LM20_TMR2615/pcb/pcb.kicad_prl M  hardware/nRF54LM20_TMR2615/pcb/pcb.kicad_pro M  hardware/nRF54LM20_TMR2615/pcb/pcb.kicad_sch M  hardware/nRF54LM20_TMR2615/pcb/switch.kicad_sch M  hardware/nRF54LM20_TMR2615/swplate/swplate.kicad_pcb M  hardware/nRF54LM20_TMR2615/swplate/swplate.kicad_sch
Parts:
- C1, C10, C19, C2, C20, C21, C22, C8, C9: footprint Capacitor_SMD:C_0402_1005Metric -> Capacitor_SMD:C_0603_1608Metric
- C11: value 0.1uF -> .1uF
- C12: moved to B.Cu
- D1, D10, D11, D12, D13, D14, D15, D16, D17, D18, D19, D2, D20, D21, D22, D23, D24, D25, D26, D27, D28, D29, D3, D30, D31, D32, D33, D34, D35, D36, D37, D38, D39, D4, D40, D41, D42, D43, D44, D45, D46, D47, D48, D49, D5, D50, D51, D52, D53, D54, D55, D56, D57, D58, D59, D6, D60, D61, D62, D63, D64, D65, D66, D67, D68, D69, D7, D70, D71, D72, D8, D9: value Green LED -> LED
- moved C12 9.60 mm to (19.5, -12.3), turned to 180 degrees
- moved C1 0.40 mm to (151.4, -7.31)
- moved C10 0.34 mm to (29.4, 21.8)
- moved C22 0.30 mm to (29.4, 23.3)
- moved C20 0.18 mm to (36.6, 14.0)
Routing:
- net GND: track 668.1 -> 688.6 mm, vias 110 -> 112
- net /GPIO_X: track 162.3 -> 164.5 mm
- net /VDD_nRF: track 220.8 -> 218.6 mm
- net /VSYS: track 162.9 -> 164.6 mm
- net /INT: track 164.6 -> 163.0 mm, vias 4 -> 6
- net Net-(PMIC1-VBUS): track 57.1 -> 58.6 mm, vias 3 -> 4
- net /SCL: track 182.4 -> 183.3 mm
- net /SDA: track 181.6 -> 182.5 mm
- net /SW0: track 842.4 -> 841.8 mm
- net /ANA_16: track 104.5 -> 105.1 mm
