File: hardware/nRF54LM20_TMR2615/pcb/pcb.kicad_pcb (KiCad board)
At the start: 2 copper layers, 297.2 x 119.5 mm, 426 parts, among them M1 Minew_ME54BS13_V1.0, SW1 SW_CK_PTS530, SW2 SW_CK_PTS530

Commit message: M  hardware/nRF54LM20_TMR2615/layout_tools/border.py M  hardware/nRF54LM20_TMR2615/layout_tools/placefp.py M  hardware/nRF54LM20_TMR2615/pcb/pcb.kicad_pcb M  hardware/nRF54LM20_TMR2615/pcb/pcb.kicad_prl M  hardware/nRF54LM20_TMR2615/pcb/pcb.kicad_pro M  hardware/nRF54LM20_TMR2615/pcb/pcb.kicad_sch M  hardware/nRF54LM20_TMR2615/swplate/swplate.kicad_pcb M  hardware/nRF54LM20_TMR2615/swplate/swplate.kicad_pro M  hardware/nRF54LM20_TMR2615/swplate/swplate.kicad_sch M  hardware/nRF54LM20_TMR2615/tmr-footprints/SMTSO_M1.6.kicad_mod
Parts:
- C11, C14, C15, C16, C17, C18, C3, C4, C5, C6, C7: value .1uF -> 0.1uF
- JTAG1: moved to F.Cu
- moved JTAG1 8.50 mm to (180.5, -12.0), turned to 180 degrees
Routing:
- net /VDD_nRF: track 218.6 -> 225.5 mm, vias 7 -> 6
- net /NRESET: track 52.5 -> 46.4 mm, vias 2 -> 3
- net /SWDIO: track 15.9 -> 21.6 mm, vias 2 -> 3
- net /SW0: track 841.8 -> 837.6 mm
- net /SWDCLK: track 14.6 -> 18.7 mm, vias 2 -> 1
- net VCCS: track 2745.0 -> 2747.7 mm
Other:
- outline, holes or cut-outs redrawn
