File: hardware/nRF54LM20_TMR2615/pcb/switch.kicad_sch (KiCad schematic)
At the start: 4 parts

Commit message: M  hardware/nRF54LM20_TMR2615/border.py D  hardware/nRF54LM20_TMR2615/cohr M  hardware/nRF54LM20_TMR2615/pcb/pcb.kicad_pcb M  hardware/nRF54LM20_TMR2615/pcb/pcb.kicad_pro M  hardware/nRF54LM20_TMR2615/pcb/pcb.kicad_sch M  hardware/nRF54LM20_TMR2615/pcb/switch.kicad_sch
Parts:
- renumbered Cvcc1 to Cvcc2, Cvout1 to Cvout2, S1 to S2, TMR1 to TMR2
Changed lines of the file:
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@@
 		(dnp no)
 		(fields_autoplaced yes)
-		(property "Reference" "Cvout1"
+		(property "Reference" "Cvout2"
 			(at 143.51 68.5862 0)
 			(show_name no)
@@
 		(dnp no)
 		(fields_autoplaced yes)
-		(property "Reference" "TMR1"
+		(property "Reference" "TMR2"
 			(at 123.19 63.4999 0)
 			(show_name no)
@@
 		(dnp no)
 		(fields_autoplaced yes)
-		(property "Reference" "#PWR04"
+		(property "Reference" "#PWR056"
 			(at 127 86.36 0)
 			(hide yes)
@@
 		(dnp no)
 		(fields_autoplaced yes)
-		(property "Reference" "Cvcc1"
+		(property "Reference" "Cvcc2"
 			(at 114.3 58.4262 0)
 			(show_name no)
@@
 		(dnp no)
 		(fields_autoplaced yes)
-		(property "Reference" "S1"
+		(property "Reference" "S2"
 			(at 104.14 64.7699 0)
 			(show_name no)

Commit message: M  hardware/nRF54LM20_TMR2615/layout_tools/border.py M  hardware/nRF54LM20_TMR2615/layout_tools/placefp.py M  hardware/nRF54LM20_TMR2615/pcb/pcb.kicad_pcb M  hardware/nRF54LM20_TMR2615/pcb/pcb.kicad_prl M  hardware/nRF54LM20_TMR2615/pcb/pcb.kicad_pro M  hardware/nRF54LM20_TMR2615/pcb/pcb.kicad_sch M  hardware/nRF54LM20_TMR2615/pcb/switch.kicad_sch M  hardware/nRF54LM20_TMR2615/swplate/swplate.kicad_pcb M  hardware/nRF54LM20_TMR2615/swplate/swplate.kicad_sch
Parts:
- Cvcc2: LCSC (none) -> C129131
- Cvout2: LCSC (none) -> C77177
- TMR2: LCSC (none) -> C9900212297
Changed lines of the file:
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@@
+			)
+		)
+		(property "LCSC" "C77177"
+			(at 140.97 69.85 0)
+			(hide yes)
+			(show_name no)
+			(do_not_autoplace no)
+			(effects
+				(font
+					(size 1.27 1.27)
+				)
 			)
 		)
@@
 			)
 		)
+		(property "LCSC" "C9900212297"
+			(at 129.54 64.77 0)
+			(hide yes)
+			(show_name no)
+			(do_not_autoplace no)
+			(effects
+				(font
+					(size 1.27 1.27)
+				)
+			)
+		)
 		(pin "3"
 		)
@@
 			(at 111.76 59.69 0)
 			(hide yes)
+			(show_name no)
+			(do_not_autoplace no)
+			(effects
+				(font
+					(size 1.27 1.27)
+				)
+			)
+		)
+		(property "LCSC" "C129131"
+			(at 111.76 59.69 0)
+			(hide yes)
