File: hardware/nRF54LM20_TMR2615/pcb/pcb.kicad_sch (KiCad schematic)
At the start: 138 parts, among them M1 Minew_ME54BS13_V1.0, SW1 SW_DIP_x01, SW2 SW_DIP_x01

Commit message: A  hardware/nRF54LM20_TMR2615/Bezier.py D  hardware/nRF54LM20_TMR2615/border.py M  hardware/nRF54LM20_TMR2615/layout_tools/placefp.py A  hardware/nRF54LM20_TMR2615/pcb/pcb-unsaved-export-VXg1D0.kicad_prl M  hardware/nRF54LM20_TMR2615/pcb/pcb.kicad_pcb M  hardware/nRF54LM20_TMR2615/pcb/pcb.kicad_prl M  hardware/nRF54LM20_TMR2615/pcb/pcb.kicad_pro M  hardware/nRF54LM20_TMR2615/pcb/pcb.kicad_sch D  hardware/nRF54LM20_TMR2615/placefp.py A  hardware/nRF54LM20_TMR2615/swplate/swplate-unsaved-export-pUvE8F.kicad_prl M  hardware/nRF54LM20_TMR2615/swplate/swplate.kicad_pcb M  hardware/nRF54LM20_TMR2615/swplate/swplate.kicad_pro A  hardware/nRF54LM20_TMR2615/tmr-footprints/SW_CK_PTS530_4.5x4.5x0.55mm.kicad_mod M  hardware/nRF54LM20_TMR2615/tmr-symbols.kicad_sym
Parts:
- removed SW1, SW2: SW_DIP_x01, tmr-lib:Aliexpress_SW_TACT_4x4x1.5mm, symbol Switch:SW_DIP_x01
- added SW1, SW2: SW_CK_PTS530, tmr-lib:SW_CK_PTS530_4.5x4.5x0.55mm, symbol tmr-lib:SW_CK_PTS530
Connections:
- net GND: now also SW1.1, SW1.2, SW2.1, SW2.2
- net NRESET: now also SW1.3 (K), SW1.4 (A)
- net at PMIC1.15 (SHPHLD): now also SW2.3 (K), SW2.4 (A)

Commit message: M  hardware/nRF54LM20_TMR2615/pcb/pcb.kicad_pcb M  hardware/nRF54LM20_TMR2615/pcb/pcb.kicad_prl M  hardware/nRF54LM20_TMR2615/pcb/pcb.kicad_sch M  hardware/nRF54LM20_TMR2615/tmr-footprints/TMR2615-DFN-3L-1.6x1.6.kicad_mod
Parts:
- C1, C10, C12, C13, C19, C2, C20, C21, C22, C23, C24, C25, C26, C8, C9: footprint Capacitor_SMD:C_0603_1608Metric -> Capacitor_SMD:C_0402_1005Metric
Changed lines of the file:
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@@
 			)
 		)
-		(property "Footprint" "Capacitor_SMD:C_0603_1608Metric"
+		(property "Footprint" "Capacitor_SMD:C_0402_1005Metric"
 			(at 491.49 288.29 0)
 			(hide yes)
@@
 			)
 		)
-		(property "Footprint" "Capacitor_SMD:C_0603_1608Metric"
+		(property "Footprint" "Capacitor_SMD:C_0402_1005Metric"
 			(at 464.82 223.52 0)
 			(hide yes)
@@
 			)
 		)
-		(property "Footprint" "Capacitor_SMD:C_0603_1608Metric"
+		(property "Footprint" "Capacitor_SMD:C_0402_1005Metric"
 			(at 481.33 245.11 0)
 			(hide yes)
@@
 			)
 		)
-		(property "Footprint" "Capacitor_SMD:C_0603_1608Metric"
+		(property "Footprint" "Capacitor_SMD:C_0402_1005Metric"
 			(at 236.22 340.36 0)
 			(hide yes)
@@
 			)
 		)
-		(property "Footprint" "Capacitor_SMD:C_0603_1608Metric"
+		(property "Footprint" "Capacitor_SMD:C_0402_1005Metric"
 			(at 251.46 408.94 0)
 			(hide yes)
@@
 			)
 		)
-		(property "Footprint" "Capacitor_SMD:C_0603_1608Metric"
+		(property "Footprint" "Capacitor_SMD:C_0402_1005Metric"
 			(at 207.01 370.84 0)
 			(hide yes)
@@
 			)
 		)
-		(property "Footprint" "Capacitor_SMD:C_0603_1608Metric"
+		(property "Footprint" "Capacitor_SMD:C_0402_1005Metric"
 			(at 482.6 313.69 0)
 			(hide yes)
@@
 			)
 		)
-		(property "Footprint" "Capacitor_SMD:C_0603_1608Metric"
+		(property "Footprint" "Capacitor_SMD:C_0402_1005Metric"
 			(at 492.76 274.32 0)
 			(hide yes)
@@
 			)
 		)
-		(property "Footprint" "Capacitor_SMD:C_0603_1608Metric"
+		(property "Footprint" "Capacitor_SMD:C_0402_1005Metric"
 			(at 454.66 223.52 0)
 			(hide yes)
@@
 			)
 		)
-		(property "Footprint" "Capacitor_SMD:C_0603_1608Metric"
+		(property "Footprint" "Capacitor_SMD:C_0402_1005Metric"
 			(at 474.98 223.52 0)
 			(hide yes)
@@
 			)
 		)
-		(property "Footprint" "Capacitor_SMD:C_0603_1608Metric"
+		(property "Footprint" "Capacitor_SMD:C_0402_1005Metric"
 			(at 436.88 99.06 0)
 			(hide yes)
@@
 			)
 		)
-		(property "Footprint" "Capacitor_SMD:C_0603_1608Metric"
+		(property "Footprint" "Capacitor_SMD:C_0402_1005Metric"
 			(at 259.08 353.06 0)
 			(hide yes)
@@
 			)
 		)
-		(property "Footprint" "Capacitor_SMD:C_0603_1608Metric"
+		(property "Footprint" "Capacitor_SMD:C_0402_1005Metric"
 			(at 492.76 261.62 0)
 			(hide yes)
@@
 			)
 		)
-		(property "Footprint" "Capacitor_SMD:C_0603_1608Metric"
+		(property "Footprint" "Capacitor_SMD:C_0402_1005Metric"
 			(at 394.97 245.11 0)
 			(hide yes)
@@
 			)
 		)
-		(property "Footprint" "Capacitor_SMD:C_0603_1608Metric"
+		(property "Footprint" "Capacitor_SMD:C_0402_1005Metric"
 			(at 312.42 116.84 0)
 			(hide yes)

Commit message: M  hardware/nRF54LM20_TMR2615/layout_tools/border.py M  hardware/nRF54LM20_TMR2615/layout_tools/placefp.py M  hardware/nRF54LM20_TMR2615/pcb/pcb.kicad_pcb M  hardware/nRF54LM20_TMR2615/pcb/pcb.kicad_prl M  hardware/nRF54LM20_TMR2615/pcb/pcb.kicad_pro M  hardware/nRF54LM20_TMR2615/pcb/pcb.kicad_sch M  hardware/nRF54LM20_TMR2615/pcb/switch.kicad_sch M  hardware/nRF54LM20_TMR2615/swplate/swplate.kicad_pcb M  hardware/nRF54LM20_TMR2615/swplate/swplate.kicad_sch
Parts:
- BAT1, BAT2, JLC1, Stb1, Stb2: now left out of the parts list
- C1, C10, C19, C2, C20, C8, C9: footprint Capacitor_SMD:C_0402_1005Metric -> Capacitor_SMD:C_0603_1608Metric; LCSC (none) -> C96446
- C11: value 0.1uF -> .1uF; LCSC (none) -> C129131
- C12, C13, C24, C25, C26: LCSC (none) -> C14445
- C14, C15, C16, C17, C18, C3, C4, C5, C6, C7: LCSC (none) -> C129131
- C21, C22: footprint Capacitor_SMD:C_0402_1005Metric -> Capacitor_SMD:C_0603_1608Metric; LCSC (none) -> C57895
- C23: LCSC (none) -> C710873
- D1, D10, D11, D12, D13, D14, D15, D16, D17, D18, D19, D2, D20, D21, D22, D23, D24, D25, D26, D27, D28, D29, D3, D30, D31, D32, D33, D34, D35, D36, D37, D38, D39, D4, D40, D41, D42, D43, D44, D45, D46, D47, D48, D49, D5, D50, D51, D52, D53, D54, D55, D56, D57, D58, D59, D6, D60, D61, D62, D63, D64, D65, D66, D67, D68, D69, D7, D70, D71, D72, D8, D9: value Green LED -> LED; LCSC (none) -> C401114
- Hs1, Hs10, Hs2, Hs3, Hs4, Hs5, Hs6, Hs7, Hs8, Hs9: LCSC (none) -> C2928167; now in the parts list
- JTAG1: LCSC (none) -> C6882278
- L1, L2: LCSC (none) -> C2049745
- LEDDR1: LCSC (none) -> C5220564
- M1: LCSC (none) -> C9900300294
- MUXA1, MUXA2: LCSC (none) -> C2673120
- MUXB1, MUXB2, MUXB3, MUXB4, MUXB5, MUXB6, MUXB7, MUXB8: LCSC (none) -> C2673274
- PMIC1: LCSC (none) -> C25346894
- R1, R2: LCSC (none) -> C25100
- R3, R4: LCSC (none) -> C25744
- Rvset1: LCSC (none) -> C25755
- Rvset2: LCSC (none) -> C25900
- SW1, SW2: LCSC (none) -> C221860

Commit message: M  hardware/nRF54LM20_TMR2615/layout_tools/border.py M  hardware/nRF54LM20_TMR2615/layout_tools/placefp.py M  hardware/nRF54LM20_TMR2615/pcb/pcb.kicad_pcb M  hardware/nRF54LM20_TMR2615/pcb/pcb.kicad_prl M  hardware/nRF54LM20_TMR2615/pcb/pcb.kicad_pro M  hardware/nRF54LM20_TMR2615/pcb/pcb.kicad_sch M  hardware/nRF54LM20_TMR2615/swplate/swplate.kicad_pcb M  hardware/nRF54LM20_TMR2615/swplate/swplate.kicad_pro M  hardware/nRF54LM20_TMR2615/swplate/swplate.kicad_sch M  hardware/nRF54LM20_TMR2615/tmr-footprints/SMTSO_M1.6.kicad_mod
Parts:
- C11, C14, C15, C16, C17, C18, C3, C4, C5, C6, C7: value .1uF -> 0.1uF
- Hs1, Hs10, Hs2, Hs3, Hs4, Hs5, Hs6, Hs7, Hs8, Hs9: LCSC C2928167 -> C42924166
Changed lines of the file:
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@@
 			)
 		)
-		(property "LCSC" "C2928167"
+		(property "LCSC" "C42924166"
 			(at 374.65 364.49 0)
 			(hide yes)
@@
 			)
 		)
-		(property "LCSC" "C2928167"
+		(property "LCSC" "C42924166"
 			(at 389.89 370.84 0)
 			(hide yes)
@@
 			)
 		)
-		(property "LCSC" "C2928167"
+		(property "LCSC" "C42924166"
 			(at 389.89 364.49 0)
 			(hide yes)
@@
 			)
 		)
-		(property "LCSC" "C2928167"
+		(property "LCSC" "C42924166"
 			(at 359.41 364.49 0)
 			(hide yes)
@@
 			)
 		)
-		(property "Value" ".1uF"
+		(property "Value" "0.1uF"
 			(at 227.3363 182.88 90)
 			(show_name no)
@@
 			)
 		)
-		(property "Value" ".1uF"
+		(property "Value" "0.1uF"
 			(at 429.26 231.1462 0)
 			(show_name no)
@@
 			)
 		)
-		(property "Value" ".1uF"
+		(property "Value" "0.1uF"
 			(at 45.7263 181.61 90)
 			(show_name no)
@@
 			)
 		)
-		(property "LCSC" "C2928167"
+		(property "LCSC" "C42924166"
 			(at 405.13 370.84 0)
 			(hide yes)
@@
 			)
 		)
-		(property "Value" ".1uF"
+		(property "Value" "0.1uF"
 			(at 227.3363 251.46 90)
 			(show_name no)
@@
 			)
 		)
-		(property "Value" ".1uF"
+		(property "Value" "0.1uF"
 			(at 184.1563 182.88 90)
 			(show_name no)
@@
 			)
 		)
-		(property "LCSC" "C2928167"
+		(property "LCSC" "C42924166"
 			(at 359.41 370.84 0)
 			(hide yes)
@@
 			)
 		)
-		(property "Value" ".1uF"
+		(property "Value" "0.1uF"
 			(at 140.9763 251.46 90)
 			(show_name no)
@@
 			)
 		)
-		(property "Value" ".1uF"
+		(property "Value" "0.1uF"
 			(at 97.7963 251.46 90)
 			(show_name no)
@@
 			)
 		)
-		(property "Value" ".1uF"
+		(property "Value" "0.1uF"
 			(at 184.1563 251.46 90)
 			(show_name no)
@@
 			)
 		)
-		(property "Value" ".1uF"
+		(property "Value" "0.1uF"
 			(at 45.7263 250.19 90)
 			(show_name no)
@@
 			)
 		)
-		(property "LCSC" "C2928167"
+		(property "LCSC" "C42924166"
 			(at 420.37 364.49 0)
 			(hide yes)
@@
 			)
 		)
-		(property "LCSC" "C2928167"
+		(property "LCSC" "C42924166"
 			(at 374.65 370.84 0)
 			(hide yes)
@@
 			)
 		)
-		(property "Value" ".1uF"
+		(property "Value" "0.1uF"
 			(at 140.9763 182.88 90)
 			(show_name no)
@@
 			)
 		)
-		(property "LCSC" "C2928167"
+		(property "LCSC" "C42924166"
 			(at 405.13 364.49 0)
 			(hide yes)
@@
 			)
 		)
-		(property "LCSC" "C2928167"
+		(property "LCSC" "C42924166"
 			(at 420.37 370.84 0)
 			(hide yes)
@@
 			)
 		)
-		(property "Value" ".1uF"
+		(property "Value" "0.1uF"
 			(at 97.7963 182.88 90)
 			(show_name no)
